Commit message: sentinel bouquet of branches

File: data/sentinel2.urdf (robot description, URDF)
Before this commit: robot sentinel, 72 links, 71 joints
Links:
- removed link branch_50
- removed link branch_50_sphere
- removed link branch_51
- removed link branch_51_sphere
- removed link branch_52
- removed link branch_52_sphere
- removed link branch_53
- removed link branch_53_sphere
- removed link branch_54
- removed link branch_54_sphere
- removed link branch_60
- removed link branch_60_sphere
- removed link branch_61
- removed link branch_61_sphere
- removed link branch_62
- removed link branch_62_sphere
- removed link branch_63
- removed link branch_63_sphere
- removed link branch_64
- removed link branch_64_sphere
- added link branch_00_spherical_joint_link, mass 0.05; collision sphere radius=0.01; visual sphere radius=0.01
- added link branch_01_spherical_joint_link, mass 0.05; collision sphere radius=0.01; visual sphere radius=0.01
- added link branch_02_spherical_joint_link, mass 0.05; collision sphere radius=0.01; visual sphere radius=0.01
- added link branch_03_spherical_joint_link, mass 0.05; collision sphere radius=0.01; visual sphere radius=0.01
- added link branch_10_spherical_joint_link, mass 0.05; collision sphere radius=0.01; visual sphere radius=0.01
- added link branch_11_spherical_joint_link, mass 0.05; collision sphere radius=0.01; visual sphere radius=0.01
- added link branch_12_spherical_joint_link, mass 0.05; collision sphere radius=0.01; visual sphere radius=0.01
- added link branch_13_spherical_joint_link, mass 0.05; collision sphere radius=0.01; visual sphere radius=0.01
- added link branch_20_spherical_joint_link, mass 0.05; collision sphere radius=0.01; visual sphere radius=0.01
- added link branch_21_spherical_joint_link, mass 0.05; collision sphere radius=0.01; visual sphere radius=0.01
- added link branch_22_spherical_joint_link, mass 0.05; collision sphere radius=0.01; visual sphere radius=0.01
- added link branch_23_spherical_joint_link, mass 0.05; collision sphere radius=0.01; visual sphere radius=0.01
- added link branch_30_spherical_joint_link, mass 0.05; collision sphere radius=0.01; visual sphere radius=0.01
- added link branch_31_spherical_joint_link, mass 0.05; collision sphere radius=0.01; visual sphere radius=0.01
- added link branch_32_spherical_joint_link, mass 0.05; collision sphere radius=0.01; visual sphere radius=0.01
- added link branch_33_spherical_joint_link, mass 0.05; collision sphere radius=0.01; visual sphere radius=0.01
- added link branch_40_spherical_joint_link, mass 0.05; collision sphere radius=0.01; visual sphere radius=0.01
- added link branch_41_spherical_joint_link, mass 0.05; collision sphere radius=0.01; visual sphere radius=0.01
- added link branch_42_spherical_joint_link, mass 0.05; collision sphere radius=0.01; visual sphere radius=0.01
- added link branch_43_spherical_joint_link, mass 0.05; collision sphere radius=0.01; visual sphere radius=0.01
- link branch_00: mass 1 -> 0.05; geometry collision cylinder length=0.15 radius=0.01; visual cylinder length=0.15 radius=0.01
- link branch_00_sphere: mass 1 -> 0.05; geometry collision sphere radius=0.02; visual sphere radius=0.02
- link branch_01: mass 1 -> 0.05; geometry collision cylinder length=0.15 radius=0.01; visual cylinder length=0.15 radius=0.01
- link branch_01_sphere: mass 1 -> 0.05; geometry collision sphere radius=0.02; visual sphere radius=0.02
- link branch_02: mass 1 -> 0.05; geometry collision cylinder length=0.15 radius=0.01; visual cylinder length=0.15 radius=0.01
- link branch_02_sphere: mass 1 -> 0.05; geometry collision sphere radius=0.02; visual sphere radius=0.02
- link branch_03: mass 1 -> 0.05; geometry collision cylinder length=0.15 radius=0.01; visual cylinder length=0.15 radius=0.01
- link branch_03_sphere: mass 1 -> 0.05; geometry collision sphere radius=0.02; visual sphere radius=0.02
- link branch_04: mass 1 -> 0.05; geometry collision cylinder length=0.15 radius=0.01; visual cylinder length=0.15 radius=0.01
- link branch_04_sphere: mass 1 -> 0.05; geometry collision sphere radius=0.02; visual sphere radius=0.02
- link branch_10: mass 1 -> 0.05; geometry collision cylinder length=0.15 radius=0.01; visual cylinder length=0.15 radius=0.01
- link branch_10_sphere: mass 1 -> 0.05; geometry collision sphere radius=0.02; visual sphere radius=0.02
- link branch_11: mass 1 -> 0.05; geometry collision cylinder length=0.15 radius=0.01; visual cylinder length=0.15 radius=0.01
- link branch_11_sphere: mass 1 -> 0.05; geometry collision sphere radius=0.02; visual sphere radius=0.02
- link branch_12: mass 1 -> 0.05; geometry collision cylinder length=0.15 radius=0.01; visual cylinder length=0.15 radius=0.01
- link branch_12_sphere: mass 1 -> 0.05; geometry collision sphere radius=0.02; visual sphere radius=0.02
- link branch_13: mass 1 -> 0.05; geometry collision cylinder length=0.15 radius=0.01; visual cylinder length=0.15 radius=0.01
- link branch_13_sphere: mass 1 -> 0.05; geometry collision sphere radius=0.02; visual sphere radius=0.02
- link branch_14: mass 1 -> 0.05; geometry collision cylinder length=0.15 radius=0.01; visual cylinder length=0.15 radius=0.01
- link branch_14_sphere: mass 1 -> 0.05; geometry collision sphere radius=0.02; visual sphere radius=0.02
- link branch_20: mass 1 -> 0.05; geometry collision cylinder length=0.15 radius=0.01; visual cylinder length=0.15 radius=0.01
- link branch_20_sphere: mass 1 -> 0.05; geometry collision sphere radius=0.02; visual sphere radius=0.02
- link branch_21: mass 1 -> 0.05; geometry collision cylinder length=0.15 radius=0.01; visual cylinder length=0.15 radius=0.01
- link branch_21_sphere: mass 1 -> 0.05; geometry collision sphere radius=0.02; visual sphere radius=0.02
- link branch_22: mass 1 -> 0.05; geometry collision cylinder length=0.15 radius=0.01; visual cylinder length=0.15 radius=0.01
- link branch_22_sphere: mass 1 -> 0.05; geometry collision sphere radius=0.02; visual sphere radius=0.02
- link branch_23: mass 1 -> 0.05; geometry collision cylinder length=0.15 radius=0.01; visual cylinder length=0.15 radius=0.01
- link branch_23_sphere: mass 1 -> 0.05; geometry collision sphere radius=0.02; visual sphere radius=0.02
- link branch_24: mass 1 -> 0.05; geometry collision cylinder length=0.15 radius=0.01; visual cylinder length=0.15 radius=0.01
- link branch_24_sphere: mass 1 -> 0.05; geometry collision sphere radius=0.02; visual sphere radius=0.02
- link branch_30: mass 1 -> 0.05; geometry collision cylinder length=0.15 radius=0.01; visual cylinder length=0.15 radius=0.01
- link branch_30_sphere: mass 1 -> 0.05; geometry collision sphere radius=0.02; visual sphere radius=0.02
- link branch_31: mass 1 -> 0.05; geometry collision cylinder length=0.15 radius=0.01; visual cylinder length=0.15 radius=0.01
- link branch_31_sphere: mass 1 -> 0.05; geometry collision sphere radius=0.02; visual sphere radius=0.02
- link branch_32: mass 1 -> 0.05; geometry collision cylinder length=0.15 radius=0.01; visual cylinder length=0.15 radius=0.01
- link branch_32_sphere: mass 1 -> 0.05; geometry collision sphere radius=0.02; visual sphere radius=0.02
- link branch_33: mass 1 -> 0.05; geometry collision cylinder length=0.15 radius=0.01; visual cylinder length=0.15 radius=0.01
- link branch_33_sphere: mass 1 -> 0.05; geometry collision sphere radius=0.02; visual sphere radius=0.02
- link branch_34: mass 1 -> 0.05; geometry collision cylinder length=0.15 radius=0.01; visual cylinder length=0.15 radius=0.01
- link branch_34_sphere: mass 1 -> 0.05; geometry collision sphere radius=0.02; visual sphere radius=0.02
- link branch_40: mass 1 -> 0.05; geometry collision cylinder length=0.15 radius=0.01; visual cylinder length=0.15 radius=0.01
- link branch_40_sphere: mass 1 -> 0.05; geometry collision sphere radius=0.02; visual sphere radius=0.02
- link branch_41: mass 1 -> 0.05; geometry collision cylinder length=0.15 radius=0.01; visual cylinder length=0.15 radius=0.01
- link branch_41_sphere: mass 1 -> 0.05; geometry collision sphere radius=0.02; visual sphere radius=0.02
- link branch_42: mass 1 -> 0.05; geometry collision cylinder length=0.15 radius=0.01; visual cylinder length=0.15 radius=0.01
- link branch_42_sphere: mass 1 -> 0.05; geometry collision sphere radius=0.02; visual sphere radius=0.02
- link branch_43: mass 1 -> 0.05; geometry collision cylinder length=0.15 radius=0.01; visual cylinder length=0.15 radius=0.01
- link branch_43_sphere: mass 1 -> 0.05; geometry collision sphere radius=0.02; visual sphere radius=0.02
- link branch_44: mass 1 -> 0.05; geometry collision cylinder length=0.15 radius=0.01; visual cylinder length=0.15 radius=0.01
- link branch_44_sphere: mass 1 -> 0.05; geometry collision sphere radius=0.02; visual sphere radius=0.02
- link eye: mass 1 -> 0.05
- link head: mass 1 -> 0.05
Joints:
- removed joint branch_00_branch_01_joint_revolute
- removed joint branch_01_branch_02_joint_revolute
- removed joint branch_02_branch_03_joint_revolute
- removed joint branch_03_branch_04_joint_revolute
- removed joint branch_10_branch_11_joint_revolute
- removed joint branch_11_branch_12_joint_revolute
- removed joint branch_12_branch_13_joint_revolute
- removed joint branch_13_branch_14_joint_revolute
- removed joint branch_20_branch_21_joint_revolute
- removed joint branch_21_branch_22_joint_revolute
- removed joint branch_22_branch_23_joint_revolute
- removed joint branch_23_branch_24_joint_revolute
- removed joint branch_30_branch_31_joint_revolute
- removed joint branch_31_branch_32_joint_revolute
- removed joint branch_32_branch_33_joint_revolute
- removed joint branch_33_branch_34_joint_revolute
- removed joint branch_40_branch_41_joint_revolute
- removed joint branch_41_branch_42_joint_revolute
- removed joint branch_42_branch_43_joint_revolute
- removed joint branch_43_branch_44_joint_revolute
- removed joint branch_50_branch_51_joint_revolute
- removed joint branch_50_fixed
- removed joint branch_51_branch_52_joint_revolute
- removed joint branch_51_fixed
- removed joint branch_52_branch_53_joint_revolute
- removed joint branch_52_fixed
- removed joint branch_53_branch_54_joint_revolute
- removed joint branch_53_fixed
- removed joint branch_54_fixed
- removed joint branch_60_branch_61_joint_revolute
- removed joint branch_60_fixed
- removed joint branch_61_branch_62_joint_revolute
- removed joint branch_61_fixed
- removed joint branch_62_branch_63_joint_revolute
- removed joint branch_62_fixed
- removed joint branch_63_branch_64_joint_revolute
- removed joint branch_63_fixed
- removed joint branch_64_fixed
- removed joint head_branch_50_joint
- removed joint head_branch_60_joint
- added joint branch_00_branch_01_joint_revolute_X: type revolute, parent branch_00_spherical_joint_link, child branch_01, origin xyz=0 0 0 rpy=0 0 0, axis 0 0 1, limit lower=-1.57 upper=1.57 effort=0.01 velocity=1000
- added joint branch_00_branch_01_joint_revolute_Y: type revolute, parent branch_00, child branch_00_spherical_joint_link, origin xyz=-0.15 0 0 rpy=0 0 0, axis 0 1 0, limit lower=-1.57 upper=1.57 effort=0.01 velocity=1000
- added joint branch_01_branch_02_joint_revolute_X: type revolute, parent branch_01_spherical_joint_link, child branch_02, origin xyz=0 0 0 rpy=0 0 0, axis 0 0 1, limit lower=-1.57 upper=1.57 effort=0.01 velocity=1000
- added joint branch_01_branch_02_joint_revolute_Y: type revolute, parent branch_01, child branch_01_spherical_joint_link, origin xyz=-0.15 0 0 rpy=0 0 0, axis 0 1 0, limit lower=-1.57 upper=1.57 effort=0.01 velocity=1000
- added joint branch_02_branch_03_joint_revolute_X: type revolute, parent branch_02_spherical_joint_link, child branch_03, origin xyz=0 0 0 rpy=0 0 0, axis 0 0 1, limit lower=-1.57 upper=1.57 effort=0.01 velocity=1000
- added joint branch_02_branch_03_joint_revolute_Y: type revolute, parent branch_02, child branch_02_spherical_joint_link, origin xyz=-0.15 0 0 rpy=0 0 0, axis 0 1 0, limit lower=-1.57 upper=1.57 effort=0.01 velocity=1000
- added joint branch_03_branch_04_joint_revolute_X: type revolute, parent branch_03_spherical_joint_link, child branch_04, origin xyz=0 0 0 rpy=0 0 0, axis 0 0 1, limit lower=-1.57 upper=1.57 effort=0.01 velocity=1000
- added joint branch_03_branch_04_joint_revolute_Y: type revolute, parent branch_03, child branch_03_spherical_joint_link, origin xyz=-0.15 0 0 rpy=0 0 0, axis 0 1 0, limit lower=-1.57 upper=1.57 effort=0.01 velocity=1000
- added joint branch_10_branch_11_joint_revolute_X: type revolute, parent branch_10_spherical_joint_link, child branch_11, origin xyz=0 0 0 rpy=0 0 0, axis 0 0 1, limit lower=-1.57 upper=1.57 effort=0.01 velocity=1000
- added joint branch_10_branch_11_joint_revolute_Y: type revolute, parent branch_10, child branch_10_spherical_joint_link, origin xyz=-0.15 0 0 rpy=0 0 0, axis 0 1 0, limit lower=-1.57 upper=1.57 effort=0.01 velocity=1000
- added joint branch_11_branch_12_joint_revolute_X: type revolute, parent branch_11_spherical_joint_link, child branch_12, origin xyz=0 0 0 rpy=0 0 0, axis 0 0 1, limit lower=-1.57 upper=1.57 effort=0.01 velocity=1000
- added joint branch_11_branch_12_joint_revolute_Y: type revolute, parent branch_11, child branch_11_spherical_joint_link, origin xyz=-0.15 0 0 rpy=0 0 0, axis 0 1 0, limit lower=-1.57 upper=1.57 effort=0.01 velocity=1000
- added joint branch_12_branch_13_joint_revolute_X: type revolute, parent branch_12_spherical_joint_link, child branch_13, origin xyz=0 0 0 rpy=0 0 0, axis 0 0 1, limit lower=-1.57 upper=1.57 effort=0.01 velocity=1000
- added joint branch_12_branch_13_joint_revolute_Y: type revolute, parent branch_12, child branch_12_spherical_joint_link, origin xyz=-0.15 0 0 rpy=0 0 0, axis 0 1 0, limit lower=-1.57 upper=1.57 effort=0.01 velocity=1000
- added joint branch_13_branch_14_joint_revolute_X: type revolute, parent branch_13_spherical_joint_link, child branch_14, origin xyz=0 0 0 rpy=0 0 0, axis 0 0 1, limit lower=-1.57 upper=1.57 effort=0.01 velocity=1000
- added joint branch_13_branch_14_joint_revolute_Y: type revolute, parent branch_13, child branch_13_spherical_joint_link, origin xyz=-0.15 0 0 rpy=0 0 0, axis 0 1 0, limit lower=-1.57 upper=1.57 effort=0.01 velocity=1000
- added joint branch_20_branch_21_joint_revolute_X: type revolute, parent branch_20_spherical_joint_link, child branch_21, origin xyz=0 0 0 rpy=0 0 0, axis 0 0 1, limit lower=-1.57 upper=1.57 effort=0.01 velocity=1000
- added joint branch_20_branch_21_joint_revolute_Y: type revolute, parent branch_20, child branch_20_spherical_joint_link, origin xyz=-0.15 0 0 rpy=0 0 0, axis 0 1 0, limit lower=-1.57 upper=1.57 effort=0.01 velocity=1000
- added joint branch_21_branch_22_joint_revolute_X: type revolute, parent branch_21_spherical_joint_link, child branch_22, origin xyz=0 0 0 rpy=0 0 0, axis 0 0 1, limit lower=-1.57 upper=1.57 effort=0.01 velocity=1000
- added joint branch_21_branch_22_joint_revolute_Y: type revolute, parent branch_21, child branch_21_spherical_joint_link, origin xyz=-0.15 0 0 rpy=0 0 0, axis 0 1 0, limit lower=-1.57 upper=1.57 effort=0.01 velocity=1000
- added joint branch_22_branch_23_joint_revolute_X: type revolute, parent branch_22_spherical_joint_link, child branch_23, origin xyz=0 0 0 rpy=0 0 0, axis 0 0 1, limit lower=-1.57 upper=1.57 effort=0.01 velocity=1000
- added joint branch_22_branch_23_joint_revolute_Y: type revolute, parent branch_22, child branch_22_spherical_joint_link, origin xyz=-0.15 0 0 rpy=0 0 0, axis 0 1 0, limit lower=-1.57 upper=1.57 effort=0.01 velocity=1000
- added joint branch_23_branch_24_joint_revolute_X: type revolute, parent branch_23_spherical_joint_link, child branch_24, origin xyz=0 0 0 rpy=0 0 0, axis 0 0 1, limit lower=-1.57 upper=1.57 effort=0.01 velocity=1000
- added joint branch_23_branch_24_joint_revolute_Y: type revolute, parent branch_23, child branch_23_spherical_joint_link, origin xyz=-0.15 0 0 rpy=0 0 0, axis 0 1 0, limit lower=-1.57 upper=1.57 effort=0.01 velocity=1000
- added joint branch_30_branch_31_joint_revolute_X: type revolute, parent branch_30_spherical_joint_link, child branch_31, origin xyz=0 0 0 rpy=0 0 0, axis 0 0 1, limit lower=-1.57 upper=1.57 effort=0.01 velocity=1000
- added joint branch_30_branch_31_joint_revolute_Y: type revolute, parent branch_30, child branch_30_spherical_joint_link, origin xyz=-0.15 0 0 rpy=0 0 0, axis 0 1 0, limit lower=-1.57 upper=1.57 effort=0.01 velocity=1000
- added joint branch_31_branch_32_joint_revolute_X: type revolute, parent branch_31_spherical_joint_link, child branch_32, origin xyz=0 0 0 rpy=0 0 0, axis 0 0 1, limit lower=-1.57 upper=1.57 effort=0.01 velocity=1000
- added joint branch_31_branch_32_joint_revolute_Y: type revolute, parent branch_31, child branch_31_spherical_joint_link, origin xyz=-0.15 0 0 rpy=0 0 0, axis 0 1 0, limit lower=-1.57 upper=1.57 effort=0.01 velocity=1000
- added joint branch_32_branch_33_joint_revolute_X: type revolute, parent branch_32_spherical_joint_link, child branch_33, origin xyz=0 0 0 rpy=0 0 0, axis 0 0 1, limit lower=-1.57 upper=1.57 effort=0.01 velocity=1000
- added joint branch_32_branch_33_joint_revolute_Y: type revolute, parent branch_32, child branch_32_spherical_joint_link, origin xyz=-0.15 0 0 rpy=0 0 0, axis 0 1 0, limit lower=-1.57 upper=1.57 effort=0.01 velocity=1000
- added joint branch_33_branch_34_joint_revolute_X: type revolute, parent branch_33_spherical_joint_link, child branch_34, origin xyz=0 0 0 rpy=0 0 0, axis 0 0 1, limit lower=-1.57 upper=1.57 effort=0.01 velocity=1000
- added joint branch_33_branch_34_joint_revolute_Y: type revolute, parent branch_33, child branch_33_spherical_joint_link, origin xyz=-0.15 0 0 rpy=0 0 0, axis 0 1 0, limit lower=-1.57 upper=1.57 effort=0.01 velocity=1000
- added joint branch_40_branch_41_joint_revolute_X: type revolute, parent branch_40_spherical_joint_link, child branch_41, origin xyz=0 0 0 rpy=0 0 0, axis 0 0 1, limit lower=-1.57 upper=1.57 effort=0.01 velocity=1000
- added joint branch_40_branch_41_joint_revolute_Y: type revolute, parent branch_40, child branch_40_spherical_joint_link, origin xyz=-0.15 0 0 rpy=0 0 0, axis 0 1 0, limit lower=-1.57 upper=1.57 effort=0.01 velocity=1000
- added joint branch_41_branch_42_joint_revolute_X: type revolute, parent branch_41_spherical_joint_link, child branch_42, origin xyz=0 0 0 rpy=0 0 0, axis 0 0 1, limit lower=-1.57 upper=1.57 effort=0.01 velocity=1000
- added joint branch_41_branch_42_joint_revolute_Y: type revolute, parent branch_41, child branch_41_spherical_joint_link, origin xyz=-0.15 0 0 rpy=0 0 0, axis 0 1 0, limit lower=-1.57 upper=1.57 effort=0.01 velocity=1000
- added joint branch_42_branch_43_joint_revolute_X: type revolute, parent branch_42_spherical_joint_link, child branch_43, origin xyz=0 0 0 rpy=0 0 0, axis 0 0 1, limit lower=-1.57 upper=1.57 effort=0.01 velocity=1000
- added joint branch_42_branch_43_joint_revolute_Y: type revolute, parent branch_42, child branch_42_spherical_joint_link, origin xyz=-0.15 0 0 rpy=0 0 0, axis 0 1 0, limit lower=-1.57 upper=1.57 effort=0.01 velocity=1000
- added joint branch_43_branch_44_joint_revolute_X: type revolute, parent branch_43_spherical_joint_link, child branch_44, origin xyz=0 0 0 rpy=0 0 0, axis 0 0 1, limit lower=-1.57 upper=1.57 effort=0.01 velocity=1000
- added joint branch_43_branch_44_joint_revolute_Y: type revolute, parent branch_43, child branch_43_spherical_joint_link, origin xyz=-0.15 0 0 rpy=0 0 0, axis 0 1 0, limit lower=-1.57 upper=1.57 effort=0.01 velocity=1000
- joint head_branch_00_joint: origin xyz=-0.1 0.08 0.0 rpy=0 0 0 -> xyz=-0.1 0.07 0.0 rpy=0 0 0
- joint head_branch_10_joint: origin xyz=-0.1 0.0498791841487 0.0625465185974 rpy=0 0 0 -> xyz=-0.1 0.0216311896062 0.0665739561407 rpy=0 0 0
- joint head_branch_20_joint: origin xyz=-0.1 -0.0178016747165 0.0779942329745 rpy=0 0 0 -> xyz=-0.1 -0.0566311896062 0.0411449676605 rpy=0 0 0
- joint head_branch_30_joint: origin xyz=-0.1 -0.0720775094322 0.0347106991294 rpy=0 0 0 -> xyz=-0.1 -0.0566311896062 -0.0411449676605 rpy=0 0 0
- joint head_branch_40_joint: origin xyz=-0.1 -0.0720775094322 -0.0347106991294 rpy=0 0 0 -> xyz=-0.1 0.0216311896062 -0.0665739561407 rpy=0 0 0
