Commit message: minor

File: data/sentinel2.urdf (robot description, URDF)
Before this commit: robot sentinel, 72 links, 71 joints
Links:
- removed link branch_01_spherical_joint_link
- removed link branch_02
- removed link branch_02_sphere
- removed link branch_02_spherical_joint_link
- removed link branch_03
- removed link branch_03_sphere
- removed link branch_03_spherical_joint_link
- removed link branch_04
- removed link branch_04_sphere
- removed link branch_10
- removed link branch_10_sphere
- removed link branch_10_spherical_joint_link
- removed link branch_11
- removed link branch_11_sphere
- removed link branch_11_spherical_joint_link
- removed link branch_12
- removed link branch_12_sphere
- removed link branch_12_spherical_joint_link
- removed link branch_13
- removed link branch_13_sphere
- removed link branch_13_spherical_joint_link
- removed link branch_14
- removed link branch_14_sphere
- removed link branch_20
- removed link branch_20_sphere
- removed link branch_20_spherical_joint_link
- removed link branch_21
- removed link branch_21_sphere
- removed link branch_21_spherical_joint_link
- removed link branch_22
- removed link branch_22_sphere
- removed link branch_22_spherical_joint_link
- removed link branch_23
- removed link branch_23_sphere
- removed link branch_23_spherical_joint_link
- removed link branch_24
- removed link branch_24_sphere
- removed link branch_30
- removed link branch_30_sphere
- removed link branch_30_spherical_joint_link
- removed link branch_31
- removed link branch_31_sphere
- removed link branch_31_spherical_joint_link
- removed link branch_32
- removed link branch_32_sphere
- removed link branch_32_spherical_joint_link
- removed link branch_33
- removed link branch_33_sphere
- removed link branch_33_spherical_joint_link
- removed link branch_34
- removed link branch_34_sphere
- removed link branch_40
- removed link branch_40_sphere
- removed link branch_40_spherical_joint_link
- removed link branch_41
- removed link branch_41_sphere
- removed link branch_41_spherical_joint_link
- removed link branch_42
- removed link branch_42_sphere
- removed link branch_42_spherical_joint_link
- removed link branch_43
- removed link branch_43_sphere
- removed link branch_43_spherical_joint_link
- removed link branch_44
- removed link branch_44_sphere
Joints:
- removed joint branch_01_branch_02_joint_revolute_X
- removed joint branch_01_branch_02_joint_revolute_Y
- removed joint branch_02_branch_03_joint_revolute_X
- removed joint branch_02_branch_03_joint_revolute_Y
- removed joint branch_02_fixed
- removed joint branch_03_branch_04_joint_revolute_X
- removed joint branch_03_branch_04_joint_revolute_Y
- removed joint branch_03_fixed
- removed joint branch_04_fixed
- removed joint branch_10_branch_11_joint_revolute_X
- removed joint branch_10_branch_11_joint_revolute_Y
- removed joint branch_10_fixed
- removed joint branch_11_branch_12_joint_revolute_X
- removed joint branch_11_branch_12_joint_revolute_Y
- removed joint branch_11_fixed
- removed joint branch_12_branch_13_joint_revolute_X
- removed joint branch_12_branch_13_joint_revolute_Y
- removed joint branch_12_fixed
- removed joint branch_13_branch_14_joint_revolute_X
- removed joint branch_13_branch_14_joint_revolute_Y
- removed joint branch_13_fixed
- removed joint branch_14_fixed
- removed joint branch_20_branch_21_joint_revolute_X
- removed joint branch_20_branch_21_joint_revolute_Y
- removed joint branch_20_fixed
- removed joint branch_21_branch_22_joint_revolute_X
- removed joint branch_21_branch_22_joint_revolute_Y
- removed joint branch_21_fixed
- removed joint branch_22_branch_23_joint_revolute_X
- removed joint branch_22_branch_23_joint_revolute_Y
- removed joint branch_22_fixed
- removed joint branch_23_branch_24_joint_revolute_X
- removed joint branch_23_branch_24_joint_revolute_Y
- removed joint branch_23_fixed
- removed joint branch_24_fixed
- removed joint branch_30_branch_31_joint_revolute_X
- removed joint branch_30_branch_31_joint_revolute_Y
- removed joint branch_30_fixed
- removed joint branch_31_branch_32_joint_revolute_X
- removed joint branch_31_branch_32_joint_revolute_Y
- removed joint branch_31_fixed
- removed joint branch_32_branch_33_joint_revolute_X
- removed joint branch_32_branch_33_joint_revolute_Y
- removed joint branch_32_fixed
- removed joint branch_33_branch_34_joint_revolute_X
- removed joint branch_33_branch_34_joint_revolute_Y
- removed joint branch_33_fixed
- removed joint branch_34_fixed
- removed joint branch_40_branch_41_joint_revolute_X
- removed joint branch_40_branch_41_joint_revolute_Y
- removed joint branch_40_fixed
- removed joint branch_41_branch_42_joint_revolute_X
- removed joint branch_41_branch_42_joint_revolute_Y
- removed joint branch_41_fixed
- removed joint branch_42_branch_43_joint_revolute_X
- removed joint branch_42_branch_43_joint_revolute_Y
- removed joint branch_42_fixed
- removed joint branch_43_branch_44_joint_revolute_X
- removed joint branch_43_branch_44_joint_revolute_Y
- removed joint branch_43_fixed
- removed joint branch_44_fixed
- removed joint head_branch_10_joint
- removed joint head_branch_20_joint
- removed joint head_branch_30_joint
- removed joint head_branch_40_joint

Commit message: fixed sentinel

File: data/sentinel2.urdf (robot description, URDF)
Before this commit: robot sentinel, 7 links, 6 joints
Links:
- removed link branch_00_sphere
- removed link branch_01_sphere
- added link branch_00_cylinder, mass 0.05; collision cylinder length=0.15 radius=0.01; visual cylinder length=0.15 radius=0.01
- added link branch_01_cylinder, mass 0.05; collision cylinder length=0.15 radius=0.01; visual cylinder length=0.15 radius=0.01
- added link branch_01_spherical_joint_link, mass 0.05; collision sphere radius=0.01; visual sphere radius=0.01
- added link branch_02, mass 0.05; collision sphere radius=0.02; visual sphere radius=0.02
- added link branch_02_cylinder, mass 0.05; collision cylinder length=0.15 radius=0.01; visual cylinder length=0.15 radius=0.01
- added link branch_02_spherical_joint_link, mass 0.05; collision sphere radius=0.01; visual sphere radius=0.01
- added link branch_03, mass 0.05; collision sphere radius=0.02; visual sphere radius=0.02
- added link branch_03_cylinder, mass 0.05; collision cylinder length=0.15 radius=0.01; visual cylinder length=0.15 radius=0.01
- added link branch_03_spherical_joint_link, mass 0.05; collision sphere radius=0.01; visual sphere radius=0.01
- added link branch_04, mass 0.05; collision sphere radius=0.02; visual sphere radius=0.02
- added link branch_04_cylinder, mass 0.05; collision cylinder length=0.15 radius=0.01; visual cylinder length=0.15 radius=0.01
- added link branch_10, mass 0.05; collision sphere radius=0.02; visual sphere radius=0.02
- added link branch_10_cylinder, mass 0.05; collision cylinder length=0.15 radius=0.01; visual cylinder length=0.15 radius=0.01
- added link branch_10_spherical_joint_link, mass 0.05; collision sphere radius=0.01; visual sphere radius=0.01
- added link branch_11, mass 0.05; collision sphere radius=0.02; visual sphere radius=0.02
- added link branch_11_cylinder, mass 0.05; collision cylinder length=0.15 radius=0.01; visual cylinder length=0.15 radius=0.01
- added link branch_11_spherical_joint_link, mass 0.05; collision sphere radius=0.01; visual sphere radius=0.01
- added link branch_12, mass 0.05; collision sphere radius=0.02; visual sphere radius=0.02
- added link branch_12_cylinder, mass 0.05; collision cylinder length=0.15 radius=0.01; visual cylinder length=0.15 radius=0.01
- added link branch_12_spherical_joint_link, mass 0.05; collision sphere radius=0.01; visual sphere radius=0.01
- added link branch_13, mass 0.05; collision sphere radius=0.02; visual sphere radius=0.02
- added link branch_13_cylinder, mass 0.05; collision cylinder length=0.15 radius=0.01; visual cylinder length=0.15 radius=0.01
- added link branch_13_spherical_joint_link, mass 0.05; collision sphere radius=0.01; visual sphere radius=0.01
- added link branch_14, mass 0.05; collision sphere radius=0.02; visual sphere radius=0.02
- added link branch_14_cylinder, mass 0.05; collision cylinder length=0.15 radius=0.01; visual cylinder length=0.15 radius=0.01
- added link branch_20, mass 0.05; collision sphere radius=0.02; visual sphere radius=0.02
- added link branch_20_cylinder, mass 0.05; collision cylinder length=0.15 radius=0.01; visual cylinder length=0.15 radius=0.01
- added link branch_20_spherical_joint_link, mass 0.05; collision sphere radius=0.01; visual sphere radius=0.01
- added link branch_21, mass 0.05; collision sphere radius=0.02; visual sphere radius=0.02
- added link branch_21_cylinder, mass 0.05; collision cylinder length=0.15 radius=0.01; visual cylinder length=0.15 radius=0.01
- added link branch_21_spherical_joint_link, mass 0.05; collision sphere radius=0.01; visual sphere radius=0.01
- added link branch_22, mass 0.05; collision sphere radius=0.02; visual sphere radius=0.02
- added link branch_22_cylinder, mass 0.05; collision cylinder length=0.15 radius=0.01; visual cylinder length=0.15 radius=0.01
- added link branch_22_spherical_joint_link, mass 0.05; collision sphere radius=0.01; visual sphere radius=0.01
- added link branch_23, mass 0.05; collision sphere radius=0.02; visual sphere radius=0.02
- added link branch_23_cylinder, mass 0.05; collision cylinder length=0.15 radius=0.01; visual cylinder length=0.15 radius=0.01
- added link branch_23_spherical_joint_link, mass 0.05; collision sphere radius=0.01; visual sphere radius=0.01
- added link branch_24, mass 0.05; collision sphere radius=0.02; visual sphere radius=0.02
- added link branch_24_cylinder, mass 0.05; collision cylinder length=0.15 radius=0.01; visual cylinder length=0.15 radius=0.01
- link branch_00: geometry collision sphere radius=0.02; visual sphere radius=0.02
- link branch_01: geometry collision sphere radius=0.02; visual sphere radius=0.02
Joints:
- added joint branch_01_branch_02_joint_revolute_X: type revolute, parent branch_01_spherical_joint_link, child branch_02_cylinder, origin xyz=0 0 0 rpy=0 0 0, axis 0 0 1, limit lower=-1.57 upper=1.57 effort=0.01 velocity=1000
- added joint branch_01_branch_02_joint_revolute_Y: type revolute, parent branch_01, child branch_01_spherical_joint_link, origin xyz=-0.15 0 0 rpy=0 0 0, axis 0 1 0, limit lower=-1.57 upper=1.57 effort=0.01 velocity=1000
- added joint branch_02_branch_03_joint_revolute_X: type revolute, parent branch_02_spherical_joint_link, child branch_03_cylinder, origin xyz=0 0 0 rpy=0 0 0, axis 0 0 1, limit lower=-1.57 upper=1.57 effort=0.01 velocity=1000
- added joint branch_02_branch_03_joint_revolute_Y: type revolute, parent branch_02, child branch_02_spherical_joint_link, origin xyz=-0.15 0 0 rpy=0 0 0, axis 0 1 0, limit lower=-1.57 upper=1.57 effort=0.01 velocity=1000
- added joint branch_02_fixed: type fixed, parent branch_02_cylinder, child branch_02, origin xyz=0 0 0 rpy=0 0 0
- added joint branch_03_branch_04_joint_revolute_X: type revolute, parent branch_03_spherical_joint_link, child branch_04_cylinder, origin xyz=0 0 0 rpy=0 0 0, axis 0 0 1, limit lower=-1.57 upper=1.57 effort=0.01 velocity=1000
- added joint branch_03_branch_04_joint_revolute_Y: type revolute, parent branch_03, child branch_03_spherical_joint_link, origin xyz=-0.15 0 0 rpy=0 0 0, axis 0 1 0, limit lower=-1.57 upper=1.57 effort=0.01 velocity=1000
- added joint branch_03_fixed: type fixed, parent branch_03_cylinder, child branch_03, origin xyz=0 0 0 rpy=0 0 0
- added joint branch_04_fixed: type fixed, parent branch_04_cylinder, child branch_04, origin xyz=0 0 0 rpy=0 0 0
- added joint branch_10_branch_11_joint_revolute_X: type revolute, parent branch_10_spherical_joint_link, child branch_11_cylinder, origin xyz=0 0 0 rpy=0 0 0, axis 0 0 1, limit lower=-1.57 upper=1.57 effort=0.01 velocity=1000
- added joint branch_10_branch_11_joint_revolute_Y: type revolute, parent branch_10, child branch_10_spherical_joint_link, origin xyz=-0.15 0 0 rpy=0 0 0, axis 0 1 0, limit lower=-1.57 upper=1.57 effort=0.01 velocity=1000
- added joint branch_10_fixed: type fixed, parent branch_10_cylinder, child branch_10, origin xyz=0 0 0 rpy=0 0 0
- added joint branch_11_branch_12_joint_revolute_X: type revolute, parent branch_11_spherical_joint_link, child branch_12_cylinder, origin xyz=0 0 0 rpy=0 0 0, axis 0 0 1, limit lower=-1.57 upper=1.57 effort=0.01 velocity=1000
- added joint branch_11_branch_12_joint_revolute_Y: type revolute, parent branch_11, child branch_11_spherical_joint_link, origin xyz=-0.15 0 0 rpy=0 0 0, axis 0 1 0, limit lower=-1.57 upper=1.57 effort=0.01 velocity=1000
- added joint branch_11_fixed: type fixed, parent branch_11_cylinder, child branch_11, origin xyz=0 0 0 rpy=0 0 0
- added joint branch_12_branch_13_joint_revolute_X: type revolute, parent branch_12_spherical_joint_link, child branch_13_cylinder, origin xyz=0 0 0 rpy=0 0 0, axis 0 0 1, limit lower=-1.57 upper=1.57 effort=0.01 velocity=1000
- added joint branch_12_branch_13_joint_revolute_Y: type revolute, parent branch_12, child branch_12_spherical_joint_link, origin xyz=-0.15 0 0 rpy=0 0 0, axis 0 1 0, limit lower=-1.57 upper=1.57 effort=0.01 velocity=1000
- added joint branch_12_fixed: type fixed, parent branch_12_cylinder, child branch_12, origin xyz=0 0 0 rpy=0 0 0
- added joint branch_13_branch_14_joint_revolute_X: type revolute, parent branch_13_spherical_joint_link, child branch_14_cylinder, origin xyz=0 0 0 rpy=0 0 0, axis 0 0 1, limit lower=-1.57 upper=1.57 effort=0.01 velocity=1000
- added joint branch_13_branch_14_joint_revolute_Y: type revolute, parent branch_13, child branch_13_spherical_joint_link, origin xyz=-0.15 0 0 rpy=0 0 0, axis 0 1 0, limit lower=-1.57 upper=1.57 effort=0.01 velocity=1000
- added joint branch_13_fixed: type fixed, parent branch_13_cylinder, child branch_13, origin xyz=0 0 0 rpy=0 0 0
- added joint branch_14_fixed: type fixed, parent branch_14_cylinder, child branch_14, origin xyz=0 0 0 rpy=0 0 0
- added joint branch_20_branch_21_joint_revolute_X: type revolute, parent branch_20_spherical_joint_link, child branch_21_cylinder, origin xyz=0 0 0 rpy=0 0 0, axis 0 0 1, limit lower=-1.57 upper=1.57 effort=0.01 velocity=1000
- added joint branch_20_branch_21_joint_revolute_Y: type revolute, parent branch_20, child branch_20_spherical_joint_link, origin xyz=-0.15 0 0 rpy=0 0 0, axis 0 1 0, limit lower=-1.57 upper=1.57 effort=0.01 velocity=1000
- added joint branch_20_fixed: type fixed, parent branch_20_cylinder, child branch_20, origin xyz=0 0 0 rpy=0 0 0
- added joint branch_21_branch_22_joint_revolute_X: type revolute, parent branch_21_spherical_joint_link, child branch_22_cylinder, origin xyz=0 0 0 rpy=0 0 0, axis 0 0 1, limit lower=-1.57 upper=1.57 effort=0.01 velocity=1000
- added joint branch_21_branch_22_joint_revolute_Y: type revolute, parent branch_21, child branch_21_spherical_joint_link, origin xyz=-0.15 0 0 rpy=0 0 0, axis 0 1 0, limit lower=-1.57 upper=1.57 effort=0.01 velocity=1000
- added joint branch_21_fixed: type fixed, parent branch_21_cylinder, child branch_21, origin xyz=0 0 0 rpy=0 0 0
- added joint branch_22_branch_23_joint_revolute_X: type revolute, parent branch_22_spherical_joint_link, child branch_23_cylinder, origin xyz=0 0 0 rpy=0 0 0, axis 0 0 1, limit lower=-1.57 upper=1.57 effort=0.01 velocity=1000
- added joint branch_22_branch_23_joint_revolute_Y: type revolute, parent branch_22, child branch_22_spherical_joint_link, origin xyz=-0.15 0 0 rpy=0 0 0, axis 0 1 0, limit lower=-1.57 upper=1.57 effort=0.01 velocity=1000
- added joint branch_22_fixed: type fixed, parent branch_22_cylinder, child branch_22, origin xyz=0 0 0 rpy=0 0 0
- added joint branch_23_branch_24_joint_revolute_X: type revolute, parent branch_23_spherical_joint_link, child branch_24_cylinder, origin xyz=0 0 0 rpy=0 0 0, axis 0 0 1, limit lower=-1.57 upper=1.57 effort=0.01 velocity=1000
- added joint branch_23_branch_24_joint_revolute_Y: type revolute, parent branch_23, child branch_23_spherical_joint_link, origin xyz=-0.15 0 0 rpy=0 0 0, axis 0 1 0, limit lower=-1.57 upper=1.57 effort=0.01 velocity=1000
- added joint branch_23_fixed: type fixed, parent branch_23_cylinder, child branch_23, origin xyz=0 0 0 rpy=0 0 0
- added joint branch_24_fixed: type fixed, parent branch_24_cylinder, child branch_24, origin xyz=0 0 0 rpy=0 0 0
- added joint head_branch_10_joint: type fixed, parent head, child branch_10_cylinder, origin xyz=-0.1 -0.025 0.0433012701892 rpy=0 0 0
- added joint head_branch_20_joint: type fixed, parent head, child branch_20_cylinder, origin xyz=-0.1 -0.025 -0.0433012701892 rpy=0 0 0
- joint branch_00_branch_01_joint_revolute_X: child branch_01 -> branch_01_cylinder
- joint branch_00_fixed: child branch_00_sphere -> branch_00; parent branch_00 -> branch_00_cylinder
- joint branch_01_fixed: child branch_01_sphere -> branch_01; origin xyz=-0.15 0 0 rpy=0 0 0 -> xyz=0 0 0 rpy=0 0 0; parent branch_01 -> branch_01_cylinder
- joint head_branch_00_joint: child branch_00 -> branch_00_cylinder; origin xyz=-0.1 0.07 0.0 rpy=0 0 0 -> xyz=-0.1 0.05 0.0 rpy=0 0 0

Commit message: fixed planning for custom urdf -- time reparameterization needs to be fixed

File: data/sentinel2.urdf (robot description, URDF)
Before this commit: robot sentinel, 44 links, 43 joints
Links:
- removed link branch_02_spherical_joint_link
- removed link branch_03
- removed link branch_03_cylinder
- removed link branch_03_spherical_joint_link
- removed link branch_04
- removed link branch_04_cylinder
- removed link branch_12_spherical_joint_link
- removed link branch_13
- removed link branch_13_cylinder
- removed link branch_13_spherical_joint_link
- removed link branch_14
- removed link branch_14_cylinder
- removed link branch_22_spherical_joint_link
- removed link branch_23
- removed link branch_23_cylinder
- removed link branch_23_spherical_joint_link
- removed link branch_24
- removed link branch_24_cylinder
- link branch_00: geometry collision sphere radius=0.019; visual sphere radius=0.019
- link branch_00_spherical_joint_link: geometry collision sphere radius=0.001; visual sphere radius=0.001
- link branch_01: geometry collision sphere radius=0.019; visual sphere radius=0.019
- link branch_01_spherical_joint_link: geometry collision sphere radius=0.001; visual sphere radius=0.001
- link branch_02: geometry collision sphere radius=0.019; visual sphere radius=0.019
- link branch_10: geometry collision sphere radius=0.019; visual sphere radius=0.019
- link branch_10_spherical_joint_link: geometry collision sphere radius=0.001; visual sphere radius=0.001
- link branch_11: geometry collision sphere radius=0.019; visual sphere radius=0.019
- link branch_11_spherical_joint_link: geometry collision sphere radius=0.001; visual sphere radius=0.001
- link branch_12: geometry collision sphere radius=0.019; visual sphere radius=0.019
- link branch_20: geometry collision sphere radius=0.019; visual sphere radius=0.019
- link branch_20_spherical_joint_link: geometry collision sphere radius=0.001; visual sphere radius=0.001
- link branch_21: geometry collision sphere radius=0.019; visual sphere radius=0.019
- link branch_21_spherical_joint_link: geometry collision sphere radius=0.001; visual sphere radius=0.001
- link branch_22: geometry collision sphere radius=0.019; visual sphere radius=0.019
Joints:
- removed joint branch_02_branch_03_joint_revolute_X
- removed joint branch_02_branch_03_joint_revolute_Y
- removed joint branch_03_branch_04_joint_revolute_X
- removed joint branch_03_branch_04_joint_revolute_Y
- removed joint branch_03_fixed
- removed joint branch_04_fixed
- removed joint branch_12_branch_13_joint_revolute_X
- removed joint branch_12_branch_13_joint_revolute_Y
- removed joint branch_13_branch_14_joint_revolute_X
- removed joint branch_13_branch_14_joint_revolute_Y
- removed joint branch_13_fixed
- removed joint branch_14_fixed
- removed joint branch_22_branch_23_joint_revolute_X
- removed joint branch_22_branch_23_joint_revolute_Y
- removed joint branch_23_branch_24_joint_revolute_X
- removed joint branch_23_branch_24_joint_revolute_Y
- removed joint branch_23_fixed
- removed joint branch_24_fixed
- joint branch_00_branch_01_joint_revolute_X: limit lower=-1.57 upper=1.57 effort=0.01 velocity=1000 -> lower=-1.57 upper=1.57 effort=0.01 velocity=100
- joint branch_00_branch_01_joint_revolute_Y: limit lower=-1.57 upper=1.57 effort=0.01 velocity=1000 -> lower=-1.57 upper=1.57 effort=0.01 velocity=100; origin xyz=-0.15 0 0 rpy=0 0 0 -> xyz=-0.17 0 0 rpy=0 0 0
- joint branch_01_branch_02_joint_revolute_X: limit lower=-1.57 upper=1.57 effort=0.01 velocity=1000 -> lower=-1.57 upper=1.57 effort=0.01 velocity=100
- joint branch_01_branch_02_joint_revolute_Y: limit lower=-1.57 upper=1.57 effort=0.01 velocity=1000 -> lower=-1.57 upper=1.57 effort=0.01 velocity=100; origin xyz=-0.15 0 0 rpy=0 0 0 -> xyz=-0.19 0 0 rpy=0 0 0
- joint branch_10_branch_11_joint_revolute_X: limit lower=-1.57 upper=1.57 effort=0.01 velocity=1000 -> lower=-1.57 upper=1.57 effort=0.01 velocity=100
- joint branch_10_branch_11_joint_revolute_Y: limit lower=-1.57 upper=1.57 effort=0.01 velocity=1000 -> lower=-1.57 upper=1.57 effort=0.01 velocity=100; origin xyz=-0.15 0 0 rpy=0 0 0 -> xyz=-0.17 0 0 rpy=0 0 0
- joint branch_11_branch_12_joint_revolute_X: limit lower=-1.57 upper=1.57 effort=0.01 velocity=1000 -> lower=-1.57 upper=1.57 effort=0.01 velocity=100
- joint branch_11_branch_12_joint_revolute_Y: limit lower=-1.57 upper=1.57 effort=0.01 velocity=1000 -> lower=-1.57 upper=1.57 effort=0.01 velocity=100; origin xyz=-0.15 0 0 rpy=0 0 0 -> xyz=-0.19 0 0 rpy=0 0 0
- joint branch_20_branch_21_joint_revolute_X: limit lower=-1.57 upper=1.57 effort=0.01 velocity=1000 -> lower=-1.57 upper=1.57 effort=0.01 velocity=100
- joint branch_20_branch_21_joint_revolute_Y: limit lower=-1.57 upper=1.57 effort=0.01 velocity=1000 -> lower=-1.57 upper=1.57 effort=0.01 velocity=100; origin xyz=-0.15 0 0 rpy=0 0 0 -> xyz=-0.17 0 0 rpy=0 0 0
- joint branch_21_branch_22_joint_revolute_X: limit lower=-1.57 upper=1.57 effort=0.01 velocity=1000 -> lower=-1.57 upper=1.57 effort=0.01 velocity=100
- joint branch_21_branch_22_joint_revolute_Y: limit lower=-1.57 upper=1.57 effort=0.01 velocity=1000 -> lower=-1.57 upper=1.57 effort=0.01 velocity=100; origin xyz=-0.15 0 0 rpy=0 0 0 -> xyz=-0.19 0 0 rpy=0 0 0
