Commit message: SE(3) planning seems to forward simulate correctly, but no solution found, need to investigate biased sampling towards goal

File: data/sentinel.urdf (robot description, URDF)
Before this commit: robot sentinel, 46 links, 45 joints
Links:
- removed link branch_00
- removed link branch_00_cylinder
- removed link branch_00_spherical_joint_link
- removed link branch_01
- removed link branch_01_cylinder
- removed link branch_01_spherical_joint_link
- removed link branch_02
- removed link branch_02_cylinder
- removed link branch_02_spherical_joint_link
- removed link branch_03
- removed link branch_03_cylinder
- removed link branch_10
- removed link branch_10_cylinder
- removed link branch_10_spherical_joint_link
- removed link branch_11
- removed link branch_11_cylinder
- removed link branch_11_spherical_joint_link
- removed link branch_12
- removed link branch_12_cylinder
- removed link branch_12_spherical_joint_link
- removed link branch_13
- removed link branch_13_cylinder
- removed link branch_20
- removed link branch_20_cylinder
- removed link branch_20_spherical_joint_link
- removed link branch_21
- removed link branch_21_cylinder
- removed link branch_21_spherical_joint_link
- removed link branch_22
- removed link branch_22_cylinder
- removed link branch_22_spherical_joint_link
- removed link branch_23
- removed link branch_23_cylinder
- removed link branch_30
- removed link branch_30_cylinder
- removed link branch_30_spherical_joint_link
- removed link branch_31
- removed link branch_31_cylinder
- removed link branch_31_spherical_joint_link
- removed link branch_32
- removed link branch_32_cylinder
- removed link branch_32_spherical_joint_link
- removed link branch_33
- removed link branch_33_cylinder
Joints:
- removed joint branch_00_branch_01_joint_revolute_X
- removed joint branch_00_branch_01_joint_revolute_Y
- removed joint branch_00_fixed
- removed joint branch_01_branch_02_joint_revolute_X
- removed joint branch_01_branch_02_joint_revolute_Y
- removed joint branch_01_fixed
- removed joint branch_02_branch_03_joint_revolute_X
- removed joint branch_02_branch_03_joint_revolute_Y
- removed joint branch_02_fixed
- removed joint branch_03_fixed
- removed joint branch_10_branch_11_joint_revolute_X
- removed joint branch_10_branch_11_joint_revolute_Y
- removed joint branch_10_fixed
- removed joint branch_11_branch_12_joint_revolute_X
- removed joint branch_11_branch_12_joint_revolute_Y
- removed joint branch_11_fixed
- removed joint branch_12_branch_13_joint_revolute_X
- removed joint branch_12_branch_13_joint_revolute_Y
- removed joint branch_12_fixed
- removed joint branch_13_fixed
- removed joint branch_20_branch_21_joint_revolute_X
- removed joint branch_20_branch_21_joint_revolute_Y
- removed joint branch_20_fixed
- removed joint branch_21_branch_22_joint_revolute_X
- removed joint branch_21_branch_22_joint_revolute_Y
- removed joint branch_21_fixed
- removed joint branch_22_branch_23_joint_revolute_X
- removed joint branch_22_branch_23_joint_revolute_Y
- removed joint branch_22_fixed
- removed joint branch_23_fixed
- removed joint branch_30_branch_31_joint_revolute_X
- removed joint branch_30_branch_31_joint_revolute_Y
- removed joint branch_30_fixed
- removed joint branch_31_branch_32_joint_revolute_X
- removed joint branch_31_branch_32_joint_revolute_Y
- removed joint branch_31_fixed
- removed joint branch_32_branch_33_joint_revolute_X
- removed joint branch_32_branch_33_joint_revolute_Y
- removed joint branch_32_fixed
- removed joint branch_33_fixed
- removed joint head_branch_00_joint
- removed joint head_branch_10_joint
- removed joint head_branch_20_joint
- removed joint head_branch_30_joint
