Commit message: refactored

File: data/snake.urdf (robot description, URDF)
Before this commit: robot snake, 28 links, 27 joints
Links:
- link body0_cylinder: geometry collision cylinder length=0.025 radius=0.075; visual cylinder length=0.025 radius=0.075
- link body1_cylinder: geometry collision cylinder length=0.1 radius=0.075; visual cylinder length=0.1 radius=0.075
- link body2_cylinder: geometry collision cylinder length=0.1 radius=0.0625; visual cylinder length=0.1 radius=0.0625
- link body3_cylinder: geometry collision cylinder length=0.1 radius=0.0520833333333; visual cylinder length=0.1 radius=0.0520833333333
- link body4_cylinder: geometry collision cylinder length=0.1 radius=0.0434027777778; visual cylinder length=0.1 radius=0.0434027777778
- link body5_cylinder: geometry collision cylinder length=0.1 radius=0.0361689814815; visual cylinder length=0.1 radius=0.0361689814815
- link body6_cylinder: geometry collision cylinder length=0.1 radius=0.0301408179012; visual cylinder length=0.1 radius=0.0301408179012
- link body7_cylinder: geometry collision cylinder length=0.1 radius=0.025117348251; visual cylinder length=0.1 radius=0.025117348251
- link body8_cylinder: geometry collision cylinder length=0.1 radius=0.0209311235425; visual cylinder length=0.1 radius=0.0209311235425
Joints:
- joint body0_body1_joint_revolute_Z: origin xyz=-0.05 0 0 rpy=0 0 0 -> xyz=-0.045 0 0 rpy=0 0 0
- joint body1_body2_joint_revolute_Z: origin xyz=-0.16 0 0 rpy=0 0 0 -> xyz=-0.14 0 0 rpy=0 0 0
- joint body2_body3_joint_revolute_Z: origin xyz=-0.16 0 0 rpy=0 0 0 -> xyz=-0.14 0 0 rpy=0 0 0
- joint body3_body4_joint_revolute_Z: origin xyz=-0.16 0 0 rpy=0 0 0 -> xyz=-0.14 0 0 rpy=0 0 0
- joint body4_body5_joint_revolute_Z: origin xyz=-0.16 0 0 rpy=0 0 0 -> xyz=-0.14 0 0 rpy=0 0 0
- joint body5_body6_joint_revolute_Z: origin xyz=-0.16 0 0 rpy=0 0 0 -> xyz=-0.14 0 0 rpy=0 0 0
- joint body6_body7_joint_revolute_Z: origin xyz=-0.16 0 0 rpy=0 0 0 -> xyz=-0.14 0 0 rpy=0 0 0
- joint body7_body8_joint_revolute_Z: origin xyz=-0.16 0 0 rpy=0 0 0 -> xyz=-0.14 0 0 rpy=0 0 0

File: data/snake_irreducible.urdf (robot description, URDF)
Before this commit: robot snake_irreducible, 4 links, 3 joints
Links:
- link body0_cylinder: geometry collision cylinder length=0.025 radius=0.075; visual cylinder length=0.025 radius=0.075

Commit message: minor

File: data/snake.urdf (robot description, URDF)
Before this commit: robot snake, 28 links, 27 joints
Links:
- link body0: mass 0.05 -> 1
- link body0_cylinder: mass 0.05 -> 1
- link body0_spherical_joint_link: mass 0.05 -> 1
- link body1: mass 0.05 -> 1
- link body1_cylinder: mass 0.05 -> 1
- link body1_spherical_joint_link: mass 0.05 -> 1
- link body2: mass 0.05 -> 1
- link body2_cylinder: mass 0.05 -> 1
- link body2_spherical_joint_link: mass 0.05 -> 1
- link body3: mass 0.05 -> 1
- link body3_cylinder: mass 0.05 -> 1
- link body3_spherical_joint_link: mass 0.05 -> 1
- link body4: mass 0.05 -> 1
- link body4_cylinder: mass 0.05 -> 1
- link body4_spherical_joint_link: mass 0.05 -> 1
- link body5: mass 0.05 -> 1
- link body5_cylinder: mass 0.05 -> 1
- link body5_spherical_joint_link: mass 0.05 -> 1
- link body6: mass 0.05 -> 1
- link body6_cylinder: mass 0.05 -> 1
- link body6_spherical_joint_link: mass 0.05 -> 1
- link body7: mass 0.05 -> 1
- link body7_cylinder: mass 0.05 -> 1
- link body7_spherical_joint_link: mass 0.05 -> 1
- link body8: mass 0.05 -> 1
- link body8_cylinder: mass 0.05 -> 1
- link eye: mass 0.05 -> 1
- link head: mass 0.05 -> 1

Commit message: simulated snake in turbine force field

File: data/snake.urdf (robot description, URDF)
Before this commit: robot snake, 28 links, 27 joints
Links:
- removed link body4_spherical_joint_link
- removed link body5
- removed link body5_cylinder
- removed link body5_spherical_joint_link
- removed link body6
- removed link body6_cylinder
- removed link body6_spherical_joint_link
- removed link body7
- removed link body7_cylinder
- removed link body7_spherical_joint_link
- removed link body8
- removed link body8_cylinder
- link body0: geometry collision sphere radius=0.095; visual sphere radius=0.095
- link body1: geometry collision sphere radius=0.095; visual sphere radius=0.095
- link body2: geometry collision sphere radius=0.095; visual sphere radius=0.095
- link body3: geometry collision sphere radius=0.095; visual sphere radius=0.095
- link body4: geometry collision sphere radius=0.095; visual sphere radius=0.095
Joints:
- removed joint body4_body5_joint_revolute_Y
- removed joint body4_body5_joint_revolute_Z
- removed joint body5_body6_joint_revolute_Y
- removed joint body5_body6_joint_revolute_Z
- removed joint body5_fixed
- removed joint body6_body7_joint_revolute_Y
- removed joint body6_body7_joint_revolute_Z
- removed joint body6_fixed
- removed joint body7_body8_joint_revolute_Y
- removed joint body7_body8_joint_revolute_Z
- removed joint body7_fixed
- removed joint body8_fixed
- joint body0_body1_joint_revolute_Z: origin xyz=-0.045 0 0 rpy=0 0 0 -> xyz=-0.125 0 0 rpy=0 0 0
- joint body1_body2_joint_revolute_Z: origin xyz=-0.14 0 0 rpy=0 0 0 -> xyz=-0.3 0 0 rpy=0 0 0
- joint body2_body3_joint_revolute_Z: origin xyz=-0.14 0 0 rpy=0 0 0 -> xyz=-0.3 0 0 rpy=0 0 0
- joint body3_body4_joint_revolute_Z: origin xyz=-0.14 0 0 rpy=0 0 0 -> xyz=-0.3 0 0 rpy=0 0 0

File: data/snake_irreducible.urdf (robot description, URDF)
Before this commit: robot snake_irreducible, 4 links, 3 joints
Links:
- link body0: mass 0.05 -> 1; geometry collision sphere radius=0.095; visual sphere radius=0.095
- link body0_cylinder: mass 0.05 -> 1
- link eye: mass 0.05 -> 1
- link head: mass 0.05 -> 1

Commit message: restructured planner output; still bug jet propulsion actuators

File: data/snake.urdf (robot description, URDF)
Before this commit: robot snake, 16 links, 15 joints
Links:
- removed link body0_spherical_joint_link
- removed link body1
- removed link body1_cylinder
- removed link body1_spherical_joint_link
- removed link body2
- removed link body2_cylinder
- removed link body2_spherical_joint_link
- removed link body3
- removed link body3_cylinder
- removed link body3_spherical_joint_link
- removed link body4
- removed link body4_cylinder
Joints:
- removed joint body0_body1_joint_revolute_Y
- removed joint body0_body1_joint_revolute_Z
- removed joint body1_body2_joint_revolute_Y
- removed joint body1_body2_joint_revolute_Z
- removed joint body1_fixed
- removed joint body2_body3_joint_revolute_Y
- removed joint body2_body3_joint_revolute_Z
- removed joint body2_fixed
- removed joint body3_body4_joint_revolute_Y
- removed joint body3_body4_joint_revolute_Z
- removed joint body3_fixed
- removed joint body4_fixed
