Commit message: fixed jet propulsion; visualized JP in gui as cone

File: data/bullet.urdf (robot description, URDF)
Before this commit: robot bullet, 2 links, 1 joints
Links:
- link head: geometry collision cylinder length=0.2 radius=0.1; visual cylinder length=0.2 radius=0.1

Commit message: torque based following seems to work, butincongruent behavior when turning around, check /w integrator

File: data/bullet.urdf (robot description, URDF)
Before this commit: robot bullet, 2 links, 1 joints
Links:
- link eye: mass 1 -> 0.5
- link head: mass 1 -> 0.5

Commit message: minor

File: data/bullet.urdf (robot description, URDF)
Before this commit: robot bullet, 2 links, 1 joints
Links:
- link eye: mass 0.5 -> 1
- link head: mass 0.5 -> 1

File: data/spider.urdf (robot description, URDF)
Before this commit: robot spider, 22 links, 21 joints
Links:
- link eye: geometry collision sphere radius=0.3; visual sphere radius=0.3
Joints:
- joint leg_0_link0_spherical_Y: limit lower=-0.785398163397 upper=0.785398163397 effort=0.5 velocity=100 -> lower=-0.196349540849 upper=0.196349540849 effort=1 velocity=100
- joint leg_0_link0_spherical_Z: limit lower=-0.785398163397 upper=0.785398163397 effort=0.5 velocity=100 -> lower=-0.196349540849 upper=0.196349540849 effort=1 velocity=100; origin xyz=0.6 0.0 0 rpy=0 0 0 -> xyz=0.4 0.0 0 rpy=0 0 0
- joint leg_0_link1_spherical_Y: limit lower=-0.785398163397 upper=0.785398163397 effort=0.5 velocity=100 -> lower=-0.196349540849 upper=0.196349540849 effort=1 velocity=100
- joint leg_0_link1_spherical_Z: limit lower=-0.785398163397 upper=0.785398163397 effort=0.5 velocity=100 -> lower=-0.196349540849 upper=0.196349540849 effort=1 velocity=100
- joint leg_1_link0_spherical_Y: limit lower=-0.785398163397 upper=0.785398163397 effort=0.5 velocity=100 -> lower=-0.196349540849 upper=0.196349540849 effort=1 velocity=100
- joint leg_1_link0_spherical_Z: limit lower=-0.785398163397 upper=0.785398163397 effort=0.5 velocity=100 -> lower=-0.196349540849 upper=0.196349540849 effort=1 velocity=100; origin xyz=-0.3 0.519615242271 0 rpy=0 0 0 -> xyz=-0.2 0.346410161514 0 rpy=0 0 0
- joint leg_1_link1_spherical_Y: limit lower=-0.785398163397 upper=0.785398163397 effort=0.5 velocity=100 -> lower=-0.196349540849 upper=0.196349540849 effort=1 velocity=100
- joint leg_1_link1_spherical_Z: limit lower=-0.785398163397 upper=0.785398163397 effort=0.5 velocity=100 -> lower=-0.196349540849 upper=0.196349540849 effort=1 velocity=100
- joint leg_2_link0_spherical_Y: limit lower=-0.785398163397 upper=0.785398163397 effort=0.5 velocity=100 -> lower=-0.196349540849 upper=0.196349540849 effort=1 velocity=100
- joint leg_2_link0_spherical_Z: limit lower=-0.785398163397 upper=0.785398163397 effort=0.5 velocity=100 -> lower=-0.196349540849 upper=0.196349540849 effort=1 velocity=100; origin xyz=-0.3 -0.519615242271 0 rpy=0 0 0 -> xyz=-0.2 -0.346410161514 0 rpy=0 0 0
- joint leg_2_link1_spherical_Y: limit lower=-0.785398163397 upper=0.785398163397 effort=0.5 velocity=100 -> lower=-0.196349540849 upper=0.196349540849 effort=1 velocity=100
- joint leg_2_link1_spherical_Z: limit lower=-0.785398163397 upper=0.785398163397 effort=0.5 velocity=100 -> lower=-0.196349540849 upper=0.196349540849 effort=1 velocity=100
