Commit message: level0 planning /w geo ompl

File: data/spider.urdf (robot description, URDF)
Before this commit: robot spider, 22 links, 21 joints
Links:
- removed link eye
- removed link eye_sphere_0
- removed link eye_sphere_0_spherical_joint_link
- removed link eye_sphere_1
- removed link eye_sphere_1_spherical_joint_link
- removed link eye_sphere_2
- removed link eye_sphere_2_spherical_joint_link
- added link brain, mass 1; collision sphere radius=0.2; visual sphere radius=0.2
- added link brain_sphere_0, mass 1; collision sphere radius=0.1; visual sphere radius=0.1
- added link brain_sphere_0_spherical_joint_link, mass 1; collision sphere radius=0.001; visual sphere radius=0.001
- added link brain_sphere_1, mass 1; collision sphere radius=0.1; visual sphere radius=0.1
- added link brain_sphere_1_spherical_joint_link, mass 1; collision sphere radius=0.001; visual sphere radius=0.001
- added link brain_sphere_2, mass 1; collision sphere radius=0.1; visual sphere radius=0.1
- added link brain_sphere_2_spherical_joint_link, mass 1; collision sphere radius=0.001; visual sphere radius=0.001
- added link container_brain, mass 1; collision sphere radius=0.12; visual sphere radius=0.12
- added link eye_brain, mass 1; collision cylinder length=0.3 radius=0.06; visual cylinder length=0.3 radius=0.06
- link leg_0_link0: geometry collision cylinder length=0.19 radius=0.04; visual cylinder length=0.19 radius=0.04
- link leg_0_link1: geometry collision cylinder length=0.54 radius=0.04; visual cylinder length=0.54 radius=0.04
- link leg_1_link0: geometry collision cylinder length=0.19 radius=0.04; visual cylinder length=0.19 radius=0.04
- link leg_1_link1: geometry collision cylinder length=0.54 radius=0.04; visual cylinder length=0.54 radius=0.04
- link leg_2_link0: geometry collision cylinder length=0.19 radius=0.04; visual cylinder length=0.19 radius=0.04
- link leg_2_link1: geometry collision cylinder length=0.54 radius=0.04; visual cylinder length=0.54 radius=0.04
Joints:
- removed joint eye_sphere_0_fixed
- removed joint eye_sphere_1_fixed
- removed joint eye_sphere_2_fixed
- added joint brain_sphere_0_fixed: type fixed, parent brain, child brain_sphere_0, origin xyz=0 0 0 rpy=0 0 0
- added joint brain_sphere_1_fixed: type fixed, parent brain, child brain_sphere_1, origin xyz=0 0 0 rpy=0 0 0
- added joint brain_sphere_2_fixed: type fixed, parent brain, child brain_sphere_2, origin xyz=0 0 0 rpy=0 0 0
- added joint joint_brain_eye_brain: type fixed, parent eye_brain, child brain, origin xyz=0 0 0 rpy=0 0 0
- added joint joint_eye_brain_container_brain: type fixed, parent container_brain, child eye_brain, origin xyz=0 0 0 rpy=0 0 0
- joint leg_0_link0_spherical_Y: parent eye_sphere_0_spherical_joint_link -> brain_sphere_0_spherical_joint_link
- joint leg_0_link0_spherical_Z: child eye_sphere_0_spherical_joint_link -> brain_sphere_0_spherical_joint_link; origin xyz=0.4 0.0 0 rpy=0 0 0 -> xyz=0.3 0.0 0 rpy=0 0 0; parent eye_sphere_0 -> brain_sphere_0
- joint leg_0_link1_spherical_Z: origin xyz=0.5 0.0 0 rpy=0 0 0 -> xyz=0.4 0.0 0 rpy=0 0 0
- joint leg_1_link0_spherical_Y: parent eye_sphere_1_spherical_joint_link -> brain_sphere_1_spherical_joint_link
- joint leg_1_link0_spherical_Z: child eye_sphere_1_spherical_joint_link -> brain_sphere_1_spherical_joint_link; origin xyz=-0.2 0.346410161514 0 rpy=0 0 0 -> xyz=-0.15 0.259807621135 0 rpy=0 0 0; parent eye_sphere_1 -> brain_sphere_1
- joint leg_1_link1_spherical_Z: origin xyz=-0.25 0.433012701892 0 rpy=0 0 0 -> xyz=-0.2 0.346410161514 0 rpy=0 0 0
- joint leg_2_link0_spherical_Y: parent eye_sphere_2_spherical_joint_link -> brain_sphere_2_spherical_joint_link
- joint leg_2_link0_spherical_Z: child eye_sphere_2_spherical_joint_link -> brain_sphere_2_spherical_joint_link; origin xyz=-0.2 -0.346410161514 0 rpy=0 0 0 -> xyz=-0.15 -0.259807621135 0 rpy=0 0 0; parent eye_sphere_2 -> brain_sphere_2
- joint leg_2_link1_spherical_Z: origin xyz=-0.25 -0.433012701892 0 rpy=0 0 0 -> xyz=-0.2 -0.346410161514 0 rpy=0 0 0
