Commit message: shortest path on simplicial complex

File: data/sphere_inner.urdf (robot description, URDF)
Before this commit: robot sphere_inner, 1 links, 0 joints
Links:
- link sphere_inner: geometry collision sphere radius=0.2; visual sphere radius=0.2

File: data/sphere_outer.urdf (robot description, URDF)
Before this commit: robot sphere_outer, 1 links, 0 joints
Links:
- link sphere_outer: geometry collision sphere radius=1; visual sphere radius=1
