Commit message: rm benchmark databases; added test cases

File: data/snake_irreducible.urdf (robot description, URDF)
Before this commit: robot snake_irreducible, 4 links, 3 joints
Links:
- added link body0_spherical_joint_link, mass 1; collision sphere radius=0.001; visual sphere radius=0.001
- added link body1, mass 1; collision sphere radius=0.019; visual sphere radius=0.019
- added link body1_cylinder, mass 1; collision cylinder length=0.2 radius=0.075; visual cylinder length=0.2 radius=0.075
- added link body1_spherical_joint_link, mass 1; collision sphere radius=0.001; visual sphere radius=0.001
- added link body2, mass 1; collision sphere radius=0.019; visual sphere radius=0.019
- added link body2_cylinder, mass 1; collision cylinder length=0.2 radius=0.0625; visual cylinder length=0.2 radius=0.0625
- added link body2_spherical_joint_link, mass 1; collision sphere radius=0.001; visual sphere radius=0.001
- added link body3, mass 1; collision sphere radius=0.019; visual sphere radius=0.019
- added link body3_cylinder, mass 1; collision cylinder length=0.2 radius=0.0520833333333; visual cylinder length=0.2 radius=0.0520833333333
- link body0: geometry collision sphere radius=0.019; visual sphere radius=0.019
Joints:
- added joint body0_body1_joint_revolute_Y: type revolute, parent body0_spherical_joint_link, child body1_cylinder, origin xyz=0 0 0 rpy=0 0 0, axis 0 1 0, limit lower=-0.785398163397 upper=0.785398163397 effort=0.01 velocity=100
- added joint body0_body1_joint_revolute_Z: type revolute, parent body0, child body0_spherical_joint_link, origin xyz=-0.045 0 0 rpy=0 0 0, axis 0 0 1, limit lower=-0.785398163397 upper=0.785398163397 effort=0.01 velocity=100
- added joint body1_body2_joint_revolute_Y: type revolute, parent body1_spherical_joint_link, child body2_cylinder, origin xyz=0 0 0 rpy=0 0 0, axis 0 1 0, limit lower=-0.785398163397 upper=0.785398163397 effort=0.01 velocity=100
- added joint body1_body2_joint_revolute_Z: type revolute, parent body1, child body1_spherical_joint_link, origin xyz=-0.24 0 0 rpy=0 0 0, axis 0 0 1, limit lower=-0.785398163397 upper=0.785398163397 effort=0.01 velocity=100
- added joint body1_fixed: type fixed, parent body1_cylinder, child body1, origin xyz=0 0 0 rpy=0 0 0
- added joint body2_body3_joint_revolute_Y: type revolute, parent body2_spherical_joint_link, child body3_cylinder, origin xyz=0 0 0 rpy=0 0 0, axis 0 1 0, limit lower=-0.785398163397 upper=0.785398163397 effort=0.01 velocity=100
- added joint body2_body3_joint_revolute_Z: type revolute, parent body2, child body2_spherical_joint_link, origin xyz=-0.24 0 0 rpy=0 0 0, axis 0 0 1, limit lower=-0.785398163397 upper=0.785398163397 effort=0.01 velocity=100
- added joint body2_fixed: type fixed, parent body2_cylinder, child body2, origin xyz=0 0 0 rpy=0 0 0
- added joint body3_fixed: type fixed, parent body3_cylinder, child body3, origin xyz=0 0 0 rpy=0 0 0
