Commit message: update nunchaku

File: data/nunchaku/nunchaku.urdf (robot description, URDF)
Before this commit: robot nunchaku, 5 links, 4 joints
Joints:
- joint joint_revolute_Z: limit lower=-3.0 upper=3.0 effort=1 velocity=100 -> lower=-2.99 upper=2.99 effort=1 velocity=100

Commit message: visualiztion of holes in the fabric of the cspace

File: data/nunchaku/nunchaku.urdf (robot description, URDF)
Before this commit: robot nunchaku, 5 links, 4 joints
Links:
- link connector: geometry collision cylinder length=0.3 radius=0.003; visual cylinder length=0.3 radius=0.003
- link connector2: geometry collision cylinder length=0.3 radius=0.003; visual cylinder length=0.3 radius=0.003
- link hinge: geometry collision cylinder length=0.06 radius=0.05; visual cylinder length=0.06 radius=0.05
- link link1: geometry collision cylinder length=0.25 radius=0.03; visual cylinder length=0.25 radius=0.03
- link link2: geometry collision cylinder length=0.25 radius=0.03; visual cylinder length=0.25 radius=0.03
Joints:
- joint joint_revolute_Z: origin xyz=0.23 0 0 rpy=0 0 0 -> xyz=0.2 0 0 rpy=0 0 0
