Commit message: different m-robots

File: data/magneto/magneto.urdf (robot description, URDF)
Before this commit: robot magneto, 7 links, 6 joints
Links:
- link foot: geometry collision cylinder length=0.08 radius=0.05; visual cylinder length=0.08 radius=0.05
- link foot2: geometry collision cylinder length=0.08 radius=0.05; visual cylinder length=0.08 radius=0.05
- link joint1: geometry collision cylinder length=0.08 radius=0.04; visual cylinder length=0.08 radius=0.04
- link joint2: geometry collision cylinder length=0.08 radius=0.04; visual cylinder length=0.08 radius=0.04
Joints:
- joint joint_leg2_joint1_Z: limit lower=-1.57 upper=1.57 effort=1 velocity=100 -> lower=-1.57 upper=1.57 effort=0.01 velocity=100; origin xyz=0.53 0 0 rpy=0 0 0 -> xyz=0.49 0 0 rpy=0 0 0
- joint joint_leg3_joint2_Z: limit lower=-1.57 upper=1.57 effort=1 velocity=100 -> lower=-1.57 upper=1.57 effort=0.01 velocity=100; origin xyz=0.66 0 0 rpy=0 0 0 -> xyz=0.58 0 0 rpy=0 0 0
