Commit message: fixed forcefields

File: data/magneto/magneto0.urdf (robot description, URDF)
Before this commit: robot magneto0, 3 links, 2 joints
Links:
- link leg: geometry collision cylinder length=0.05 radius=0.04; visual cylinder length=0.05 radius=0.04
Joints:
- joint joint_leg_foot2_Z: origin xyz=0.11 0 0 rpy=0 0 0 -> xyz=0.15 0 0 rpy=0 0 0

Commit message: updated nesting

File: data/magneto/magneto0.urdf (robot description, URDF)
Before this commit: robot magneto0, 3 links, 2 joints
Links:
- link leg: geometry collision cylinder length=0.07 radius=0.04; visual cylinder length=0.07 radius=0.04
Joints:
- joint joint_leg_foot2_Z: origin xyz=0.15 0 0 rpy=0 0 0 -> xyz=0.17 0 0 rpy=0 0 0
