Commit message: algorithm properties can be changed individually in xml

File: data/Lshape/Lshape.urdf (robot description, URDF)
Before this commit: robot Lshape, 2 links, 1 joints
Links:
- link link1: geometry collision box size=2.0 0.4 0.4; visual box size=2.0 0.4 0.4

File: data/Lshape/Lshape_capsule_inner.urdf (robot description, URDF)
Before this commit: robot Lshape_capsule_inner, 1 links, 0 joints
Links:
- link body: geometry collision cylinder length=2.0 radius=0.2; visual cylinder length=2.0 radius=0.2

File: data/Lshape/Lshape_capsule_outer.urdf (robot description, URDF)
Before this commit: robot Lshape_capsule_outer, 1 links, 0 joints
Links:
- link body: geometry collision cylinder length=2.0 radius=1.7; visual cylinder length=2.0 radius=1.7

File: data/Lshape/Lshape_sphere_outer.urdf (robot description, URDF)
Before this commit: robot Lshape_sphere_outer, 1 links, 0 joints
Links:
- link body: geometry collision sphere radius=1.80277563773; visual sphere radius=1.80277563773

Commit message: clean up of hierarchy planner

File: data/Lshape/Lshape.urdf (robot description, URDF)
Before this commit: robot Lshape, 2 links, 1 joints
Links:
- link link1: geometry collision box size=1.7 1.5 0.2; visual box size=1.7 1.5 0.2
- link link2: geometry collision box size=0.2 1.5 1.2; visual box size=0.2 1.5 1.2

File: data/Lshape/Lshape_capsule_inner.urdf (robot description, URDF)
Before this commit: robot Lshape_capsule_inner, 1 links, 0 joints
Links:
- link body: geometry collision cylinder length=1.7 radius=0.1; visual cylinder length=1.7 radius=0.1

File: data/Lshape/Lshape_capsule_outer.urdf (robot description, URDF)
Before this commit: robot Lshape_capsule_outer, 1 links, 0 joints
Links:
- link body: geometry collision cylinder length=1.7 radius=1.3; visual cylinder length=1.7 radius=1.3

File: data/Lshape/Lshape_sphere_inner.urdf (robot description, URDF)
Before this commit: robot Lshape_sphere_inner, 1 links, 0 joints
Links:
- link body: geometry collision sphere radius=0.1; visual sphere radius=0.1

File: data/Lshape/Lshape_sphere_outer.urdf (robot description, URDF)
Before this commit: robot Lshape_sphere_outer, 1 links, 0 joints
Links:
- link body: geometry collision sphere radius=1.47054411699; visual sphere radius=1.47054411699
