Commit message: planning telescope working

File: data/robots/hubble.urdf (robot description, URDF)
Before this commit: robot hubble, 6 links, 5 joints
Links:
- added link lid1, mass 1; collision cylinder length=0.05 radius=0.5; visual cylinder length=0.05 radius=0.5
- added link lid_hinge1, mass 1; collision cylinder length=0.25 radius=0.05; visual cylinder length=0.25 radius=0.05
Joints:
- added joint joint_b1_lid_hinge1: type fixed, parent body1, child lid_hinge1, origin xyz=0 0 0 rpy=0 0 0
- added joint joint_lid_hinge1_lid1_Z: type revolute, parent lid_hinge1, child lid1, origin xyz=1.5 0 0.5 rpy=0 0 0, axis 0 1 0, limit lower=-2.0 upper=0 effort=0.01 velocity=100
