Commit message: added snake; fixed vector bounds during QS computation

File: data/robots/snake.urdf (robot description, URDF)
Before this commit: robot robots/snake, 12 links, 11 joints
Links:
- removed link body2
- removed link body2_spherical_joint_link
- removed link body3_cylinder
- link body0: geometry collision sphere radius=0.0475; visual sphere radius=0.0475
- link body0_cylinder: geometry collision cylinder length=0.025 radius=0.06; visual cylinder length=0.025 radius=0.06
- link body1: geometry collision sphere radius=0.0475; visual sphere radius=0.0475
- link body1_cylinder: geometry collision cylinder length=0.2 radius=0.06; visual cylinder length=0.2 radius=0.06
- link body2_cylinder: geometry collision cylinder length=0.2 radius=0.06; visual cylinder length=0.2 radius=0.06
Joints:
- removed joint body2_body3_joint_revolute_Y
- removed joint body2_body3_joint_revolute_Z
- removed joint body2_fixed
- joint body0_body1_joint_revolute_Z: origin xyz=-0.045 0 0 rpy=0 0 0 -> xyz=-0.075 0 0 rpy=0 0 0
- joint body1_body2_joint_revolute_Z: origin xyz=-0.24 0 0 rpy=0 0 0 -> xyz=-0.3 0 0 rpy=0 0 0

File: data/robots/snake_sphere_outer.urdf (robot description, URDF)
Before this commit: robot robots/snake_sphere_outer, 1 links, 0 joints
Links:
- link body: geometry collision sphere radius=0.6; visual sphere radius=0.6

Commit message: adjusted RRTUni; 4 QS snake;

File: data/robots/snake.urdf (robot description, URDF)
Before this commit: robot robots/snake, 9 links, 8 joints
Links:
- link body0: geometry collision sphere radius=0.07125; visual sphere radius=0.07125
- link body0_cylinder: geometry collision cylinder length=0.025 radius=0.09; visual cylinder length=0.025 radius=0.09
- link body1: geometry collision sphere radius=0.07125; visual sphere radius=0.07125
- link body1_cylinder: geometry collision cylinder length=0.2 radius=0.09; visual cylinder length=0.2 radius=0.09
- link body2_cylinder: geometry collision cylinder length=0.2 radius=0.09; visual cylinder length=0.2 radius=0.09
- link eye: geometry collision sphere radius=0.15; visual sphere radius=0.15
- link head: geometry collision cylinder length=0.15 radius=0.15; visual cylinder length=0.15 radius=0.15
Joints:
- joint body0_body1_joint_revolute_Z: origin xyz=-0.075 0 0 rpy=0 0 0 -> xyz=-0.1 0 0 rpy=0 0 0
- joint body1_body2_joint_revolute_Z: origin xyz=-0.3 0 0 rpy=0 0 0 -> xyz=-0.35 0 0 rpy=0 0 0
- joint head_body0_joint: origin xyz=-0.11 0 0 rpy=0 0 0 -> xyz=-0.16 0 0 rpy=0 0 0

File: data/robots/snake_sphere_inner.urdf (robot description, URDF)
Before this commit: robot robots/snake_sphere_inner, 1 links, 0 joints
Links:
- link body: geometry collision sphere radius=0.15; visual sphere radius=0.15

Commit message: fixed several bugs related to distance/connect when using the graph metric;

File: data/robots/snake.urdf (robot description, URDF)
Before this commit: robot robots/snake, 9 links, 8 joints
Links:
- link body0: geometry collision sphere radius=0.057; visual sphere radius=0.057
- link body0_cylinder: geometry collision cylinder length=0.0375 radius=0.12; visual cylinder length=0.0375 radius=0.12
- link body1: geometry collision sphere radius=0.057; visual sphere radius=0.057
- link body1_cylinder: geometry collision cylinder length=0.3 radius=0.12; visual cylinder length=0.3 radius=0.12
- link body2_cylinder: geometry collision cylinder length=0.3 radius=0.12; visual cylinder length=0.3 radius=0.12
- link eye: geometry collision sphere radius=0.12; visual sphere radius=0.12
- link head: geometry collision cylinder length=0.12 radius=0.12; visual cylinder length=0.12 radius=0.12
Joints:
- joint body0_body1_joint_revolute_Z: origin xyz=-0.1 0 0 rpy=0 0 0 -> xyz=-0.0975 0 0 rpy=0 0 0
- joint body1_body2_joint_revolute_Z: origin xyz=-0.35 0 0 rpy=0 0 0 -> xyz=-0.42 0 0 rpy=0 0 0
- joint head_body0_joint: origin xyz=-0.16 0 0 rpy=0 0 0 -> xyz=-0.13 0 0 rpy=0 0 0

File: data/robots/snake_sphere_inner.urdf (robot description, URDF)
Before this commit: robot robots/snake_sphere_inner, 1 links, 0 joints
Links:
- link body: geometry collision sphere radius=0.12; visual sphere radius=0.12

File: data/robots/snake_sphere_outer.urdf (robot description, URDF)
Before this commit: robot robots/snake_sphere_outer, 1 links, 0 joints
Links:
- link body: geometry collision sphere radius=0.9; visual sphere radius=0.9
