Commit message: component visualization

File: data/robots/DoubleLshape_sphere_inner.urdf (robot description, URDF)
Before this commit: robot DoubleLshape_sphere_inner, 1 links, 0 joints
Links:
- link body: geometry collision sphere radius=0.4; visual sphere radius=0.4

Commit message: alpha 0.1

File: data/robots/DoubleLshape_sphere_inner.urdf (robot description, URDF)
Before this commit: robot DoubleLshape_sphere_inner, 1 links, 0 joints
Links:
- link body: geometry collision sphere radius=0.1; visual sphere radius=0.1

File: data/robots/Xshape_sphere_inner.urdf (robot description, URDF)
Before this commit: robot Xshape_sphere_inner, 1 links, 0 joints
Links:
- link body: geometry collision sphere radius=0.15; visual sphere radius=0.15

File: data/robots/snake_head_inner.urdf (robot description, URDF)
Before this commit: robot robots/snake_head_inner, 2 links, 1 joints
Links:
- link eye: geometry collision sphere radius=0.2; visual sphere radius=0.2
- link head: geometry collision cylinder length=0.12 radius=0.2; visual cylinder length=0.12 radius=0.2

File: data/robots/snake_sphere_inner.urdf (robot description, URDF)
Before this commit: robot robots/snake_sphere_inner, 1 links, 0 joints
Links:
- link body: geometry collision sphere radius=0.21; visual sphere radius=0.21
