Commit message: rewrote prm to use bundled boost properties

File: data/robots/Xshape.urdf (robot description, URDF)
Before this commit: robot Xshape, 5 links, 4 joints
Links:
- link link0: geometry collision box size=0.3 1.4 0.3; visual box size=0.3 1.4 0.3
- link link1: geometry collision box size=1.4 1.4 0.3; visual box size=1.4 1.4 0.3
- link link2: geometry collision box size=0.3 1.4 1.4; visual box size=0.3 1.4 1.4
- link link3: geometry collision box size=0.3 1.4 1.4; visual box size=0.3 1.4 1.4
- link link4: geometry collision box size=1.4 1.4 0.3; visual box size=1.4 1.4 0.3

File: data/robots/Xshape_capsule_inner.urdf (robot description, URDF)
Before this commit: robot Xshape_capsule_inner, 1 links, 0 joints
Links:
- link body: geometry collision cylinder length=1.4 radius=0.15; visual cylinder length=1.4 radius=0.15

File: data/robots/Xshape_capsule_outer.urdf (robot description, URDF)
Before this commit: robot Xshape_capsule_outer, 1 links, 0 joints
Links:
- link body: geometry collision cylinder length=1.4 radius=1.55; visual cylinder length=1.4 radius=1.55

File: data/robots/Xshape_sphere_inner.urdf (robot description, URDF)
Before this commit: robot Xshape_sphere_inner, 1 links, 0 joints
Links:
- link body: geometry collision sphere radius=0.15; visual sphere radius=0.15
