Commit message: planar nested robot sphere->cylinder

File: data/robots/PlanarLshape_sphere_inner.urdf (robot description, URDF)
Before this commit: robot PlanarLshape_sphere_inner, 1 links, 0 joints
Links:
- link body: geometry collision cylinder length=0.1 radius=0.35; visual cylinder length=0.1 radius=0.35

File: data/robots/PlanarLshape_sphere_outer.urdf (robot description, URDF)
Before this commit: robot PlanarLshape_sphere_outer, 1 links, 0 joints
Links:
- link body: geometry collision cylinder length=0.1 radius=1.3416407865; visual cylinder length=0.1 radius=1.3416407865
