Commit message: added gudhi support

File: data/robots/PlanarLshape.urdf (robot description, URDF)
Before this commit: robot PlanarLshape, 2 links, 1 joints
Links:
- link link1: geometry collision box size=1.8 0.7 0.1; visual box size=1.8 0.7 0.1
- link link2: geometry collision box size=0.7 1.8 0.1; visual box size=0.7 1.8 0.1

File: data/robots/PlanarLshape_sphere_inner.urdf (robot description, URDF)
Before this commit: robot PlanarLshape_sphere_inner, 1 links, 0 joints
Links:
- link body: geometry collision sphere radius=0.35; visual sphere radius=0.35

File: data/robots/PlanarLshape_sphere_outer.urdf (robot description, URDF)
Before this commit: robot PlanarLshape_sphere_outer, 1 links, 0 joints
Links:
- link body: geometry collision sphere radius=2.01246117975; visual sphere radius=2.01246117975

Commit message: plotted sufficient samples on 2d grid

File: data/robots/PlanarLshape.urdf (robot description, URDF)
Before this commit: robot PlanarLshape, 2 links, 1 joints
Links:
- added link link3, mass 1; collision box size=1.2 0.7 0.1; visual box size=1.2 0.7 0.1
- link link1: geometry collision box size=0.7 0.7 0.1; visual box size=0.7 0.7 0.1
- link link2: geometry collision box size=0.7 1.2 0.1; visual box size=0.7 1.2 0.1
Joints:
- added joint joint_l1_l3: type fixed, parent link1, child link3, origin xyz=0 0 0 rpy=0 0 0

File: data/robots/PlanarLshape_sphere_outer.urdf (robot description, URDF)
Before this commit: robot PlanarLshape_sphere_outer, 1 links, 0 joints
Links:
- link body: geometry collision sphere radius=1.3416407865; visual sphere radius=1.3416407865

Commit message: fixed planarLshape; added cylinder primitive; visualization of QS and CS

File: data/robots/PlanarLshape.urdf (robot description, URDF)
Before this commit: robot PlanarLshape, 3 links, 2 joints
Links:
- link link2: geometry collision box size=0.7 1.1999999999 0.1; visual box size=0.7 1.1999999999 0.1

File: data/robots/PlanarLshape_cylinder_inner.urdf (robot description, URDF)
Before this commit: robot PlanarLshape_sphere_outer, 1 links, 0 joints
Links:
- link body: geometry collision cylinder length=0.2 radius=0.35; visual cylinder length=0.2 radius=0.35

File: data/robots/PlanarLshape_sphere_inner.urdf (robot description, URDF)
Before this commit: robot PlanarLshape_sphere_inner, 1 links, 0 joints
Links:
- link body: geometry collision cylinder length=0.05 radius=0.35; visual cylinder length=0.05 radius=0.35
