Commit message: refactored visualization qspace scripts;

File: data/robots/2dof_manip.urdf (robot description, URDF)
Before this commit: robot 2dof_manip, 4 links, 3 joints
Joints:
- joint joint_jlink1_link1_Z: limit lower=-1.57 upper=1.57 effort=0.01 velocity=100 -> lower=-3.14 upper=3.14 effort=0.01 velocity=100
- joint joint_jlink2_link2_Z: limit lower=-1.57 upper=1.57 effort=0.01 velocity=100 -> lower=-3.14 upper=3.14 effort=0.01 velocity=100

File: data/robots/2dof_manip_1dof_inner.urdf (robot description, URDF)
Before this commit: robot 2dof_manip_1dof_inner, 3 links, 2 joints
Joints:
- joint joint_jlink1_link1_Z: limit lower=-1.57 upper=1.57 effort=0.01 velocity=100 -> lower=-3.14 upper=3.14 effort=0.01 velocity=100

File: data/robots/2dof_manip_1dof_outer.urdf (robot description, URDF)
Before this commit: robot 2dof_manip_1dof_inner, 2 links, 1 joints
Joints:
- joint joint_link1_link2_Z: limit lower=-1.57 upper=1.57 effort=0.01 velocity=100 -> lower=-3.14 upper=3.14 effort=0.01 velocity=100
