Commit message: Implement rejection of samples if inside cover; Update estimation of best next state

File: data/robots/cylinder_anti_voronoi_bias.urdf (robot description, URDF)
Before this commit: robot cylinder, 1 links, 0 joints
Links:
- link body: geometry collision cylinder length=0.1 radius=0.38; visual cylinder length=0.1 radius=0.38
