Commit message: Implement NBH expansion on single level

File: data/robots/PlanarRectangle.urdf (robot description, URDF)
Before this commit: robot PlanarRectangle, 1 links, 0 joints
Links:
- removed link link1
- added link link, mass 1; collision box size=1.2 0.7 0.1; visual box size=1.2 0.7 0.1

Commit message: Add cspace constant to compute lower bound on neighborhood

File: data/robots/PlanarRectangle.urdf (robot description, URDF)
Before this commit: robot PlanarRectangle, 1 links, 0 joints
Links:
- link link: geometry collision box size=2.0 0.7 0.1; visual box size=2.0 0.7 0.1

File: data/robots/PlanarRectangle_cylinder_outer.urdf (robot description, URDF)
Before this commit: robot PlanarRectangle_cylinder_outer, 1 links, 0 joints
Links:
- link body: geometry collision cylinder length=0.05 radius=1.05948100502; visual cylinder length=0.05 radius=1.05948100502

File: data/robots/snake_head_inner.urdf (robot description, URDF)
Before this commit: robot robots/snake_head_inner, 2 links, 1 joints
Links:
- link eye: geometry collision sphere radius=0.12; visual sphere radius=0.12
- link head: geometry collision cylinder length=0.12 radius=0.12; visual cylinder length=0.12 radius=0.12

File: data/robots/snake_sphere_inner.urdf (robot description, URDF)
Before this commit: robot robots/snake_sphere_inner, 1 links, 0 joints
Links:
- link body: geometry collision sphere radius=0.12; visual sphere radius=0.12
