Commit message: Added airplane scenario

File: data/robots/airplane.urdf (robot description, URDF)
Before this commit: robot airplane, 1 links, 0 joints
Links:
- link planeLink: mass 10 -> None; geometry collision mesh filename=airplane_small.stl scale=1 1 1; visual mesh filename=airplane_small.stl scale=1 1 1

Commit message: Fix dubins plane scenario.

File: data/robots/airplane.urdf (robot description, URDF)
Before this commit: robot airplane, 1 links, 0 joints
Links:
- link planeLink: geometry collision mesh filename=airplane_small.stl; visual mesh filename=airplane_small.stl

File: data/robots/airplane_inner_sphere.urdf (robot description, URDF)
Before this commit: robot sphere, 1 links, 0 joints
Links:
- link body: geometry collision sphere radius=0.15; visual sphere radius=0.15

Commit message: Fix integrator to consider mass of rigid body

File: data/robots/airplane.urdf (robot description, URDF)
Before this commit: robot airplane, 1 links, 0 joints
Links:
- link planeLink: mass None -> 10
