Commit message: Add new environments

File: data/robots/sentinel.urdf (robot description, URDF)
Before this commit: robot sentinel, 138 links, 137 joints
Links:
- link head: geometry collision cylinder length=0.3 radius=0.1; visual cylinder length=0.3 radius=0.1
Joints:
- joint joint_fixed_head_branch_00_cylinder: origin xyz=-0.1 0.07 0.0 rpy=0 0 0 -> xyz=-0.1 0.06999999999999999 0.0 rpy=0 0 0
- joint joint_fixed_head_branch_10_cylinder: origin xyz=-0.1 0.0494974746831 0.0494974746831 rpy=0 0 0 -> xyz=-0.1 0.049497474683058325 0.04949747468305832 rpy=0 0 0
- joint joint_fixed_head_branch_20_cylinder: origin xyz=-0.1 4.28626379702e-18 0.07 rpy=0 0 0 -> xyz=-0.1 4.286263797015736e-18 0.06999999999999999 rpy=0 0 0
- joint joint_fixed_head_branch_30_cylinder: origin xyz=-0.1 -0.0494974746831 0.0494974746831 rpy=0 0 0 -> xyz=-0.1 -0.04949747468305832 0.049497474683058325 rpy=0 0 0
- joint joint_fixed_head_branch_40_cylinder: origin xyz=-0.1 -0.07 8.57252759403e-18 rpy=0 0 0 -> xyz=-0.1 -0.06999999999999999 8.572527594031472e-18 rpy=0 0 0
- joint joint_fixed_head_branch_50_cylinder: origin xyz=-0.1 -0.0494974746831 -0.0494974746831 rpy=0 0 0 -> xyz=-0.1 -0.04949747468305833 -0.04949747468305832 rpy=0 0 0
- joint joint_fixed_head_branch_60_cylinder: origin xyz=-0.1 -1.2858791391e-17 -0.07 rpy=0 0 0 -> xyz=-0.1 -1.2858791391047206e-17 -0.06999999999999999 rpy=0 0 0
- joint joint_fixed_head_branch_70_cylinder: origin xyz=-0.1 0.0494974746831 -0.0494974746831 rpy=0 0 0 -> xyz=-0.1 0.04949747468305831 -0.04949747468305833 rpy=0 0 0
- joint joint_spherical_branch_00_branch_01_cylinder_Y: limit lower=-1.57079632679 upper=1.57079632679 effort=0.01 velocity=100 -> lower=-1.5707963267948966 upper=1.5707963267948966 effort=0.01 velocity=100
- joint joint_spherical_branch_00_branch_01_cylinder_Z: limit lower=-1.57079632679 upper=1.57079632679 effort=0.01 velocity=100 -> lower=-1.5707963267948966 upper=1.5707963267948966 effort=0.01 velocity=100
- joint joint_spherical_branch_01_branch_02_cylinder_Y: limit lower=-1.57079632679 upper=1.57079632679 effort=0.01 velocity=100 -> lower=-1.5707963267948966 upper=1.5707963267948966 effort=0.01 velocity=100
- joint joint_spherical_branch_01_branch_02_cylinder_Z: limit lower=-1.57079632679 upper=1.57079632679 effort=0.01 velocity=100 -> lower=-1.5707963267948966 upper=1.5707963267948966 effort=0.01 velocity=100
- joint joint_spherical_branch_02_branch_03_cylinder_Y: limit lower=-1.57079632679 upper=1.57079632679 effort=0.01 velocity=100 -> lower=-1.5707963267948966 upper=1.5707963267948966 effort=0.01 velocity=100
- joint joint_spherical_branch_02_branch_03_cylinder_Z: limit lower=-1.57079632679 upper=1.57079632679 effort=0.01 velocity=100 -> lower=-1.5707963267948966 upper=1.5707963267948966 effort=0.01 velocity=100
- joint joint_spherical_branch_03_branch_04_cylinder_Y: limit lower=-1.57079632679 upper=1.57079632679 effort=0.01 velocity=100 -> lower=-1.5707963267948966 upper=1.5707963267948966 effort=0.01 velocity=100
- joint joint_spherical_branch_03_branch_04_cylinder_Z: limit lower=-1.57079632679 upper=1.57079632679 effort=0.01 velocity=100 -> lower=-1.5707963267948966 upper=1.5707963267948966 effort=0.01 velocity=100
- joint joint_spherical_branch_04_branch_05_cylinder_Y: limit lower=-1.57079632679 upper=1.57079632679 effort=0.01 velocity=100 -> lower=-1.5707963267948966 upper=1.5707963267948966 effort=0.01 velocity=100
- joint joint_spherical_branch_04_branch_05_cylinder_Z: limit lower=-1.57079632679 upper=1.57079632679 effort=0.01 velocity=100 -> lower=-1.5707963267948966 upper=1.5707963267948966 effort=0.01 velocity=100
- joint joint_spherical_branch_10_branch_11_cylinder_Y: limit lower=-1.57079632679 upper=1.57079632679 effort=0.01 velocity=100 -> lower=-1.5707963267948966 upper=1.5707963267948966 effort=0.01 velocity=100
- joint joint_spherical_branch_10_branch_11_cylinder_Z: limit lower=-1.57079632679 upper=1.57079632679 effort=0.01 velocity=100 -> lower=-1.5707963267948966 upper=1.5707963267948966 effort=0.01 velocity=100
- joint joint_spherical_branch_11_branch_12_cylinder_Y: limit lower=-1.57079632679 upper=1.57079632679 effort=0.01 velocity=100 -> lower=-1.5707963267948966 upper=1.5707963267948966 effort=0.01 velocity=100
- joint joint_spherical_branch_11_branch_12_cylinder_Z: limit lower=-1.57079632679 upper=1.57079632679 effort=0.01 velocity=100 -> lower=-1.5707963267948966 upper=1.5707963267948966 effort=0.01 velocity=100
- joint joint_spherical_branch_12_branch_13_cylinder_Y: limit lower=-1.57079632679 upper=1.57079632679 effort=0.01 velocity=100 -> lower=-1.5707963267948966 upper=1.5707963267948966 effort=0.01 velocity=100
- joint joint_spherical_branch_12_branch_13_cylinder_Z: limit lower=-1.57079632679 upper=1.57079632679 effort=0.01 velocity=100 -> lower=-1.5707963267948966 upper=1.5707963267948966 effort=0.01 velocity=100
- joint joint_spherical_branch_13_branch_14_cylinder_Y: limit lower=-1.57079632679 upper=1.57079632679 effort=0.01 velocity=100 -> lower=-1.5707963267948966 upper=1.5707963267948966 effort=0.01 velocity=100
- joint joint_spherical_branch_13_branch_14_cylinder_Z: limit lower=-1.57079632679 upper=1.57079632679 effort=0.01 velocity=100 -> lower=-1.5707963267948966 upper=1.5707963267948966 effort=0.01 velocity=100
- joint joint_spherical_branch_14_branch_15_cylinder_Y: limit lower=-1.57079632679 upper=1.57079632679 effort=0.01 velocity=100 -> lower=-1.5707963267948966 upper=1.5707963267948966 effort=0.01 velocity=100
- joint joint_spherical_branch_14_branch_15_cylinder_Z: limit lower=-1.57079632679 upper=1.57079632679 effort=0.01 velocity=100 -> lower=-1.5707963267948966 upper=1.5707963267948966 effort=0.01 velocity=100
- joint joint_spherical_branch_20_branch_21_cylinder_Y: limit lower=-1.57079632679 upper=1.57079632679 effort=0.01 velocity=100 -> lower=-1.5707963267948966 upper=1.5707963267948966 effort=0.01 velocity=100
- joint joint_spherical_branch_20_branch_21_cylinder_Z: limit lower=-1.57079632679 upper=1.57079632679 effort=0.01 velocity=100 -> lower=-1.5707963267948966 upper=1.5707963267948966 effort=0.01 velocity=100
- joint joint_spherical_branch_21_branch_22_cylinder_Y: limit lower=-1.57079632679 upper=1.57079632679 effort=0.01 velocity=100 -> lower=-1.5707963267948966 upper=1.5707963267948966 effort=0.01 velocity=100
- joint joint_spherical_branch_21_branch_22_cylinder_Z: limit lower=-1.57079632679 upper=1.57079632679 effort=0.01 velocity=100 -> lower=-1.5707963267948966 upper=1.5707963267948966 effort=0.01 velocity=100
- joint joint_spherical_branch_22_branch_23_cylinder_Y: limit lower=-1.57079632679 upper=1.57079632679 effort=0.01 velocity=100 -> lower=-1.5707963267948966 upper=1.5707963267948966 effort=0.01 velocity=100
- joint joint_spherical_branch_22_branch_23_cylinder_Z: limit lower=-1.57079632679 upper=1.57079632679 effort=0.01 velocity=100 -> lower=-1.5707963267948966 upper=1.5707963267948966 effort=0.01 velocity=100
- joint joint_spherical_branch_23_branch_24_cylinder_Y: limit lower=-1.57079632679 upper=1.57079632679 effort=0.01 velocity=100 -> lower=-1.5707963267948966 upper=1.5707963267948966 effort=0.01 velocity=100
- joint joint_spherical_branch_23_branch_24_cylinder_Z: limit lower=-1.57079632679 upper=1.57079632679 effort=0.01 velocity=100 -> lower=-1.5707963267948966 upper=1.5707963267948966 effort=0.01 velocity=100
- joint joint_spherical_branch_24_branch_25_cylinder_Y: limit lower=-1.57079632679 upper=1.57079632679 effort=0.01 velocity=100 -> lower=-1.5707963267948966 upper=1.5707963267948966 effort=0.01 velocity=100
- joint joint_spherical_branch_24_branch_25_cylinder_Z: limit lower=-1.57079632679 upper=1.57079632679 effort=0.01 velocity=100 -> lower=-1.5707963267948966 upper=1.5707963267948966 effort=0.01 velocity=100
- joint joint_spherical_branch_30_branch_31_cylinder_Y: limit lower=-1.57079632679 upper=1.57079632679 effort=0.01 velocity=100 -> lower=-1.5707963267948966 upper=1.5707963267948966 effort=0.01 velocity=100
- joint joint_spherical_branch_30_branch_31_cylinder_Z: limit lower=-1.57079632679 upper=1.57079632679 effort=0.01 velocity=100 -> lower=-1.5707963267948966 upper=1.5707963267948966 effort=0.01 velocity=100
- joint joint_spherical_branch_31_branch_32_cylinder_Y: limit lower=-1.57079632679 upper=1.57079632679 effort=0.01 velocity=100 -> lower=-1.5707963267948966 upper=1.5707963267948966 effort=0.01 velocity=100
- joint joint_spherical_branch_31_branch_32_cylinder_Z: limit lower=-1.57079632679 upper=1.57079632679 effort=0.01 velocity=100 -> lower=-1.5707963267948966 upper=1.5707963267948966 effort=0.01 velocity=100
- joint joint_spherical_branch_32_branch_33_cylinder_Y: limit lower=-1.57079632679 upper=1.57079632679 effort=0.01 velocity=100 -> lower=-1.5707963267948966 upper=1.5707963267948966 effort=0.01 velocity=100
- joint joint_spherical_branch_32_branch_33_cylinder_Z: limit lower=-1.57079632679 upper=1.57079632679 effort=0.01 velocity=100 -> lower=-1.5707963267948966 upper=1.5707963267948966 effort=0.01 velocity=100
- joint joint_spherical_branch_33_branch_34_cylinder_Y: limit lower=-1.57079632679 upper=1.57079632679 effort=0.01 velocity=100 -> lower=-1.5707963267948966 upper=1.5707963267948966 effort=0.01 velocity=100
- joint joint_spherical_branch_33_branch_34_cylinder_Z: limit lower=-1.57079632679 upper=1.57079632679 effort=0.01 velocity=100 -> lower=-1.5707963267948966 upper=1.5707963267948966 effort=0.01 velocity=100
- joint joint_spherical_branch_34_branch_35_cylinder_Y: limit lower=-1.57079632679 upper=1.57079632679 effort=0.01 velocity=100 -> lower=-1.5707963267948966 upper=1.5707963267948966 effort=0.01 velocity=100
- joint joint_spherical_branch_34_branch_35_cylinder_Z: limit lower=-1.57079632679 upper=1.57079632679 effort=0.01 velocity=100 -> lower=-1.5707963267948966 upper=1.5707963267948966 effort=0.01 velocity=100
- joint joint_spherical_branch_40_branch_41_cylinder_Y: limit lower=-1.57079632679 upper=1.57079632679 effort=0.01 velocity=100 -> lower=-1.5707963267948966 upper=1.5707963267948966 effort=0.01 velocity=100
- joint joint_spherical_branch_40_branch_41_cylinder_Z: limit lower=-1.57079632679 upper=1.57079632679 effort=0.01 velocity=100 -> lower=-1.5707963267948966 upper=1.5707963267948966 effort=0.01 velocity=100
- joint joint_spherical_branch_41_branch_42_cylinder_Y: limit lower=-1.57079632679 upper=1.57079632679 effort=0.01 velocity=100 -> lower=-1.5707963267948966 upper=1.5707963267948966 effort=0.01 velocity=100
- joint joint_spherical_branch_41_branch_42_cylinder_Z: limit lower=-1.57079632679 upper=1.57079632679 effort=0.01 velocity=100 -> lower=-1.5707963267948966 upper=1.5707963267948966 effort=0.01 velocity=100
- joint joint_spherical_branch_42_branch_43_cylinder_Y: limit lower=-1.57079632679 upper=1.57079632679 effort=0.01 velocity=100 -> lower=-1.5707963267948966 upper=1.5707963267948966 effort=0.01 velocity=100
- joint joint_spherical_branch_42_branch_43_cylinder_Z: limit lower=-1.57079632679 upper=1.57079632679 effort=0.01 velocity=100 -> lower=-1.5707963267948966 upper=1.5707963267948966 effort=0.01 velocity=100
- joint joint_spherical_branch_43_branch_44_cylinder_Y: limit lower=-1.57079632679 upper=1.57079632679 effort=0.01 velocity=100 -> lower=-1.5707963267948966 upper=1.5707963267948966 effort=0.01 velocity=100
- joint joint_spherical_branch_43_branch_44_cylinder_Z: limit lower=-1.57079632679 upper=1.57079632679 effort=0.01 velocity=100 -> lower=-1.5707963267948966 upper=1.5707963267948966 effort=0.01 velocity=100
- joint joint_spherical_branch_44_branch_45_cylinder_Y: limit lower=-1.57079632679 upper=1.57079632679 effort=0.01 velocity=100 -> lower=-1.5707963267948966 upper=1.5707963267948966 effort=0.01 velocity=100
- joint joint_spherical_branch_44_branch_45_cylinder_Z: limit lower=-1.57079632679 upper=1.57079632679 effort=0.01 velocity=100 -> lower=-1.5707963267948966 upper=1.5707963267948966 effort=0.01 velocity=100
- joint joint_spherical_branch_50_branch_51_cylinder_Y: limit lower=-1.57079632679 upper=1.57079632679 effort=0.01 velocity=100 -> lower=-1.5707963267948966 upper=1.5707963267948966 effort=0.01 velocity=100
- joint joint_spherical_branch_50_branch_51_cylinder_Z: limit lower=-1.57079632679 upper=1.57079632679 effort=0.01 velocity=100 -> lower=-1.5707963267948966 upper=1.5707963267948966 effort=0.01 velocity=100
- joint joint_spherical_branch_51_branch_52_cylinder_Y: limit lower=-1.57079632679 upper=1.57079632679 effort=0.01 velocity=100 -> lower=-1.5707963267948966 upper=1.5707963267948966 effort=0.01 velocity=100
- joint joint_spherical_branch_51_branch_52_cylinder_Z: limit lower=-1.57079632679 upper=1.57079632679 effort=0.01 velocity=100 -> lower=-1.5707963267948966 upper=1.5707963267948966 effort=0.01 velocity=100
- joint joint_spherical_branch_52_branch_53_cylinder_Y: limit lower=-1.57079632679 upper=1.57079632679 effort=0.01 velocity=100 -> lower=-1.5707963267948966 upper=1.5707963267948966 effort=0.01 velocity=100
- joint joint_spherical_branch_52_branch_53_cylinder_Z: limit lower=-1.57079632679 upper=1.57079632679 effort=0.01 velocity=100 -> lower=-1.5707963267948966 upper=1.5707963267948966 effort=0.01 velocity=100
- joint joint_spherical_branch_53_branch_54_cylinder_Y: limit lower=-1.57079632679 upper=1.57079632679 effort=0.01 velocity=100 -> lower=-1.5707963267948966 upper=1.5707963267948966 effort=0.01 velocity=100
- joint joint_spherical_branch_53_branch_54_cylinder_Z: limit lower=-1.57079632679 upper=1.57079632679 effort=0.01 velocity=100 -> lower=-1.5707963267948966 upper=1.5707963267948966 effort=0.01 velocity=100
- joint joint_spherical_branch_54_branch_55_cylinder_Y: limit lower=-1.57079632679 upper=1.57079632679 effort=0.01 velocity=100 -> lower=-1.5707963267948966 upper=1.5707963267948966 effort=0.01 velocity=100
- joint joint_spherical_branch_54_branch_55_cylinder_Z: limit lower=-1.57079632679 upper=1.57079632679 effort=0.01 velocity=100 -> lower=-1.5707963267948966 upper=1.5707963267948966 effort=0.01 velocity=100
- joint joint_spherical_branch_60_branch_61_cylinder_Y: limit lower=-1.57079632679 upper=1.57079632679 effort=0.01 velocity=100 -> lower=-1.5707963267948966 upper=1.5707963267948966 effort=0.01 velocity=100
- joint joint_spherical_branch_60_branch_61_cylinder_Z: limit lower=-1.57079632679 upper=1.57079632679 effort=0.01 velocity=100 -> lower=-1.5707963267948966 upper=1.5707963267948966 effort=0.01 velocity=100
- joint joint_spherical_branch_61_branch_62_cylinder_Y: limit lower=-1.57079632679 upper=1.57079632679 effort=0.01 velocity=100 -> lower=-1.5707963267948966 upper=1.5707963267948966 effort=0.01 velocity=100
- joint joint_spherical_branch_61_branch_62_cylinder_Z: limit lower=-1.57079632679 upper=1.57079632679 effort=0.01 velocity=100 -> lower=-1.5707963267948966 upper=1.5707963267948966 effort=0.01 velocity=100
- joint joint_spherical_branch_62_branch_63_cylinder_Y: limit lower=-1.57079632679 upper=1.57079632679 effort=0.01 velocity=100 -> lower=-1.5707963267948966 upper=1.5707963267948966 effort=0.01 velocity=100
- joint joint_spherical_branch_62_branch_63_cylinder_Z: limit lower=-1.57079632679 upper=1.57079632679 effort=0.01 velocity=100 -> lower=-1.5707963267948966 upper=1.5707963267948966 effort=0.01 velocity=100
- joint joint_spherical_branch_63_branch_64_cylinder_Y: limit lower=-1.57079632679 upper=1.57079632679 effort=0.01 velocity=100 -> lower=-1.5707963267948966 upper=1.5707963267948966 effort=0.01 velocity=100
- joint joint_spherical_branch_63_branch_64_cylinder_Z: limit lower=-1.57079632679 upper=1.57079632679 effort=0.01 velocity=100 -> lower=-1.5707963267948966 upper=1.5707963267948966 effort=0.01 velocity=100
- joint joint_spherical_branch_64_branch_65_cylinder_Y: limit lower=-1.57079632679 upper=1.57079632679 effort=0.01 velocity=100 -> lower=-1.5707963267948966 upper=1.5707963267948966 effort=0.01 velocity=100
- joint joint_spherical_branch_64_branch_65_cylinder_Z: limit lower=-1.57079632679 upper=1.57079632679 effort=0.01 velocity=100 -> lower=-1.5707963267948966 upper=1.5707963267948966 effort=0.01 velocity=100
- joint joint_spherical_branch_70_branch_71_cylinder_Y: limit lower=-1.57079632679 upper=1.57079632679 effort=0.01 velocity=100 -> lower=-1.5707963267948966 upper=1.5707963267948966 effort=0.01 velocity=100
- joint joint_spherical_branch_70_branch_71_cylinder_Z: limit lower=-1.57079632679 upper=1.57079632679 effort=0.01 velocity=100 -> lower=-1.5707963267948966 upper=1.5707963267948966 effort=0.01 velocity=100
- joint joint_spherical_branch_71_branch_72_cylinder_Y: limit lower=-1.57079632679 upper=1.57079632679 effort=0.01 velocity=100 -> lower=-1.5707963267948966 upper=1.5707963267948966 effort=0.01 velocity=100
- joint joint_spherical_branch_71_branch_72_cylinder_Z: limit lower=-1.57079632679 upper=1.57079632679 effort=0.01 velocity=100 -> lower=-1.5707963267948966 upper=1.5707963267948966 effort=0.01 velocity=100
- joint joint_spherical_branch_72_branch_73_cylinder_Y: limit lower=-1.57079632679 upper=1.57079632679 effort=0.01 velocity=100 -> lower=-1.5707963267948966 upper=1.5707963267948966 effort=0.01 velocity=100
- joint joint_spherical_branch_72_branch_73_cylinder_Z: limit lower=-1.57079632679 upper=1.57079632679 effort=0.01 velocity=100 -> lower=-1.5707963267948966 upper=1.5707963267948966 effort=0.01 velocity=100
- joint joint_spherical_branch_73_branch_74_cylinder_Y: limit lower=-1.57079632679 upper=1.57079632679 effort=0.01 velocity=100 -> lower=-1.5707963267948966 upper=1.5707963267948966 effort=0.01 velocity=100
- joint joint_spherical_branch_73_branch_74_cylinder_Z: limit lower=-1.57079632679 upper=1.57079632679 effort=0.01 velocity=100 -> lower=-1.5707963267948966 upper=1.5707963267948966 effort=0.01 velocity=100
- joint joint_spherical_branch_74_branch_75_cylinder_Y: limit lower=-1.57079632679 upper=1.57079632679 effort=0.01 velocity=100 -> lower=-1.5707963267948966 upper=1.5707963267948966 effort=0.01 velocity=100
- joint joint_spherical_branch_74_branch_75_cylinder_Z: limit lower=-1.57079632679 upper=1.57079632679 effort=0.01 velocity=100 -> lower=-1.5707963267948966 upper=1.5707963267948966 effort=0.01 velocity=100
