Commit message: Add planar manipulator with N dofs

File: data/robots/planar_manipulator/2dof_manip_1dof_inner.urdf (robot description, URDF)
Before this commit: robot 2dof_manipulator/2dof_manip_1dof_inner, 3 links, 2 joints
Links:
- removed link jlink2
- removed link link1
- added link jlink0, mass 1; collision cylinder length=0.1 radius=0.2; visual cylinder length=0.1 radius=0.2
- added link link0, mass 1; collision box size=0.4 1.5 0.1; visual box size=0.4 1.5 0.1
Joints:
- removed joint joint_fixed_link1_jlink2
- removed joint joint_revolute_jlink1_link1_Z
- added joint joint_fixed_link0_jlink1: type fixed, parent link0, child jlink1, origin xyz=0 1.9 0 rpy=0 0 0
- added joint joint_revolute_jlink0_link0_Z: type revolute, parent jlink0, child link0, origin xyz=0 0 0 rpy=0 0 0, axis 0 0 1, limit lower=-3.14 upper=3.14 effort=0.01 velocity=100

File: data/robots/planar_manipulator/3dof_manip.urdf (robot description, URDF)
Before this commit: robot 2dof_manipulator/2dof_manip, 6 links, 5 joints
Links:
- removed link endeffectorL
- removed link endeffectorR
- added link jlink0, mass 1; collision cylinder length=0.1 radius=0.2; visual cylinder length=0.1 radius=0.2
- added link jlink3, mass 1; collision cylinder length=0.1 radius=0.2; visual cylinder length=0.1 radius=0.2
- added link link0, mass 1; collision box size=0.4 1.5 0.1; visual box size=0.4 1.5 0.1
- link link2: geometry collision box size=0.4 1.5 0.1; visual box size=0.4 1.5 0.1
Joints:
- removed joint joint_fixed_link2_endeffectorL
- removed joint joint_fixed_link2_endeffectorR
- added joint joint_fixed_link0_jlink1: type fixed, parent link0, child jlink1, origin xyz=0 1.9 0 rpy=0 0 0
- added joint joint_fixed_link2_jlink3: type fixed, parent link2, child jlink3, origin xyz=0 1.9 0 rpy=0 0 0
- added joint joint_revolute_jlink0_link0_Z: type revolute, parent jlink0, child link0, origin xyz=0 0 0 rpy=0 0 0, axis 0 0 1, limit lower=-3.14 upper=3.14 effort=0.01 velocity=100
