Commit message: Add planar manipulator with N dofs

File: data/robots/sentinel.urdf (robot description, URDF)
Before this commit: robot sentinel_pipedreamin_complete, 138 links, 137 joints
Joints:
- removed joint branch_00_branch_01_joint_revolute_Y
- removed joint branch_00_branch_01_joint_revolute_Z
- removed joint branch_01_branch_02_joint_revolute_Y
- removed joint branch_01_branch_02_joint_revolute_Z
- removed joint branch_02_branch_03_joint_revolute_Y
- removed joint branch_02_branch_03_joint_revolute_Z
- removed joint branch_03_branch_04_joint_revolute_Y
- removed joint branch_03_branch_04_joint_revolute_Z
- removed joint branch_04_branch_05_joint_revolute_Y
- removed joint branch_04_branch_05_joint_revolute_Z
- removed joint branch_10_branch_11_joint_revolute_Y
- removed joint branch_10_branch_11_joint_revolute_Z
- removed joint branch_11_branch_12_joint_revolute_Y
- removed joint branch_11_branch_12_joint_revolute_Z
- removed joint branch_12_branch_13_joint_revolute_Y
- removed joint branch_12_branch_13_joint_revolute_Z
- removed joint branch_13_branch_14_joint_revolute_Y
- removed joint branch_13_branch_14_joint_revolute_Z
- removed joint branch_14_branch_15_joint_revolute_Y
- removed joint branch_14_branch_15_joint_revolute_Z
- removed joint branch_20_branch_21_joint_revolute_Y
- removed joint branch_20_branch_21_joint_revolute_Z
- removed joint branch_21_branch_22_joint_revolute_Y
- removed joint branch_21_branch_22_joint_revolute_Z
- removed joint branch_22_branch_23_joint_revolute_Y
- removed joint branch_22_branch_23_joint_revolute_Z
- removed joint branch_23_branch_24_joint_revolute_Y
- removed joint branch_23_branch_24_joint_revolute_Z
- removed joint branch_24_branch_25_joint_revolute_Y
- removed joint branch_24_branch_25_joint_revolute_Z
- removed joint branch_30_branch_31_joint_revolute_Y
- removed joint branch_30_branch_31_joint_revolute_Z
- removed joint branch_31_branch_32_joint_revolute_Y
- removed joint branch_31_branch_32_joint_revolute_Z
- removed joint branch_32_branch_33_joint_revolute_Y
- removed joint branch_32_branch_33_joint_revolute_Z
- removed joint branch_33_branch_34_joint_revolute_Y
- removed joint branch_33_branch_34_joint_revolute_Z
- removed joint branch_34_branch_35_joint_revolute_Y
- removed joint branch_34_branch_35_joint_revolute_Z
- removed joint branch_40_branch_41_joint_revolute_Y
- removed joint branch_40_branch_41_joint_revolute_Z
- removed joint branch_41_branch_42_joint_revolute_Y
- removed joint branch_41_branch_42_joint_revolute_Z
- removed joint branch_42_branch_43_joint_revolute_Y
- removed joint branch_42_branch_43_joint_revolute_Z
- removed joint branch_43_branch_44_joint_revolute_Y
- removed joint branch_43_branch_44_joint_revolute_Z
- removed joint branch_44_branch_45_joint_revolute_Y
- removed joint branch_44_branch_45_joint_revolute_Z
- removed joint branch_50_branch_51_joint_revolute_Y
- removed joint branch_50_branch_51_joint_revolute_Z
- removed joint branch_51_branch_52_joint_revolute_Y
- removed joint branch_51_branch_52_joint_revolute_Z
- removed joint branch_52_branch_53_joint_revolute_Y
- removed joint branch_52_branch_53_joint_revolute_Z
- removed joint branch_53_branch_54_joint_revolute_Y
- removed joint branch_53_branch_54_joint_revolute_Z
- removed joint branch_54_branch_55_joint_revolute_Y
- removed joint branch_54_branch_55_joint_revolute_Z
- removed joint branch_60_branch_61_joint_revolute_Y
- removed joint branch_60_branch_61_joint_revolute_Z
- removed joint branch_61_branch_62_joint_revolute_Y
- removed joint branch_61_branch_62_joint_revolute_Z
- removed joint branch_62_branch_63_joint_revolute_Y
- removed joint branch_62_branch_63_joint_revolute_Z
- removed joint branch_63_branch_64_joint_revolute_Y
- removed joint branch_63_branch_64_joint_revolute_Z
- removed joint branch_64_branch_65_joint_revolute_Y
- removed joint branch_64_branch_65_joint_revolute_Z
- removed joint branch_70_branch_71_joint_revolute_Y
- removed joint branch_70_branch_71_joint_revolute_Z
- removed joint branch_71_branch_72_joint_revolute_Y
- removed joint branch_71_branch_72_joint_revolute_Z
- removed joint branch_72_branch_73_joint_revolute_Y
- removed joint branch_72_branch_73_joint_revolute_Z
- removed joint branch_73_branch_74_joint_revolute_Y
- removed joint branch_73_branch_74_joint_revolute_Z
- removed joint branch_74_branch_75_joint_revolute_Y
- removed joint branch_74_branch_75_joint_revolute_Z
- removed joint joint_branch_00_cylinder_branch_00
- removed joint joint_branch_01_cylinder_branch_01
- removed joint joint_branch_02_cylinder_branch_02
- removed joint joint_branch_03_cylinder_branch_03
- removed joint joint_branch_04_cylinder_branch_04
- removed joint joint_branch_05_cylinder_branch_05
- removed joint joint_branch_10_cylinder_branch_10
- removed joint joint_branch_11_cylinder_branch_11
- removed joint joint_branch_12_cylinder_branch_12
- removed joint joint_branch_13_cylinder_branch_13
- removed joint joint_branch_14_cylinder_branch_14
- removed joint joint_branch_15_cylinder_branch_15
- removed joint joint_branch_20_cylinder_branch_20
- removed joint joint_branch_21_cylinder_branch_21
- removed joint joint_branch_22_cylinder_branch_22
- removed joint joint_branch_23_cylinder_branch_23
- removed joint joint_branch_24_cylinder_branch_24
- removed joint joint_branch_25_cylinder_branch_25
- removed joint joint_branch_30_cylinder_branch_30
- removed joint joint_branch_31_cylinder_branch_31
- removed joint joint_branch_32_cylinder_branch_32
- removed joint joint_branch_33_cylinder_branch_33
- removed joint joint_branch_34_cylinder_branch_34
- removed joint joint_branch_35_cylinder_branch_35
- removed joint joint_branch_40_cylinder_branch_40
- removed joint joint_branch_41_cylinder_branch_41
- removed joint joint_branch_42_cylinder_branch_42
- removed joint joint_branch_43_cylinder_branch_43
- removed joint joint_branch_44_cylinder_branch_44
- removed joint joint_branch_45_cylinder_branch_45
- removed joint joint_branch_50_cylinder_branch_50
- removed joint joint_branch_51_cylinder_branch_51
- removed joint joint_branch_52_cylinder_branch_52
- removed joint joint_branch_53_cylinder_branch_53
- removed joint joint_branch_54_cylinder_branch_54
- removed joint joint_branch_55_cylinder_branch_55
- removed joint joint_branch_60_cylinder_branch_60
- removed joint joint_branch_61_cylinder_branch_61
- removed joint joint_branch_62_cylinder_branch_62
- removed joint joint_branch_63_cylinder_branch_63
- removed joint joint_branch_64_cylinder_branch_64
- removed joint joint_branch_65_cylinder_branch_65
- removed joint joint_branch_70_cylinder_branch_70
- removed joint joint_branch_71_cylinder_branch_71
- removed joint joint_branch_72_cylinder_branch_72
- removed joint joint_branch_73_cylinder_branch_73
- removed joint joint_branch_74_cylinder_branch_74
- removed joint joint_branch_75_cylinder_branch_75
- removed joint joint_eye_head
- removed joint joint_head_branch_00_cylinder
- removed joint joint_head_branch_10_cylinder
- removed joint joint_head_branch_20_cylinder
- removed joint joint_head_branch_30_cylinder
- removed joint joint_head_branch_40_cylinder
- removed joint joint_head_branch_50_cylinder
- removed joint joint_head_branch_60_cylinder
- removed joint joint_head_branch_70_cylinder
- added joint joint_fixed_branch_00_cylinder_branch_00: type fixed, parent branch_00_cylinder, child branch_00, origin xyz=0 0 0 rpy=0 0 0
- added joint joint_fixed_branch_01_cylinder_branch_01: type fixed, parent branch_01_cylinder, child branch_01, origin xyz=0 0 0 rpy=0 0 0
- added joint joint_fixed_branch_02_cylinder_branch_02: type fixed, parent branch_02_cylinder, child branch_02, origin xyz=0 0 0 rpy=0 0 0
- added joint joint_fixed_branch_03_cylinder_branch_03: type fixed, parent branch_03_cylinder, child branch_03, origin xyz=0 0 0 rpy=0 0 0
- added joint joint_fixed_branch_04_cylinder_branch_04: type fixed, parent branch_04_cylinder, child branch_04, origin xyz=0 0 0 rpy=0 0 0
- added joint joint_fixed_branch_05_cylinder_branch_05: type fixed, parent branch_05_cylinder, child branch_05, origin xyz=0 0 0 rpy=0 0 0
- added joint joint_fixed_branch_10_cylinder_branch_10: type fixed, parent branch_10_cylinder, child branch_10, origin xyz=0 0 0 rpy=0 0 0
- added joint joint_fixed_branch_11_cylinder_branch_11: type fixed, parent branch_11_cylinder, child branch_11, origin xyz=0 0 0 rpy=0 0 0
- added joint joint_fixed_branch_12_cylinder_branch_12: type fixed, parent branch_12_cylinder, child branch_12, origin xyz=0 0 0 rpy=0 0 0
- added joint joint_fixed_branch_13_cylinder_branch_13: type fixed, parent branch_13_cylinder, child branch_13, origin xyz=0 0 0 rpy=0 0 0
- added joint joint_fixed_branch_14_cylinder_branch_14: type fixed, parent branch_14_cylinder, child branch_14, origin xyz=0 0 0 rpy=0 0 0
- added joint joint_fixed_branch_15_cylinder_branch_15: type fixed, parent branch_15_cylinder, child branch_15, origin xyz=0 0 0 rpy=0 0 0
- added joint joint_fixed_branch_20_cylinder_branch_20: type fixed, parent branch_20_cylinder, child branch_20, origin xyz=0 0 0 rpy=0 0 0
- added joint joint_fixed_branch_21_cylinder_branch_21: type fixed, parent branch_21_cylinder, child branch_21, origin xyz=0 0 0 rpy=0 0 0
- added joint joint_fixed_branch_22_cylinder_branch_22: type fixed, parent branch_22_cylinder, child branch_22, origin xyz=0 0 0 rpy=0 0 0
- added joint joint_fixed_branch_23_cylinder_branch_23: type fixed, parent branch_23_cylinder, child branch_23, origin xyz=0 0 0 rpy=0 0 0
- added joint joint_fixed_branch_24_cylinder_branch_24: type fixed, parent branch_24_cylinder, child branch_24, origin xyz=0 0 0 rpy=0 0 0
- added joint joint_fixed_branch_25_cylinder_branch_25: type fixed, parent branch_25_cylinder, child branch_25, origin xyz=0 0 0 rpy=0 0 0
- added joint joint_fixed_branch_30_cylinder_branch_30: type fixed, parent branch_30_cylinder, child branch_30, origin xyz=0 0 0 rpy=0 0 0
- added joint joint_fixed_branch_31_cylinder_branch_31: type fixed, parent branch_31_cylinder, child branch_31, origin xyz=0 0 0 rpy=0 0 0
- added joint joint_fixed_branch_32_cylinder_branch_32: type fixed, parent branch_32_cylinder, child branch_32, origin xyz=0 0 0 rpy=0 0 0
- added joint joint_fixed_branch_33_cylinder_branch_33: type fixed, parent branch_33_cylinder, child branch_33, origin xyz=0 0 0 rpy=0 0 0
- added joint joint_fixed_branch_34_cylinder_branch_34: type fixed, parent branch_34_cylinder, child branch_34, origin xyz=0 0 0 rpy=0 0 0
- added joint joint_fixed_branch_35_cylinder_branch_35: type fixed, parent branch_35_cylinder, child branch_35, origin xyz=0 0 0 rpy=0 0 0
- added joint joint_fixed_branch_40_cylinder_branch_40: type fixed, parent branch_40_cylinder, child branch_40, origin xyz=0 0 0 rpy=0 0 0
- added joint joint_fixed_branch_41_cylinder_branch_41: type fixed, parent branch_41_cylinder, child branch_41, origin xyz=0 0 0 rpy=0 0 0
- added joint joint_fixed_branch_42_cylinder_branch_42: type fixed, parent branch_42_cylinder, child branch_42, origin xyz=0 0 0 rpy=0 0 0
- added joint joint_fixed_branch_43_cylinder_branch_43: type fixed, parent branch_43_cylinder, child branch_43, origin xyz=0 0 0 rpy=0 0 0
- added joint joint_fixed_branch_44_cylinder_branch_44: type fixed, parent branch_44_cylinder, child branch_44, origin xyz=0 0 0 rpy=0 0 0
- added joint joint_fixed_branch_45_cylinder_branch_45: type fixed, parent branch_45_cylinder, child branch_45, origin xyz=0 0 0 rpy=0 0 0
- added joint joint_fixed_branch_50_cylinder_branch_50: type fixed, parent branch_50_cylinder, child branch_50, origin xyz=0 0 0 rpy=0 0 0
- added joint joint_fixed_branch_51_cylinder_branch_51: type fixed, parent branch_51_cylinder, child branch_51, origin xyz=0 0 0 rpy=0 0 0
- added joint joint_fixed_branch_52_cylinder_branch_52: type fixed, parent branch_52_cylinder, child branch_52, origin xyz=0 0 0 rpy=0 0 0
- added joint joint_fixed_branch_53_cylinder_branch_53: type fixed, parent branch_53_cylinder, child branch_53, origin xyz=0 0 0 rpy=0 0 0
- added joint joint_fixed_branch_54_cylinder_branch_54: type fixed, parent branch_54_cylinder, child branch_54, origin xyz=0 0 0 rpy=0 0 0
- added joint joint_fixed_branch_55_cylinder_branch_55: type fixed, parent branch_55_cylinder, child branch_55, origin xyz=0 0 0 rpy=0 0 0
- added joint joint_fixed_branch_60_cylinder_branch_60: type fixed, parent branch_60_cylinder, child branch_60, origin xyz=0 0 0 rpy=0 0 0
- added joint joint_fixed_branch_61_cylinder_branch_61: type fixed, parent branch_61_cylinder, child branch_61, origin xyz=0 0 0 rpy=0 0 0
- added joint joint_fixed_branch_62_cylinder_branch_62: type fixed, parent branch_62_cylinder, child branch_62, origin xyz=0 0 0 rpy=0 0 0
- added joint joint_fixed_branch_63_cylinder_branch_63: type fixed, parent branch_63_cylinder, child branch_63, origin xyz=0 0 0 rpy=0 0 0
- added joint joint_fixed_branch_64_cylinder_branch_64: type fixed, parent branch_64_cylinder, child branch_64, origin xyz=0 0 0 rpy=0 0 0
- added joint joint_fixed_branch_65_cylinder_branch_65: type fixed, parent branch_65_cylinder, child branch_65, origin xyz=0 0 0 rpy=0 0 0
- added joint joint_fixed_branch_70_cylinder_branch_70: type fixed, parent branch_70_cylinder, child branch_70, origin xyz=0 0 0 rpy=0 0 0
- added joint joint_fixed_branch_71_cylinder_branch_71: type fixed, parent branch_71_cylinder, child branch_71, origin xyz=0 0 0 rpy=0 0 0
- added joint joint_fixed_branch_72_cylinder_branch_72: type fixed, parent branch_72_cylinder, child branch_72, origin xyz=0 0 0 rpy=0 0 0
- added joint joint_fixed_branch_73_cylinder_branch_73: type fixed, parent branch_73_cylinder, child branch_73, origin xyz=0 0 0 rpy=0 0 0
- added joint joint_fixed_branch_74_cylinder_branch_74: type fixed, parent branch_74_cylinder, child branch_74, origin xyz=0 0 0 rpy=0 0 0
- added joint joint_fixed_branch_75_cylinder_branch_75: type fixed, parent branch_75_cylinder, child branch_75, origin xyz=0 0 0 rpy=0 0 0
- added joint joint_fixed_eye_head: type fixed, parent eye, child head, origin xyz=0 0 0 rpy=0 0 0
- added joint joint_fixed_head_branch_00_cylinder: type fixed, parent head, child branch_00_cylinder, origin xyz=-0.1 0.07 0.0 rpy=0 0 0
- added joint joint_fixed_head_branch_10_cylinder: type fixed, parent head, child branch_10_cylinder, origin xyz=-0.1 0.0494974746831 0.0494974746831 rpy=0 0 0
- added joint joint_fixed_head_branch_20_cylinder: type fixed, parent head, child branch_20_cylinder, origin xyz=-0.1 4.28626379702e-18 0.07 rpy=0 0 0
- added joint joint_fixed_head_branch_30_cylinder: type fixed, parent head, child branch_30_cylinder, origin xyz=-0.1 -0.0494974746831 0.0494974746831 rpy=0 0 0
- added joint joint_fixed_head_branch_40_cylinder: type fixed, parent head, child branch_40_cylinder, origin xyz=-0.1 -0.07 8.57252759403e-18 rpy=0 0 0
- added joint joint_fixed_head_branch_50_cylinder: type fixed, parent head, child branch_50_cylinder, origin xyz=-0.1 -0.0494974746831 -0.0494974746831 rpy=0 0 0
- added joint joint_fixed_head_branch_60_cylinder: type fixed, parent head, child branch_60_cylinder, origin xyz=-0.1 -1.2858791391e-17 -0.07 rpy=0 0 0
- added joint joint_fixed_head_branch_70_cylinder: type fixed, parent head, child branch_70_cylinder, origin xyz=-0.1 0.0494974746831 -0.0494974746831 rpy=0 0 0
- added joint joint_spherical_branch_00_branch_01_cylinder_Y: type revolute, parent branch_00_spherical_joint_link, child branch_01_cylinder, origin xyz=0 0 0 rpy=0 0 0, axis 0 1 0, limit lower=-1.57079632679 upper=1.57079632679 effort=0.01 velocity=100
- added joint joint_spherical_branch_00_branch_01_cylinder_Z: type revolute, parent branch_00, child branch_00_spherical_joint_link, origin xyz=-0.03875 0 0 rpy=0 0 0, axis 0 0 1, limit lower=-1.57079632679 upper=1.57079632679 effort=0.01 velocity=100
- added joint joint_spherical_branch_01_branch_02_cylinder_Y: type revolute, parent branch_01_spherical_joint_link, child branch_02_cylinder, origin xyz=0 0 0 rpy=0 0 0, axis 0 1 0, limit lower=-1.57079632679 upper=1.57079632679 effort=0.01 velocity=100
- added joint joint_spherical_branch_01_branch_02_cylinder_Z: type revolute, parent branch_01, child branch_01_spherical_joint_link, origin xyz=-0.19 0 0 rpy=0 0 0, axis 0 0 1, limit lower=-1.57079632679 upper=1.57079632679 effort=0.01 velocity=100
- added joint joint_spherical_branch_02_branch_03_cylinder_Y: type revolute, parent branch_02_spherical_joint_link, child branch_03_cylinder, origin xyz=0 0 0 rpy=0 0 0, axis 0 1 0, limit lower=-1.57079632679 upper=1.57079632679 effort=0.01 velocity=100
- added joint joint_spherical_branch_02_branch_03_cylinder_Z: type revolute, parent branch_02, child branch_02_spherical_joint_link, origin xyz=-0.19 0 0 rpy=0 0 0, axis 0 0 1, limit lower=-1.57079632679 upper=1.57079632679 effort=0.01 velocity=100
- added joint joint_spherical_branch_03_branch_04_cylinder_Y: type revolute, parent branch_03_spherical_joint_link, child branch_04_cylinder, origin xyz=0 0 0 rpy=0 0 0, axis 0 1 0, limit lower=-1.57079632679 upper=1.57079632679 effort=0.01 velocity=100
- added joint joint_spherical_branch_03_branch_04_cylinder_Z: type revolute, parent branch_03, child branch_03_spherical_joint_link, origin xyz=-0.19 0 0 rpy=0 0 0, axis 0 0 1, limit lower=-1.57079632679 upper=1.57079632679 effort=0.01 velocity=100
- added joint joint_spherical_branch_04_branch_05_cylinder_Y: type revolute, parent branch_04_spherical_joint_link, child branch_05_cylinder, origin xyz=0 0 0 rpy=0 0 0, axis 0 1 0, limit lower=-1.57079632679 upper=1.57079632679 effort=0.01 velocity=100
- added joint joint_spherical_branch_04_branch_05_cylinder_Z: type revolute, parent branch_04, child branch_04_spherical_joint_link, origin xyz=-0.19 0 0 rpy=0 0 0, axis 0 0 1, limit lower=-1.57079632679 upper=1.57079632679 effort=0.01 velocity=100
- added joint joint_spherical_branch_10_branch_11_cylinder_Y: type revolute, parent branch_10_spherical_joint_link, child branch_11_cylinder, origin xyz=0 0 0 rpy=0 0 0, axis 0 1 0, limit lower=-1.57079632679 upper=1.57079632679 effort=0.01 velocity=100
- added joint joint_spherical_branch_10_branch_11_cylinder_Z: type revolute, parent branch_10, child branch_10_spherical_joint_link, origin xyz=-0.03875 0 0 rpy=0 0 0, axis 0 0 1, limit lower=-1.57079632679 upper=1.57079632679 effort=0.01 velocity=100
- added joint joint_spherical_branch_11_branch_12_cylinder_Y: type revolute, parent branch_11_spherical_joint_link, child branch_12_cylinder, origin xyz=0 0 0 rpy=0 0 0, axis 0 1 0, limit lower=-1.57079632679 upper=1.57079632679 effort=0.01 velocity=100
- added joint joint_spherical_branch_11_branch_12_cylinder_Z: type revolute, parent branch_11, child branch_11_spherical_joint_link, origin xyz=-0.19 0 0 rpy=0 0 0, axis 0 0 1, limit lower=-1.57079632679 upper=1.57079632679 effort=0.01 velocity=100
- added joint joint_spherical_branch_12_branch_13_cylinder_Y: type revolute, parent branch_12_spherical_joint_link, child branch_13_cylinder, origin xyz=0 0 0 rpy=0 0 0, axis 0 1 0, limit lower=-1.57079632679 upper=1.57079632679 effort=0.01 velocity=100
- added joint joint_spherical_branch_12_branch_13_cylinder_Z: type revolute, parent branch_12, child branch_12_spherical_joint_link, origin xyz=-0.19 0 0 rpy=0 0 0, axis 0 0 1, limit lower=-1.57079632679 upper=1.57079632679 effort=0.01 velocity=100
- added joint joint_spherical_branch_13_branch_14_cylinder_Y: type revolute, parent branch_13_spherical_joint_link, child branch_14_cylinder, origin xyz=0 0 0 rpy=0 0 0, axis 0 1 0, limit lower=-1.57079632679 upper=1.57079632679 effort=0.01 velocity=100
- added joint joint_spherical_branch_13_branch_14_cylinder_Z: type revolute, parent branch_13, child branch_13_spherical_joint_link, origin xyz=-0.19 0 0 rpy=0 0 0, axis 0 0 1, limit lower=-1.57079632679 upper=1.57079632679 effort=0.01 velocity=100
- added joint joint_spherical_branch_14_branch_15_cylinder_Y: type revolute, parent branch_14_spherical_joint_link, child branch_15_cylinder, origin xyz=0 0 0 rpy=0 0 0, axis 0 1 0, limit lower=-1.57079632679 upper=1.57079632679 effort=0.01 velocity=100
- added joint joint_spherical_branch_14_branch_15_cylinder_Z: type revolute, parent branch_14, child branch_14_spherical_joint_link, origin xyz=-0.19 0 0 rpy=0 0 0, axis 0 0 1, limit lower=-1.57079632679 upper=1.57079632679 effort=0.01 velocity=100
- added joint joint_spherical_branch_20_branch_21_cylinder_Y: type revolute, parent branch_20_spherical_joint_link, child branch_21_cylinder, origin xyz=0 0 0 rpy=0 0 0, axis 0 1 0, limit lower=-1.57079632679 upper=1.57079632679 effort=0.01 velocity=100
- added joint joint_spherical_branch_20_branch_21_cylinder_Z: type revolute, parent branch_20, child branch_20_spherical_joint_link, origin xyz=-0.03875 0 0 rpy=0 0 0, axis 0 0 1, limit lower=-1.57079632679 upper=1.57079632679 effort=0.01 velocity=100
- added joint joint_spherical_branch_21_branch_22_cylinder_Y: type revolute, parent branch_21_spherical_joint_link, child branch_22_cylinder, origin xyz=0 0 0 rpy=0 0 0, axis 0 1 0, limit lower=-1.57079632679 upper=1.57079632679 effort=0.01 velocity=100
- added joint joint_spherical_branch_21_branch_22_cylinder_Z: type revolute, parent branch_21, child branch_21_spherical_joint_link, origin xyz=-0.19 0 0 rpy=0 0 0, axis 0 0 1, limit lower=-1.57079632679 upper=1.57079632679 effort=0.01 velocity=100
- added joint joint_spherical_branch_22_branch_23_cylinder_Y: type revolute, parent branch_22_spherical_joint_link, child branch_23_cylinder, origin xyz=0 0 0 rpy=0 0 0, axis 0 1 0, limit lower=-1.57079632679 upper=1.57079632679 effort=0.01 velocity=100
- added joint joint_spherical_branch_22_branch_23_cylinder_Z: type revolute, parent branch_22, child branch_22_spherical_joint_link, origin xyz=-0.19 0 0 rpy=0 0 0, axis 0 0 1, limit lower=-1.57079632679 upper=1.57079632679 effort=0.01 velocity=100
- added joint joint_spherical_branch_23_branch_24_cylinder_Y: type revolute, parent branch_23_spherical_joint_link, child branch_24_cylinder, origin xyz=0 0 0 rpy=0 0 0, axis 0 1 0, limit lower=-1.57079632679 upper=1.57079632679 effort=0.01 velocity=100
- added joint joint_spherical_branch_23_branch_24_cylinder_Z: type revolute, parent branch_23, child branch_23_spherical_joint_link, origin xyz=-0.19 0 0 rpy=0 0 0, axis 0 0 1, limit lower=-1.57079632679 upper=1.57079632679 effort=0.01 velocity=100
- added joint joint_spherical_branch_24_branch_25_cylinder_Y: type revolute, parent branch_24_spherical_joint_link, child branch_25_cylinder, origin xyz=0 0 0 rpy=0 0 0, axis 0 1 0, limit lower=-1.57079632679 upper=1.57079632679 effort=0.01 velocity=100
- added joint joint_spherical_branch_24_branch_25_cylinder_Z: type revolute, parent branch_24, child branch_24_spherical_joint_link, origin xyz=-0.19 0 0 rpy=0 0 0, axis 0 0 1, limit lower=-1.57079632679 upper=1.57079632679 effort=0.01 velocity=100
- added joint joint_spherical_branch_30_branch_31_cylinder_Y: type revolute, parent branch_30_spherical_joint_link, child branch_31_cylinder, origin xyz=0 0 0 rpy=0 0 0, axis 0 1 0, limit lower=-1.57079632679 upper=1.57079632679 effort=0.01 velocity=100
- added joint joint_spherical_branch_30_branch_31_cylinder_Z: type revolute, parent branch_30, child branch_30_spherical_joint_link, origin xyz=-0.03875 0 0 rpy=0 0 0, axis 0 0 1, limit lower=-1.57079632679 upper=1.57079632679 effort=0.01 velocity=100
- added joint joint_spherical_branch_31_branch_32_cylinder_Y: type revolute, parent branch_31_spherical_joint_link, child branch_32_cylinder, origin xyz=0 0 0 rpy=0 0 0, axis 0 1 0, limit lower=-1.57079632679 upper=1.57079632679 effort=0.01 velocity=100
- added joint joint_spherical_branch_31_branch_32_cylinder_Z: type revolute, parent branch_31, child branch_31_spherical_joint_link, origin xyz=-0.19 0 0 rpy=0 0 0, axis 0 0 1, limit lower=-1.57079632679 upper=1.57079632679 effort=0.01 velocity=100
- added joint joint_spherical_branch_32_branch_33_cylinder_Y: type revolute, parent branch_32_spherical_joint_link, child branch_33_cylinder, origin xyz=0 0 0 rpy=0 0 0, axis 0 1 0, limit lower=-1.57079632679 upper=1.57079632679 effort=0.01 velocity=100
- added joint joint_spherical_branch_32_branch_33_cylinder_Z: type revolute, parent branch_32, child branch_32_spherical_joint_link, origin xyz=-0.19 0 0 rpy=0 0 0, axis 0 0 1, limit lower=-1.57079632679 upper=1.57079632679 effort=0.01 velocity=100
- added joint joint_spherical_branch_33_branch_34_cylinder_Y: type revolute, parent branch_33_spherical_joint_link, child branch_34_cylinder, origin xyz=0 0 0 rpy=0 0 0, axis 0 1 0, limit lower=-1.57079632679 upper=1.57079632679 effort=0.01 velocity=100
- added joint joint_spherical_branch_33_branch_34_cylinder_Z: type revolute, parent branch_33, child branch_33_spherical_joint_link, origin xyz=-0.19 0 0 rpy=0 0 0, axis 0 0 1, limit lower=-1.57079632679 upper=1.57079632679 effort=0.01 velocity=100
- added joint joint_spherical_branch_34_branch_35_cylinder_Y: type revolute, parent branch_34_spherical_joint_link, child branch_35_cylinder, origin xyz=0 0 0 rpy=0 0 0, axis 0 1 0, limit lower=-1.57079632679 upper=1.57079632679 effort=0.01 velocity=100
- added joint joint_spherical_branch_34_branch_35_cylinder_Z: type revolute, parent branch_34, child branch_34_spherical_joint_link, origin xyz=-0.19 0 0 rpy=0 0 0, axis 0 0 1, limit lower=-1.57079632679 upper=1.57079632679 effort=0.01 velocity=100
- added joint joint_spherical_branch_40_branch_41_cylinder_Y: type revolute, parent branch_40_spherical_joint_link, child branch_41_cylinder, origin xyz=0 0 0 rpy=0 0 0, axis 0 1 0, limit lower=-1.57079632679 upper=1.57079632679 effort=0.01 velocity=100
- added joint joint_spherical_branch_40_branch_41_cylinder_Z: type revolute, parent branch_40, child branch_40_spherical_joint_link, origin xyz=-0.03875 0 0 rpy=0 0 0, axis 0 0 1, limit lower=-1.57079632679 upper=1.57079632679 effort=0.01 velocity=100
- added joint joint_spherical_branch_41_branch_42_cylinder_Y: type revolute, parent branch_41_spherical_joint_link, child branch_42_cylinder, origin xyz=0 0 0 rpy=0 0 0, axis 0 1 0, limit lower=-1.57079632679 upper=1.57079632679 effort=0.01 velocity=100
- added joint joint_spherical_branch_41_branch_42_cylinder_Z: type revolute, parent branch_41, child branch_41_spherical_joint_link, origin xyz=-0.19 0 0 rpy=0 0 0, axis 0 0 1, limit lower=-1.57079632679 upper=1.57079632679 effort=0.01 velocity=100
- added joint joint_spherical_branch_42_branch_43_cylinder_Y: type revolute, parent branch_42_spherical_joint_link, child branch_43_cylinder, origin xyz=0 0 0 rpy=0 0 0, axis 0 1 0, limit lower=-1.57079632679 upper=1.57079632679 effort=0.01 velocity=100
- added joint joint_spherical_branch_42_branch_43_cylinder_Z: type revolute, parent branch_42, child branch_42_spherical_joint_link, origin xyz=-0.19 0 0 rpy=0 0 0, axis 0 0 1, limit lower=-1.57079632679 upper=1.57079632679 effort=0.01 velocity=100
- added joint joint_spherical_branch_43_branch_44_cylinder_Y: type revolute, parent branch_43_spherical_joint_link, child branch_44_cylinder, origin xyz=0 0 0 rpy=0 0 0, axis 0 1 0, limit lower=-1.57079632679 upper=1.57079632679 effort=0.01 velocity=100
- added joint joint_spherical_branch_43_branch_44_cylinder_Z: type revolute, parent branch_43, child branch_43_spherical_joint_link, origin xyz=-0.19 0 0 rpy=0 0 0, axis 0 0 1, limit lower=-1.57079632679 upper=1.57079632679 effort=0.01 velocity=100
- added joint joint_spherical_branch_44_branch_45_cylinder_Y: type revolute, parent branch_44_spherical_joint_link, child branch_45_cylinder, origin xyz=0 0 0 rpy=0 0 0, axis 0 1 0, limit lower=-1.57079632679 upper=1.57079632679 effort=0.01 velocity=100
- added joint joint_spherical_branch_44_branch_45_cylinder_Z: type revolute, parent branch_44, child branch_44_spherical_joint_link, origin xyz=-0.19 0 0 rpy=0 0 0, axis 0 0 1, limit lower=-1.57079632679 upper=1.57079632679 effort=0.01 velocity=100
- added joint joint_spherical_branch_50_branch_51_cylinder_Y: type revolute, parent branch_50_spherical_joint_link, child branch_51_cylinder, origin xyz=0 0 0 rpy=0 0 0, axis 0 1 0, limit lower=-1.57079632679 upper=1.57079632679 effort=0.01 velocity=100
- added joint joint_spherical_branch_50_branch_51_cylinder_Z: type revolute, parent branch_50, child branch_50_spherical_joint_link, origin xyz=-0.03875 0 0 rpy=0 0 0, axis 0 0 1, limit lower=-1.57079632679 upper=1.57079632679 effort=0.01 velocity=100
- added joint joint_spherical_branch_51_branch_52_cylinder_Y: type revolute, parent branch_51_spherical_joint_link, child branch_52_cylinder, origin xyz=0 0 0 rpy=0 0 0, axis 0 1 0, limit lower=-1.57079632679 upper=1.57079632679 effort=0.01 velocity=100
- added joint joint_spherical_branch_51_branch_52_cylinder_Z: type revolute, parent branch_51, child branch_51_spherical_joint_link, origin xyz=-0.19 0 0 rpy=0 0 0, axis 0 0 1, limit lower=-1.57079632679 upper=1.57079632679 effort=0.01 velocity=100
- added joint joint_spherical_branch_52_branch_53_cylinder_Y: type revolute, parent branch_52_spherical_joint_link, child branch_53_cylinder, origin xyz=0 0 0 rpy=0 0 0, axis 0 1 0, limit lower=-1.57079632679 upper=1.57079632679 effort=0.01 velocity=100
- added joint joint_spherical_branch_52_branch_53_cylinder_Z: type revolute, parent branch_52, child branch_52_spherical_joint_link, origin xyz=-0.19 0 0 rpy=0 0 0, axis 0 0 1, limit lower=-1.57079632679 upper=1.57079632679 effort=0.01 velocity=100
- added joint joint_spherical_branch_53_branch_54_cylinder_Y: type revolute, parent branch_53_spherical_joint_link, child branch_54_cylinder, origin xyz=0 0 0 rpy=0 0 0, axis 0 1 0, limit lower=-1.57079632679 upper=1.57079632679 effort=0.01 velocity=100
- added joint joint_spherical_branch_53_branch_54_cylinder_Z: type revolute, parent branch_53, child branch_53_spherical_joint_link, origin xyz=-0.19 0 0 rpy=0 0 0, axis 0 0 1, limit lower=-1.57079632679 upper=1.57079632679 effort=0.01 velocity=100
- added joint joint_spherical_branch_54_branch_55_cylinder_Y: type revolute, parent branch_54_spherical_joint_link, child branch_55_cylinder, origin xyz=0 0 0 rpy=0 0 0, axis 0 1 0, limit lower=-1.57079632679 upper=1.57079632679 effort=0.01 velocity=100
- added joint joint_spherical_branch_54_branch_55_cylinder_Z: type revolute, parent branch_54, child branch_54_spherical_joint_link, origin xyz=-0.19 0 0 rpy=0 0 0, axis 0 0 1, limit lower=-1.57079632679 upper=1.57079632679 effort=0.01 velocity=100
- added joint joint_spherical_branch_60_branch_61_cylinder_Y: type revolute, parent branch_60_spherical_joint_link, child branch_61_cylinder, origin xyz=0 0 0 rpy=0 0 0, axis 0 1 0, limit lower=-1.57079632679 upper=1.57079632679 effort=0.01 velocity=100
- added joint joint_spherical_branch_60_branch_61_cylinder_Z: type revolute, parent branch_60, child branch_60_spherical_joint_link, origin xyz=-0.03875 0 0 rpy=0 0 0, axis 0 0 1, limit lower=-1.57079632679 upper=1.57079632679 effort=0.01 velocity=100
- added joint joint_spherical_branch_61_branch_62_cylinder_Y: type revolute, parent branch_61_spherical_joint_link, child branch_62_cylinder, origin xyz=0 0 0 rpy=0 0 0, axis 0 1 0, limit lower=-1.57079632679 upper=1.57079632679 effort=0.01 velocity=100
- added joint joint_spherical_branch_61_branch_62_cylinder_Z: type revolute, parent branch_61, child branch_61_spherical_joint_link, origin xyz=-0.19 0 0 rpy=0 0 0, axis 0 0 1, limit lower=-1.57079632679 upper=1.57079632679 effort=0.01 velocity=100
- added joint joint_spherical_branch_62_branch_63_cylinder_Y: type revolute, parent branch_62_spherical_joint_link, child branch_63_cylinder, origin xyz=0 0 0 rpy=0 0 0, axis 0 1 0, limit lower=-1.57079632679 upper=1.57079632679 effort=0.01 velocity=100
- added joint joint_spherical_branch_62_branch_63_cylinder_Z: type revolute, parent branch_62, child branch_62_spherical_joint_link, origin xyz=-0.19 0 0 rpy=0 0 0, axis 0 0 1, limit lower=-1.57079632679 upper=1.57079632679 effort=0.01 velocity=100
- added joint joint_spherical_branch_63_branch_64_cylinder_Y: type revolute, parent branch_63_spherical_joint_link, child branch_64_cylinder, origin xyz=0 0 0 rpy=0 0 0, axis 0 1 0, limit lower=-1.57079632679 upper=1.57079632679 effort=0.01 velocity=100
- added joint joint_spherical_branch_63_branch_64_cylinder_Z: type revolute, parent branch_63, child branch_63_spherical_joint_link, origin xyz=-0.19 0 0 rpy=0 0 0, axis 0 0 1, limit lower=-1.57079632679 upper=1.57079632679 effort=0.01 velocity=100
- added joint joint_spherical_branch_64_branch_65_cylinder_Y: type revolute, parent branch_64_spherical_joint_link, child branch_65_cylinder, origin xyz=0 0 0 rpy=0 0 0, axis 0 1 0, limit lower=-1.57079632679 upper=1.57079632679 effort=0.01 velocity=100
- added joint joint_spherical_branch_64_branch_65_cylinder_Z: type revolute, parent branch_64, child branch_64_spherical_joint_link, origin xyz=-0.19 0 0 rpy=0 0 0, axis 0 0 1, limit lower=-1.57079632679 upper=1.57079632679 effort=0.01 velocity=100
- added joint joint_spherical_branch_70_branch_71_cylinder_Y: type revolute, parent branch_70_spherical_joint_link, child branch_71_cylinder, origin xyz=0 0 0 rpy=0 0 0, axis 0 1 0, limit lower=-1.57079632679 upper=1.57079632679 effort=0.01 velocity=100
- added joint joint_spherical_branch_70_branch_71_cylinder_Z: type revolute, parent branch_70, child branch_70_spherical_joint_link, origin xyz=-0.03875 0 0 rpy=0 0 0, axis 0 0 1, limit lower=-1.57079632679 upper=1.57079632679 effort=0.01 velocity=100
- added joint joint_spherical_branch_71_branch_72_cylinder_Y: type revolute, parent branch_71_spherical_joint_link, child branch_72_cylinder, origin xyz=0 0 0 rpy=0 0 0, axis 0 1 0, limit lower=-1.57079632679 upper=1.57079632679 effort=0.01 velocity=100
- added joint joint_spherical_branch_71_branch_72_cylinder_Z: type revolute, parent branch_71, child branch_71_spherical_joint_link, origin xyz=-0.19 0 0 rpy=0 0 0, axis 0 0 1, limit lower=-1.57079632679 upper=1.57079632679 effort=0.01 velocity=100
- added joint joint_spherical_branch_72_branch_73_cylinder_Y: type revolute, parent branch_72_spherical_joint_link, child branch_73_cylinder, origin xyz=0 0 0 rpy=0 0 0, axis 0 1 0, limit lower=-1.57079632679 upper=1.57079632679 effort=0.01 velocity=100
- added joint joint_spherical_branch_72_branch_73_cylinder_Z: type revolute, parent branch_72, child branch_72_spherical_joint_link, origin xyz=-0.19 0 0 rpy=0 0 0, axis 0 0 1, limit lower=-1.57079632679 upper=1.57079632679 effort=0.01 velocity=100
- added joint joint_spherical_branch_73_branch_74_cylinder_Y: type revolute, parent branch_73_spherical_joint_link, child branch_74_cylinder, origin xyz=0 0 0 rpy=0 0 0, axis 0 1 0, limit lower=-1.57079632679 upper=1.57079632679 effort=0.01 velocity=100
- added joint joint_spherical_branch_73_branch_74_cylinder_Z: type revolute, parent branch_73, child branch_73_spherical_joint_link, origin xyz=-0.19 0 0 rpy=0 0 0, axis 0 0 1, limit lower=-1.57079632679 upper=1.57079632679 effort=0.01 velocity=100
- added joint joint_spherical_branch_74_branch_75_cylinder_Y: type revolute, parent branch_74_spherical_joint_link, child branch_75_cylinder, origin xyz=0 0 0 rpy=0 0 0, axis 0 1 0, limit lower=-1.57079632679 upper=1.57079632679 effort=0.01 velocity=100
- added joint joint_spherical_branch_74_branch_75_cylinder_Z: type revolute, parent branch_74, child branch_74_spherical_joint_link, origin xyz=-0.19 0 0 rpy=0 0 0, axis 0 0 1, limit lower=-1.57079632679 upper=1.57079632679 effort=0.01 velocity=100
