Commit message: Add more planar manipulators

File: data/robots/planar_manipulator/10dof_manip.urdf (robot description, URDF)
Before this commit: robot planar_manipulator/10dof_manip, 21 links, 20 joints
Links:
- removed link jlink10
- added link endeffectorL, mass 1; collision box size=0.1 0.4 0.1; visual box size=0.1 0.4 0.1
- added link endeffectorR, mass 1; collision box size=0.1 0.4 0.1; visual box size=0.1 0.4 0.1
Joints:
- removed joint joint_fixed_link9_jlink10
- added joint joint_fixed_link9_endeffectorL: type fixed, parent link9, child endeffectorL, origin xyz=0 1.7 0 rpy=0 0 0
- added joint joint_fixed_link9_endeffectorR: type fixed, parent link9, child endeffectorR, origin xyz=0 1.7 0 rpy=0 0 0

File: data/robots/planar_manipulator/10dof_manip_no_endeffector.urdf (robot description, URDF)
Before this commit: robot planar_manipulator/7dof_manip, 16 links, 15 joints
Links:
- removed link endeffectorL
- removed link endeffectorR
- added link jlink10, mass 1; collision cylinder length=0.1 radius=0.2; visual cylinder length=0.1 radius=0.2
- added link jlink7, mass 1; collision cylinder length=0.1 radius=0.2; visual cylinder length=0.1 radius=0.2
- added link jlink8, mass 1; collision cylinder length=0.1 radius=0.2; visual cylinder length=0.1 radius=0.2
- added link jlink9, mass 1; collision cylinder length=0.1 radius=0.2; visual cylinder length=0.1 radius=0.2
- added link link7, mass 1; collision box size=0.4 1.5 0.1; visual box size=0.4 1.5 0.1
- added link link8, mass 1; collision box size=0.4 1.5 0.1; visual box size=0.4 1.5 0.1
- added link link9, mass 1; collision box size=0.4 1.5 0.1; visual box size=0.4 1.5 0.1
Joints:
- removed joint joint_fixed_link6_endeffectorL
- removed joint joint_fixed_link6_endeffectorR
- added joint joint_fixed_link6_jlink7: type fixed, parent link6, child jlink7, origin xyz=0 1.9 0 rpy=0 0 0
- added joint joint_fixed_link7_jlink8: type fixed, parent link7, child jlink8, origin xyz=0 1.9 0 rpy=0 0 0
- added joint joint_fixed_link8_jlink9: type fixed, parent link8, child jlink9, origin xyz=0 1.9 0 rpy=0 0 0
- added joint joint_fixed_link9_jlink10: type fixed, parent link9, child jlink10, origin xyz=0 1.9 0 rpy=0 0 0
- added joint joint_revolute_jlink7_link7_Z: type revolute, parent jlink7, child link7, origin xyz=0 0 0 rpy=0 0 0, axis 0 0 1, limit lower=-3.14 upper=3.14 effort=0.01 velocity=100
- added joint joint_revolute_jlink8_link8_Z: type revolute, parent jlink8, child link8, origin xyz=0 0 0 rpy=0 0 0, axis 0 0 1, limit lower=-3.14 upper=3.14 effort=0.01 velocity=100
- added joint joint_revolute_jlink9_link9_Z: type revolute, parent jlink9, child link9, origin xyz=0 0 0 rpy=0 0 0, axis 0 0 1, limit lower=-3.14 upper=3.14 effort=0.01 velocity=100

File: data/robots/planar_manipulator/11dof_manip.urdf (robot description, URDF)
Before this commit: robot planar_manipulator/11dof_manip, 23 links, 22 joints
Links:
- removed link jlink11
- added link endeffectorL, mass 1; collision box size=0.1 0.4 0.1; visual box size=0.1 0.4 0.1
- added link endeffectorR, mass 1; collision box size=0.1 0.4 0.1; visual box size=0.1 0.4 0.1
Joints:
- removed joint joint_fixed_link10_jlink11
- added joint joint_fixed_link10_endeffectorL: type fixed, parent link10, child endeffectorL, origin xyz=0 1.7 0 rpy=0 0 0
- added joint joint_fixed_link10_endeffectorR: type fixed, parent link10, child endeffectorR, origin xyz=0 1.7 0 rpy=0 0 0

File: data/robots/planar_manipulator/11dof_manip_no_endeffector.urdf (robot description, URDF)
Before this commit: robot planar_manipulator/7dof_manip, 16 links, 15 joints
Links:
- removed link endeffectorL
- removed link endeffectorR
- added link jlink10, mass 1; collision cylinder length=0.1 radius=0.2; visual cylinder length=0.1 radius=0.2
- added link jlink11, mass 1; collision cylinder length=0.1 radius=0.2; visual cylinder length=0.1 radius=0.2
- added link jlink7, mass 1; collision cylinder length=0.1 radius=0.2; visual cylinder length=0.1 radius=0.2
- added link jlink8, mass 1; collision cylinder length=0.1 radius=0.2; visual cylinder length=0.1 radius=0.2
- added link jlink9, mass 1; collision cylinder length=0.1 radius=0.2; visual cylinder length=0.1 radius=0.2
- added link link10, mass 1; collision box size=0.4 1.5 0.1; visual box size=0.4 1.5 0.1
- added link link7, mass 1; collision box size=0.4 1.5 0.1; visual box size=0.4 1.5 0.1
- added link link8, mass 1; collision box size=0.4 1.5 0.1; visual box size=0.4 1.5 0.1
- added link link9, mass 1; collision box size=0.4 1.5 0.1; visual box size=0.4 1.5 0.1
Joints:
- removed joint joint_fixed_link6_endeffectorL
- removed joint joint_fixed_link6_endeffectorR
- added joint joint_fixed_link10_jlink11: type fixed, parent link10, child jlink11, origin xyz=0 1.9 0 rpy=0 0 0
- added joint joint_fixed_link6_jlink7: type fixed, parent link6, child jlink7, origin xyz=0 1.9 0 rpy=0 0 0
- added joint joint_fixed_link7_jlink8: type fixed, parent link7, child jlink8, origin xyz=0 1.9 0 rpy=0 0 0
- added joint joint_fixed_link8_jlink9: type fixed, parent link8, child jlink9, origin xyz=0 1.9 0 rpy=0 0 0
- added joint joint_fixed_link9_jlink10: type fixed, parent link9, child jlink10, origin xyz=0 1.9 0 rpy=0 0 0
- added joint joint_revolute_jlink10_link10_Z: type revolute, parent jlink10, child link10, origin xyz=0 0 0 rpy=0 0 0, axis 0 0 1, limit lower=-3.14 upper=3.14 effort=0.01 velocity=100
- added joint joint_revolute_jlink7_link7_Z: type revolute, parent jlink7, child link7, origin xyz=0 0 0 rpy=0 0 0, axis 0 0 1, limit lower=-3.14 upper=3.14 effort=0.01 velocity=100
- added joint joint_revolute_jlink8_link8_Z: type revolute, parent jlink8, child link8, origin xyz=0 0 0 rpy=0 0 0, axis 0 0 1, limit lower=-3.14 upper=3.14 effort=0.01 velocity=100
- added joint joint_revolute_jlink9_link9_Z: type revolute, parent jlink9, child link9, origin xyz=0 0 0 rpy=0 0 0, axis 0 0 1, limit lower=-3.14 upper=3.14 effort=0.01 velocity=100

File: data/robots/planar_manipulator/12dof_manip.urdf (robot description, URDF)
Before this commit: robot planar_manipulator/12dof_manip, 25 links, 24 joints
Links:
- removed link jlink12
- added link endeffectorL, mass 1; collision box size=0.1 0.4 0.1; visual box size=0.1 0.4 0.1
- added link endeffectorR, mass 1; collision box size=0.1 0.4 0.1; visual box size=0.1 0.4 0.1
Joints:
- removed joint joint_fixed_link11_jlink12
- added joint joint_fixed_link11_endeffectorL: type fixed, parent link11, child endeffectorL, origin xyz=0 1.7 0 rpy=0 0 0
- added joint joint_fixed_link11_endeffectorR: type fixed, parent link11, child endeffectorR, origin xyz=0 1.7 0 rpy=0 0 0

File: data/robots/planar_manipulator/12dof_manip_no_endeffector.urdf (robot description, URDF)
Before this commit: robot planar_manipulator/7dof_manip, 16 links, 15 joints
Links:
- removed link endeffectorL
- removed link endeffectorR
- added link jlink10, mass 1; collision cylinder length=0.1 radius=0.2; visual cylinder length=0.1 radius=0.2
- added link jlink11, mass 1; collision cylinder length=0.1 radius=0.2; visual cylinder length=0.1 radius=0.2
- added link jlink12, mass 1; collision cylinder length=0.1 radius=0.2; visual cylinder length=0.1 radius=0.2
- added link jlink7, mass 1; collision cylinder length=0.1 radius=0.2; visual cylinder length=0.1 radius=0.2
- added link jlink8, mass 1; collision cylinder length=0.1 radius=0.2; visual cylinder length=0.1 radius=0.2
- added link jlink9, mass 1; collision cylinder length=0.1 radius=0.2; visual cylinder length=0.1 radius=0.2
- added link link10, mass 1; collision box size=0.4 1.5 0.1; visual box size=0.4 1.5 0.1
- added link link11, mass 1; collision box size=0.4 1.5 0.1; visual box size=0.4 1.5 0.1
- added link link7, mass 1; collision box size=0.4 1.5 0.1; visual box size=0.4 1.5 0.1
- added link link8, mass 1; collision box size=0.4 1.5 0.1; visual box size=0.4 1.5 0.1
- added link link9, mass 1; collision box size=0.4 1.5 0.1; visual box size=0.4 1.5 0.1
Joints:
- removed joint joint_fixed_link6_endeffectorL
- removed joint joint_fixed_link6_endeffectorR
- added joint joint_fixed_link10_jlink11: type fixed, parent link10, child jlink11, origin xyz=0 1.9 0 rpy=0 0 0
- added joint joint_fixed_link11_jlink12: type fixed, parent link11, child jlink12, origin xyz=0 1.9 0 rpy=0 0 0
- added joint joint_fixed_link6_jlink7: type fixed, parent link6, child jlink7, origin xyz=0 1.9 0 rpy=0 0 0
- added joint joint_fixed_link7_jlink8: type fixed, parent link7, child jlink8, origin xyz=0 1.9 0 rpy=0 0 0
- added joint joint_fixed_link8_jlink9: type fixed, parent link8, child jlink9, origin xyz=0 1.9 0 rpy=0 0 0
- added joint joint_fixed_link9_jlink10: type fixed, parent link9, child jlink10, origin xyz=0 1.9 0 rpy=0 0 0
- added joint joint_revolute_jlink10_link10_Z: type revolute, parent jlink10, child link10, origin xyz=0 0 0 rpy=0 0 0, axis 0 0 1, limit lower=-3.14 upper=3.14 effort=0.01 velocity=100
- added joint joint_revolute_jlink11_link11_Z: type revolute, parent jlink11, child link11, origin xyz=0 0 0 rpy=0 0 0, axis 0 0 1, limit lower=-3.14 upper=3.14 effort=0.01 velocity=100
- added joint joint_revolute_jlink7_link7_Z: type revolute, parent jlink7, child link7, origin xyz=0 0 0 rpy=0 0 0, axis 0 0 1, limit lower=-3.14 upper=3.14 effort=0.01 velocity=100
- added joint joint_revolute_jlink8_link8_Z: type revolute, parent jlink8, child link8, origin xyz=0 0 0 rpy=0 0 0, axis 0 0 1, limit lower=-3.14 upper=3.14 effort=0.01 velocity=100
- added joint joint_revolute_jlink9_link9_Z: type revolute, parent jlink9, child link9, origin xyz=0 0 0 rpy=0 0 0, axis 0 0 1, limit lower=-3.14 upper=3.14 effort=0.01 velocity=100

File: data/robots/planar_manipulator/13dof_manip.urdf (robot description, URDF)
Before this commit: robot planar_manipulator/13dof_manip, 27 links, 26 joints
Links:
- removed link jlink13
- added link endeffectorL, mass 1; collision box size=0.1 0.4 0.1; visual box size=0.1 0.4 0.1
- added link endeffectorR, mass 1; collision box size=0.1 0.4 0.1; visual box size=0.1 0.4 0.1
Joints:
- removed joint joint_fixed_link12_jlink13
- added joint joint_fixed_link12_endeffectorL: type fixed, parent link12, child endeffectorL, origin xyz=0 1.7 0 rpy=0 0 0
- added joint joint_fixed_link12_endeffectorR: type fixed, parent link12, child endeffectorR, origin xyz=0 1.7 0 rpy=0 0 0

File: data/robots/planar_manipulator/13dof_manip_no_endeffector.urdf (robot description, URDF)
Before this commit: robot planar_manipulator/7dof_manip, 16 links, 15 joints
Links:
- removed link endeffectorL
- removed link endeffectorR
- added link jlink10, mass 1; collision cylinder length=0.1 radius=0.2; visual cylinder length=0.1 radius=0.2
- added link jlink11, mass 1; collision cylinder length=0.1 radius=0.2; visual cylinder length=0.1 radius=0.2
- added link jlink12, mass 1; collision cylinder length=0.1 radius=0.2; visual cylinder length=0.1 radius=0.2
- added link jlink13, mass 1; collision cylinder length=0.1 radius=0.2; visual cylinder length=0.1 radius=0.2
- added link jlink7, mass 1; collision cylinder length=0.1 radius=0.2; visual cylinder length=0.1 radius=0.2
- added link jlink8, mass 1; collision cylinder length=0.1 radius=0.2; visual cylinder length=0.1 radius=0.2
- added link jlink9, mass 1; collision cylinder length=0.1 radius=0.2; visual cylinder length=0.1 radius=0.2
- added link link10, mass 1; collision box size=0.4 1.5 0.1; visual box size=0.4 1.5 0.1
- added link link11, mass 1; collision box size=0.4 1.5 0.1; visual box size=0.4 1.5 0.1
- added link link12, mass 1; collision box size=0.4 1.5 0.1; visual box size=0.4 1.5 0.1
- added link link7, mass 1; collision box size=0.4 1.5 0.1; visual box size=0.4 1.5 0.1
- added link link8, mass 1; collision box size=0.4 1.5 0.1; visual box size=0.4 1.5 0.1
- added link link9, mass 1; collision box size=0.4 1.5 0.1; visual box size=0.4 1.5 0.1
Joints:
- removed joint joint_fixed_link6_endeffectorL
- removed joint joint_fixed_link6_endeffectorR
- added joint joint_fixed_link10_jlink11: type fixed, parent link10, child jlink11, origin xyz=0 1.9 0 rpy=0 0 0
- added joint joint_fixed_link11_jlink12: type fixed, parent link11, child jlink12, origin xyz=0 1.9 0 rpy=0 0 0
- added joint joint_fixed_link12_jlink13: type fixed, parent link12, child jlink13, origin xyz=0 1.9 0 rpy=0 0 0
- added joint joint_fixed_link6_jlink7: type fixed, parent link6, child jlink7, origin xyz=0 1.9 0 rpy=0 0 0
- added joint joint_fixed_link7_jlink8: type fixed, parent link7, child jlink8, origin xyz=0 1.9 0 rpy=0 0 0
- added joint joint_fixed_link8_jlink9: type fixed, parent link8, child jlink9, origin xyz=0 1.9 0 rpy=0 0 0
- added joint joint_fixed_link9_jlink10: type fixed, parent link9, child jlink10, origin xyz=0 1.9 0 rpy=0 0 0
- added joint joint_revolute_jlink10_link10_Z: type revolute, parent jlink10, child link10, origin xyz=0 0 0 rpy=0 0 0, axis 0 0 1, limit lower=-3.14 upper=3.14 effort=0.01 velocity=100
- added joint joint_revolute_jlink11_link11_Z: type revolute, parent jlink11, child link11, origin xyz=0 0 0 rpy=0 0 0, axis 0 0 1, limit lower=-3.14 upper=3.14 effort=0.01 velocity=100
- added joint joint_revolute_jlink12_link12_Z: type revolute, parent jlink12, child link12, origin xyz=0 0 0 rpy=0 0 0, axis 0 0 1, limit lower=-3.14 upper=3.14 effort=0.01 velocity=100
- added joint joint_revolute_jlink7_link7_Z: type revolute, parent jlink7, child link7, origin xyz=0 0 0 rpy=0 0 0, axis 0 0 1, limit lower=-3.14 upper=3.14 effort=0.01 velocity=100
- added joint joint_revolute_jlink8_link8_Z: type revolute, parent jlink8, child link8, origin xyz=0 0 0 rpy=0 0 0, axis 0 0 1, limit lower=-3.14 upper=3.14 effort=0.01 velocity=100
- added joint joint_revolute_jlink9_link9_Z: type revolute, parent jlink9, child link9, origin xyz=0 0 0 rpy=0 0 0, axis 0 0 1, limit lower=-3.14 upper=3.14 effort=0.01 velocity=100

File: data/robots/planar_manipulator/14dof_manip.urdf (robot description, URDF)
Before this commit: robot planar_manipulator/14dof_manip, 29 links, 28 joints
Links:
- removed link jlink14
- added link endeffectorL, mass 1; collision box size=0.1 0.4 0.1; visual box size=0.1 0.4 0.1
- added link endeffectorR, mass 1; collision box size=0.1 0.4 0.1; visual box size=0.1 0.4 0.1
Joints:
- removed joint joint_fixed_link13_jlink14
- added joint joint_fixed_link13_endeffectorL: type fixed, parent link13, child endeffectorL, origin xyz=0 1.7 0 rpy=0 0 0
- added joint joint_fixed_link13_endeffectorR: type fixed, parent link13, child endeffectorR, origin xyz=0 1.7 0 rpy=0 0 0

File: data/robots/planar_manipulator/14dof_manip_no_endeffector.urdf (robot description, URDF)
Before this commit: robot planar_manipulator/9dof_manip, 20 links, 19 joints
Links:
- removed link endeffectorL
- removed link endeffectorR
- added link jlink10, mass 1; collision cylinder length=0.1 radius=0.2; visual cylinder length=0.1 radius=0.2
- added link jlink11, mass 1; collision cylinder length=0.1 radius=0.2; visual cylinder length=0.1 radius=0.2
- added link jlink12, mass 1; collision cylinder length=0.1 radius=0.2; visual cylinder length=0.1 radius=0.2
- added link jlink13, mass 1; collision cylinder length=0.1 radius=0.2; visual cylinder length=0.1 radius=0.2
- added link jlink14, mass 1; collision cylinder length=0.1 radius=0.2; visual cylinder length=0.1 radius=0.2
- added link jlink9, mass 1; collision cylinder length=0.1 radius=0.2; visual cylinder length=0.1 radius=0.2
- added link link10, mass 1; collision box size=0.4 1.5 0.1; visual box size=0.4 1.5 0.1
- added link link11, mass 1; collision box size=0.4 1.5 0.1; visual box size=0.4 1.5 0.1
- added link link12, mass 1; collision box size=0.4 1.5 0.1; visual box size=0.4 1.5 0.1
- added link link13, mass 1; collision box size=0.4 1.5 0.1; visual box size=0.4 1.5 0.1
- added link link9, mass 1; collision box size=0.4 1.5 0.1; visual box size=0.4 1.5 0.1
Joints:
- removed joint joint_fixed_link8_endeffectorL
- removed joint joint_fixed_link8_endeffectorR
- added joint joint_fixed_link10_jlink11: type fixed, parent link10, child jlink11, origin xyz=0 1.9 0 rpy=0 0 0
- added joint joint_fixed_link11_jlink12: type fixed, parent link11, child jlink12, origin xyz=0 1.9 0 rpy=0 0 0
- added joint joint_fixed_link12_jlink13: type fixed, parent link12, child jlink13, origin xyz=0 1.9 0 rpy=0 0 0
- added joint joint_fixed_link13_jlink14: type fixed, parent link13, child jlink14, origin xyz=0 1.9 0 rpy=0 0 0
- added joint joint_fixed_link8_jlink9: type fixed, parent link8, child jlink9, origin xyz=0 1.9 0 rpy=0 0 0
- added joint joint_fixed_link9_jlink10: type fixed, parent link9, child jlink10, origin xyz=0 1.9 0 rpy=0 0 0
- added joint joint_revolute_jlink10_link10_Z: type revolute, parent jlink10, child link10, origin xyz=0 0 0 rpy=0 0 0, axis 0 0 1, limit lower=-3.14 upper=3.14 effort=0.01 velocity=100
- added joint joint_revolute_jlink11_link11_Z: type revolute, parent jlink11, child link11, origin xyz=0 0 0 rpy=0 0 0, axis 0 0 1, limit lower=-3.14 upper=3.14 effort=0.01 velocity=100
- added joint joint_revolute_jlink12_link12_Z: type revolute, parent jlink12, child link12, origin xyz=0 0 0 rpy=0 0 0, axis 0 0 1, limit lower=-3.14 upper=3.14 effort=0.01 velocity=100
- added joint joint_revolute_jlink13_link13_Z: type revolute, parent jlink13, child link13, origin xyz=0 0 0 rpy=0 0 0, axis 0 0 1, limit lower=-3.14 upper=3.14 effort=0.01 velocity=100
- added joint joint_revolute_jlink9_link9_Z: type revolute, parent jlink9, child link9, origin xyz=0 0 0 rpy=0 0 0, axis 0 0 1, limit lower=-3.14 upper=3.14 effort=0.01 velocity=100

File: data/robots/planar_manipulator/2dof_manip_no_endeffector.urdf (robot description, URDF)
Before this commit: robot planar_manipulator/3dof_manip, 8 links, 7 joints
Links:
- removed link endeffectorL
- removed link endeffectorR
- removed link link2
Joints:
- removed joint joint_fixed_link2_endeffectorL
- removed joint joint_fixed_link2_endeffectorR
- removed joint joint_revolute_jlink2_link2_Z

File: data/robots/planar_manipulator/3dof_manip_no_endeffector.urdf (robot description, URDF)
Before this commit: robot planar_manipulator/4dof_manip, 10 links, 9 joints
Links:
- removed link endeffectorL
- removed link endeffectorR
- removed link link3
Joints:
- removed joint joint_fixed_link3_endeffectorL
- removed joint joint_fixed_link3_endeffectorR
- removed joint joint_revolute_jlink3_link3_Z

File: data/robots/planar_manipulator/4dof_manip_no_endeffector.urdf (robot description, URDF)
Before this commit: robot planar_manipulator/7dof_manip, 16 links, 15 joints
Links:
- removed link endeffectorL
- removed link endeffectorR
- removed link jlink5
- removed link jlink6
- removed link link4
- removed link link5
- removed link link6
Joints:
- removed joint joint_fixed_link4_jlink5
- removed joint joint_fixed_link5_jlink6
- removed joint joint_fixed_link6_endeffectorL
- removed joint joint_fixed_link6_endeffectorR
- removed joint joint_revolute_jlink4_link4_Z
- removed joint joint_revolute_jlink5_link5_Z
- removed joint joint_revolute_jlink6_link6_Z

File: data/robots/planar_manipulator/5dof_manip.urdf (robot description, URDF)
Before this commit: robot planar_manipulator/5dof_manip, 11 links, 10 joints
Links:
- removed link jlink5
- added link endeffectorL, mass 1; collision box size=0.1 0.4 0.1; visual box size=0.1 0.4 0.1
- added link endeffectorR, mass 1; collision box size=0.1 0.4 0.1; visual box size=0.1 0.4 0.1
Joints:
- removed joint joint_fixed_link4_jlink5
- added joint joint_fixed_link4_endeffectorL: type fixed, parent link4, child endeffectorL, origin xyz=0 1.7 0 rpy=0 0 0
- added joint joint_fixed_link4_endeffectorR: type fixed, parent link4, child endeffectorR, origin xyz=0 1.7 0 rpy=0 0 0

File: data/robots/planar_manipulator/5dof_manip_no_endeffector.urdf (robot description, URDF)
Before this commit: robot planar_manipulator/7dof_manip, 16 links, 15 joints
Links:
- removed link endeffectorL
- removed link endeffectorR
- removed link jlink6
- removed link link5
- removed link link6
Joints:
- removed joint joint_fixed_link5_jlink6
- removed joint joint_fixed_link6_endeffectorL
- removed joint joint_fixed_link6_endeffectorR
- removed joint joint_revolute_jlink5_link5_Z
- removed joint joint_revolute_jlink6_link6_Z

File: data/robots/planar_manipulator/6dof_manip.urdf (robot description, URDF)
Before this commit: robot planar_manipulator/6dof_manip, 13 links, 12 joints
Links:
- removed link jlink6
- added link endeffectorL, mass 1; collision box size=0.1 0.4 0.1; visual box size=0.1 0.4 0.1
- added link endeffectorR, mass 1; collision box size=0.1 0.4 0.1; visual box size=0.1 0.4 0.1
Joints:
- removed joint joint_fixed_link5_jlink6
- added joint joint_fixed_link5_endeffectorL: type fixed, parent link5, child endeffectorL, origin xyz=0 1.7 0 rpy=0 0 0
- added joint joint_fixed_link5_endeffectorR: type fixed, parent link5, child endeffectorR, origin xyz=0 1.7 0 rpy=0 0 0

File: data/robots/planar_manipulator/6dof_manip_no_endeffector.urdf (robot description, URDF)
Before this commit: robot planar_manipulator/7dof_manip, 16 links, 15 joints
Links:
- removed link endeffectorL
- removed link endeffectorR
- removed link link6
Joints:
- removed joint joint_fixed_link6_endeffectorL
- removed joint joint_fixed_link6_endeffectorR
- removed joint joint_revolute_jlink6_link6_Z

File: data/robots/planar_manipulator/7dof_manip_no_endeffector.urdf (robot description, URDF)
Before this commit: robot planar_manipulator/7dof_manip, 16 links, 15 joints
Links:
- removed link endeffectorL
- removed link endeffectorR
- added link jlink7, mass 1; collision cylinder length=0.1 radius=0.2; visual cylinder length=0.1 radius=0.2
Joints:
- removed joint joint_fixed_link6_endeffectorL
- removed joint joint_fixed_link6_endeffectorR
- added joint joint_fixed_link6_jlink7: type fixed, parent link6, child jlink7, origin xyz=0 1.9 0 rpy=0 0 0

File: data/robots/planar_manipulator/8dof_manip.urdf (robot description, URDF)
Before this commit: robot planar_manipulator/8dof_manip, 17 links, 16 joints
Links:
- removed link jlink8
- added link endeffectorL, mass 1; collision box size=0.1 0.4 0.1; visual box size=0.1 0.4 0.1
- added link endeffectorR, mass 1; collision box size=0.1 0.4 0.1; visual box size=0.1 0.4 0.1
Joints:
- removed joint joint_fixed_link7_jlink8
- added joint joint_fixed_link7_endeffectorL: type fixed, parent link7, child endeffectorL, origin xyz=0 1.7 0 rpy=0 0 0
- added joint joint_fixed_link7_endeffectorR: type fixed, parent link7, child endeffectorR, origin xyz=0 1.7 0 rpy=0 0 0
