Commit message: Add more planar manipulators

File: data/robots/planar_manipulator/8dof_manip_no_endeffector.urdf (robot description, URDF)
Before this commit: robot planar_manipulator/7dof_manip, 16 links, 15 joints
Links:
- removed link endeffectorL
- removed link endeffectorR
- added link jlink7, mass 1; collision cylinder length=0.1 radius=0.2; visual cylinder length=0.1 radius=0.2
- added link jlink8, mass 1; collision cylinder length=0.1 radius=0.2; visual cylinder length=0.1 radius=0.2
- added link link7, mass 1; collision box size=0.4 1.5 0.1; visual box size=0.4 1.5 0.1
Joints:
- removed joint joint_fixed_link6_endeffectorL
- removed joint joint_fixed_link6_endeffectorR
- added joint joint_fixed_link6_jlink7: type fixed, parent link6, child jlink7, origin xyz=0 1.9 0 rpy=0 0 0
- added joint joint_fixed_link7_jlink8: type fixed, parent link7, child jlink8, origin xyz=0 1.9 0 rpy=0 0 0
- added joint joint_revolute_jlink7_link7_Z: type revolute, parent jlink7, child link7, origin xyz=0 0 0 rpy=0 0 0, axis 0 0 1, limit lower=-3.14 upper=3.14 effort=0.01 velocity=100
