Commit message: Multiple contacts wip2

File: data/robots/planar_manipulator/3dof_manip_no_endeffector_test_object.urdf (robot description, URDF)
Before this commit: robot planar_manipulator/2dof_manip_no_endeffector, 5 links, 4 joints
Links:
- added link jlink3, mass 1
- added link link2, mass 1; collision box size=0.1 1.5 0.1; visual box size=0.1 1.5 0.1
- link jlink2: geometry collision cylinder length=0.1 radius=0.2; visual cylinder length=0.1 radius=0.2
Joints:
- added joint joint_fixed_link2_jlink3: type fixed, parent link2, child jlink3, origin xyz=0 1.9 0 rpy=0 0 0
- added joint joint_revolute_jlink2_link2_Z: type revolute, parent jlink2, child link2, origin xyz=0 0 0 rpy=0 0 0, axis 0 0 1, limit lower=-3.14 upper=3.14 effort=0.01 velocity=100
