Commit message: Transition Constraint 1.0

File: data/robots/planar_manipulator/3dof_manip_no_endeffector.urdf (robot description, URDF)
Before this commit: robot planar_manipulator/3dof_manip_no_endeffector, 7 links, 6 joints
Links:
- link jlink0: geometry 
- link jlink1: geometry collision cylinder length=0.1 radius=0.1; visual cylinder length=0.1 radius=0.1
- link jlink2: geometry collision cylinder length=0.1 radius=0.1; visual cylinder length=0.1 radius=0.1
- link jlink3: geometry 
- link link0: geometry collision box size=0.1 1.5 0.1; visual box size=0.1 1.5 0.1
- link link1: geometry collision box size=0.1 1.5 0.1; visual box size=0.1 1.5 0.1
- link link2: geometry collision box size=0.25 1.5 0.1; visual box size=0.25 1.5 0.1

Commit message: New Scenarios 7D manip, 3D sphere

File: data/robots/planar_manipulator/3dof_manip_no_endeffector.urdf (robot description, URDF)
Before this commit: robot planar_manipulator/3dof_manip_no_endeffector, 7 links, 6 joints
Links:
- link link1: geometry collision box size=0.25 1.5 0.1; visual box size=0.25 1.5 0.1

Commit message: Add contact point visualization

File: data/robots/planar_manipulator/3dof_manip_no_endeffector.urdf (robot description, URDF)
Before this commit: robot planar_manipulator/3dof_manip_no_endeffector, 7 links, 6 joints
Links:
- link jlink3: geometry visual sphere radius=0.15
