Commit message: Fix URDF script to generate snake

File: data/robots/snake/snake_0_segments.urdf (robot description, URDF)
Before this commit: robot snake/snake_head_inner, 2 links, 1 joints
Links:
- removed link head
- added link body0, mass 1; collision cylinder length=0.12 radius=0.12; visual cylinder length=0.12 radius=0.12
Joints:
- removed joint joint_eye_head
- added joint joint_fixed_eye_body0: type fixed, parent eye, child body0, origin xyz=-0.06 0 0 rpy=0 0 0

File: data/robots/snake/snake_0_segments_sphere_outer.urdf (robot description, URDF)
Before this commit: robot snake/snake_sphere_outer, 1 links, 0 joints
Links:
- link body: geometry collision sphere radius=0.169705627485; visual sphere radius=0.169705627485

Commit message: Clean up QRRT

File: data/robots/snake/snake_0_segments.urdf (robot description, URDF)
Before this commit: robot snake/snake_0_segments, 2 links, 1 joints
Links:
- link body0: geometry collision cylinder length=0.1 radius=0.1; visual cylinder length=0.1 radius=0.1
- link eye: geometry collision sphere radius=0.1; visual sphere radius=0.1
Joints:
- joint joint_fixed_eye_body0: origin xyz=-0.06 0 0 rpy=0 0 0 -> xyz=-0.05 0 0 rpy=0 0 0

File: data/robots/snake/snake_0_segments_sphere_inner.urdf (robot description, URDF)
Before this commit: robot snake/snake_0_segments_sphere_inner, 1 links, 0 joints
Links:
- link body: geometry collision sphere radius=0.1; visual sphere radius=0.1

File: data/robots/snake/snake_0_segments_sphere_outer.urdf (robot description, URDF)
Before this commit: robot snake/snake_0_segments_sphere_outer, 1 links, 0 joints
Links:
- link body: geometry collision sphere radius=0.141421356237; visual sphere radius=0.141421356237

File: data/robots/snake/snake_1_segments.urdf (robot description, URDF)
Before this commit: robot snake/snake_1_segments, 5 links, 4 joints
Links:
- link body0: geometry collision cylinder length=0.1 radius=0.1; visual cylinder length=0.1 radius=0.1
- link body1: geometry collision cylinder length=0.3 radius=0.1; visual cylinder length=0.3 radius=0.1
- link body1_joint_link: geometry collision sphere radius=0.07; visual sphere radius=0.07
- link eye: geometry collision sphere radius=0.1; visual sphere radius=0.1
Joints:
- joint joint_fixed_eye_body0: origin xyz=-0.06 0 0 rpy=0 0 0 -> xyz=-0.05 0 0 rpy=0 0 0
- joint joint_spherical_body1_joint_link_body1_Y: limit lower=-0.785398163397 upper=0.785398163397 effort=0.01 velocity=100 -> lower=-1.1780972451 upper=1.1780972451 effort=0.01 velocity=100
- joint joint_spherical_body1_joint_link_body1_Z: limit lower=-0.785398163397 upper=0.785398163397 effort=0.01 velocity=100 -> lower=-1.1780972451 upper=1.1780972451 effort=0.01 velocity=100

File: data/robots/snake/snake_2_segments.urdf (robot description, URDF)
Before this commit: robot snake/snake_2_segments, 8 links, 7 joints
Links:
- link body0: geometry collision cylinder length=0.1 radius=0.1; visual cylinder length=0.1 radius=0.1
- link body1: geometry collision cylinder length=0.3 radius=0.1; visual cylinder length=0.3 radius=0.1
- link body1_joint_link: geometry collision sphere radius=0.07; visual sphere radius=0.07
- link body2: geometry collision cylinder length=0.3 radius=0.1; visual cylinder length=0.3 radius=0.1
- link body2_joint_link: geometry collision sphere radius=0.07; visual sphere radius=0.07
- link eye: geometry collision sphere radius=0.1; visual sphere radius=0.1
Joints:
- joint joint_fixed_body1_body2_joint_link: origin xyz=-0.42001 0 0 rpy=0 0 0 -> xyz=-0.44001 0 0 rpy=0 0 0
- joint joint_fixed_eye_body0: origin xyz=-0.06 0 0 rpy=0 0 0 -> xyz=-0.05 0 0 rpy=0 0 0
- joint joint_spherical_body1_joint_link_body1_Y: limit lower=-0.785398163397 upper=0.785398163397 effort=0.01 velocity=100 -> lower=-1.1780972451 upper=1.1780972451 effort=0.01 velocity=100
- joint joint_spherical_body1_joint_link_body1_Z: limit lower=-0.785398163397 upper=0.785398163397 effort=0.01 velocity=100 -> lower=-1.1780972451 upper=1.1780972451 effort=0.01 velocity=100
- joint joint_spherical_body2_joint_link_body2_Y: limit lower=-0.785398163397 upper=0.785398163397 effort=0.01 velocity=100 -> lower=-1.1780972451 upper=1.1780972451 effort=0.01 velocity=100
- joint joint_spherical_body2_joint_link_body2_Z: limit lower=-0.785398163397 upper=0.785398163397 effort=0.01 velocity=100 -> lower=-1.1780972451 upper=1.1780972451 effort=0.01 velocity=100

File: data/robots/snake/snake_2_segments_sphere_outer.urdf (robot description, URDF)
Before this commit: robot snake/snake_2_segments_sphere_outer, 1 links, 0 joints
Links:
- link body: geometry collision sphere radius=0.98; visual sphere radius=0.98
