Commit message: Fix box

File: data/robots/snake/snake_0_segments_sphere_outer.urdf (robot description, URDF)
Before this commit: robot snake/snake_0_segments_sphere_outer, 1 links, 0 joints
Links:
- link body: geometry collision sphere radius=0.14142135623730953; visual sphere radius=0.14142135623730953

File: data/robots/snake/snake_1_segments.urdf (robot description, URDF)
Before this commit: robot snake/snake_1_segments, 5 links, 4 joints
Links:
- link body1: geometry collision cylinder length=0.30000000000000004 radius=0.1; visual cylinder length=0.30000000000000004 radius=0.1
- link body1_joint_link: geometry collision sphere radius=0.06999999999999999; visual sphere radius=0.06999999999999999
Joints:
- joint joint_fixed_body0_body1_joint_link: origin xyz=-0.12001 0 0 rpy=0 0 0 -> xyz=-0.12000999999999999 0 0 rpy=0 0 0
- joint joint_spherical_body1_joint_link_body1_Y: limit lower=-1.1780972451 upper=1.1780972451 effort=0.01 velocity=100 -> lower=-1.1780972450961724 upper=1.1780972450961724 effort=0.01 velocity=100
- joint joint_spherical_body1_joint_link_body1_Z: limit lower=-1.1780972451 upper=1.1780972451 effort=0.01 velocity=100 -> lower=-1.1780972450961724 upper=1.1780972450961724 effort=0.01 velocity=100

File: data/robots/snake/snake_2_segments.urdf (robot description, URDF)
Before this commit: robot snake/snake_2_segments, 8 links, 7 joints
Links:
- link body1: geometry collision cylinder length=0.30000000000000004 radius=0.1; visual cylinder length=0.30000000000000004 radius=0.1
- link body1_joint_link: geometry collision sphere radius=0.06999999999999999; visual sphere radius=0.06999999999999999
- link body2: geometry collision cylinder length=0.30000000000000004 radius=0.1; visual cylinder length=0.30000000000000004 radius=0.1
- link body2_joint_link: geometry collision sphere radius=0.06999999999999999; visual sphere radius=0.06999999999999999
Joints:
- joint joint_fixed_body0_body1_joint_link: origin xyz=-0.12001 0 0 rpy=0 0 0 -> xyz=-0.12000999999999999 0 0 rpy=0 0 0
- joint joint_fixed_body1_body2_joint_link: origin xyz=-0.44001 0 0 rpy=0 0 0 -> xyz=-0.44001000000000007 0 0 rpy=0 0 0
- joint joint_spherical_body1_joint_link_body1_Y: limit lower=-1.1780972451 upper=1.1780972451 effort=0.01 velocity=100 -> lower=-1.1780972450961724 upper=1.1780972450961724 effort=0.01 velocity=100
- joint joint_spherical_body1_joint_link_body1_Z: limit lower=-1.1780972451 upper=1.1780972451 effort=0.01 velocity=100 -> lower=-1.1780972450961724 upper=1.1780972450961724 effort=0.01 velocity=100
- joint joint_spherical_body2_joint_link_body2_Y: limit lower=-1.1780972451 upper=1.1780972451 effort=0.01 velocity=100 -> lower=-1.1780972450961724 upper=1.1780972450961724 effort=0.01 velocity=100
- joint joint_spherical_body2_joint_link_body2_Z: limit lower=-1.1780972451 upper=1.1780972451 effort=0.01 velocity=100 -> lower=-1.1780972450961724 upper=1.1780972450961724 effort=0.01 velocity=100

File: data/robots/snake/snake_2_segments_sphere_outer.urdf (robot description, URDF)
Before this commit: robot snake/snake_2_segments_sphere_outer, 1 links, 0 joints
Links:
- link body: geometry collision sphere radius=0.9800000000000001; visual sphere radius=0.9800000000000001
