Commit message: Add PR2 decomposition and environment.

File: data/robots/PR2/pr2_34D.urdf (robot description, URDF)
Before this commit: robot pr2, 47 links, 46 joints
Links:
- added link l_elbow_flex_link, mass 1.90327; collision mesh filename=meshes/upper_arm_v0/elbow_flex.stl; visual mesh filename=meshes/upper_arm_v0/elbow_flex.stl
- added link l_forearm_cam_frame, mass 0.01
- added link l_forearm_cam_optical_frame
- added link l_forearm_link, mass 2.57968; collision mesh filename=meshes/forearm_v0/forearm.stl; visual mesh filename=meshes/forearm_v0/forearm.stl
- added link l_forearm_roll_link, mass 0.1; collision mesh filename=meshes/upper_arm_v0/forearm_roll.stl; visual mesh filename=meshes/upper_arm_v0/forearm_roll.stl
- added link l_gripper_l_finger_link, mass 0.17126; collision mesh filename=meshes/gripper_v0/ll_finger.stl; visual mesh filename=meshes/gripper_v0/ll_finger.stl
- added link l_gripper_l_finger_tip_frame
- added link l_gripper_l_finger_tip_link, mass 0.04419; collision mesh filename=meshes/gripper_v0/ll_finger_tip.stl; visual mesh filename=meshes/gripper_v0/ll_finger_tip.stl
- added link l_gripper_led_frame
- added link l_gripper_motor_accelerometer_link, mass 0.001; collision box size=0.001 0.001 0.001; visual box size=0.001 0.001 0.001
- added link l_gripper_motor_screw_link, mass 0.01
- added link l_gripper_motor_slider_link, mass 0.01
- added link l_gripper_palm_link, mass 0.58007; collision mesh filename=meshes/gripper_v0/gripper_palm.stl; visual mesh filename=meshes/gripper_v0/gripper_palm.stl
- added link l_gripper_r_finger_link, mass 0.17389; collision mesh filename=meshes/gripper_v0/lr_finger.stl; visual mesh filename=meshes/gripper_v0/lr_finger.stl
- added link l_gripper_r_finger_tip_link, mass 0.04419; collision mesh filename=meshes/gripper_v0/lr_finger_tip.stl; visual mesh filename=meshes/gripper_v0/lr_finger_tip.stl
- added link l_gripper_tool_frame
- added link l_shoulder_lift_link, mass 2.74988; collision mesh filename=meshes/shoulder_v0/shoulder_lift.stl; visual mesh filename=meshes/shoulder_v0/shoulder_lift.stl
- added link l_shoulder_pan_link, mass 25.799322; collision mesh filename=meshes/shoulder_v0/shoulder_pan.stl; visual mesh filename=meshes/shoulder_v0/shoulder_pan.stl
- added link l_upper_arm_link, mass 6.01769; collision mesh filename=meshes/upper_arm_v0/upper_arm.stl; visual mesh filename=meshes/upper_arm_v0/upper_arm.stl
- added link l_upper_arm_roll_link, mass 0.1; collision mesh filename=meshes/shoulder_v0/upper_arm_roll_L.stl; visual mesh filename=meshes/shoulder_v0/upper_arm_roll.stl
- added link l_wrist_flex_link, mass 0.61402; collision mesh filename=meshes/forearm_v0/wrist_flex.stl; visual mesh filename=meshes/forearm_v0/wrist_flex.stl
- added link l_wrist_roll_link, mass 0.1; collision mesh filename=meshes/forearm_v0/wrist_roll_L.stl; visual mesh filename=meshes/forearm_v0/wrist_roll.stl
- added link r_elbow_flex_link, mass 1.90327; collision mesh filename=meshes/upper_arm_v0/elbow_flex.stl; visual mesh filename=meshes/upper_arm_v0/elbow_flex.stl
- added link r_forearm_link, mass 2.57968; collision mesh filename=meshes/forearm_v0/forearm.stl; visual mesh filename=meshes/forearm_v0/forearm.stl
- added link r_forearm_roll_link, mass 0.1; collision mesh filename=meshes/upper_arm_v0/forearm_roll_L.stl; visual mesh filename=meshes/upper_arm_v0/forearm_roll.stl
- added link r_gripper_l_finger_link, mass 0.17126; collision mesh filename=meshes/gripper_v0/rl_finger.stl; visual mesh filename=meshes/gripper_v0/rl_finger.stl
- added link r_gripper_l_finger_tip_link, mass 0.04419; collision mesh filename=meshes/gripper_v0/rl_finger_tip.stl; visual mesh filename=meshes/gripper_v0/rl_finger_tip.stl
- added link r_gripper_led_frame
- added link r_gripper_motor_accelerometer_link, mass 0.001; collision box size=0.001 0.001 0.001; visual box size=0.001 0.001 0.001
- added link r_gripper_motor_screw_link, mass 0.01
- added link r_gripper_motor_slider_link, mass 0.01
- added link r_gripper_palm_link, mass 0.58007; collision mesh filename=meshes/gripper_v0/gripper_palm.stl; visual mesh filename=meshes/gripper_v0/gripper_palm.stl
- added link r_gripper_r_finger_link, mass 0.17389; collision mesh filename=meshes/gripper_v0/rr_finger.stl; visual mesh filename=meshes/gripper_v0/rr_finger.stl
- added link r_gripper_r_finger_tip_link, mass 0.04419; collision mesh filename=meshes/gripper_v0/rr_finger_tip.stl; visual mesh filename=meshes/gripper_v0/rr_finger_tip.stl
- added link r_gripper_tool_frame
- added link r_upper_arm_link, mass 6.01769; collision mesh filename=meshes/upper_arm_v0/upper_arm.stl; visual mesh filename=meshes/upper_arm_v0/upper_arm.stl
- added link r_wrist_flex_link, mass 0.61402; collision mesh filename=meshes/forearm_v0/wrist_flex.stl; visual mesh filename=meshes/forearm_v0/wrist_flex.stl
- added link r_wrist_roll_link, mass 0.1; collision mesh filename=meshes/forearm_v0/wrist_roll.stl; visual mesh filename=meshes/forearm_v0/wrist_roll.stl
- link base_link: geometry collision mesh filename=meshes/base_v0/base_L.stl; visual mesh filename=meshes/base_v0/base.stl
- link bl_caster_l_wheel_link: geometry collision cylinder length=0.034 radius=0.074792; visual mesh filename=meshes/base_v0/wheel.stl
- link bl_caster_r_wheel_link: geometry collision cylinder length=0.034 radius=0.074792; visual mesh filename=meshes/base_v0/wheel.stl
- link br_caster_l_wheel_link: geometry collision cylinder length=0.034 radius=0.074792; visual mesh filename=meshes/base_v0/wheel.stl
- link br_caster_r_wheel_link: geometry collision cylinder length=0.034 radius=0.074792; visual mesh filename=meshes/base_v0/wheel.stl
- link fl_caster_l_wheel_link: geometry collision cylinder length=0.034 radius=0.074792; visual mesh filename=meshes/base_v0/wheel.stl
- link fl_caster_r_wheel_link: geometry collision cylinder length=0.034 radius=0.074792; visual mesh filename=meshes/base_v0/wheel.stl
- link fr_caster_l_wheel_link: geometry collision cylinder length=0.034 radius=0.074792; visual mesh filename=meshes/base_v0/wheel.stl
- link fr_caster_r_wheel_link: geometry collision cylinder length=0.034 radius=0.074792; visual mesh filename=meshes/base_v0/wheel.stl
- link head_pan_link: geometry collision mesh filename=meshes/head_v0/head_pan_L.stl; visual mesh filename=meshes/head_v0/head_pan.stl
- link head_tilt_link: geometry collision mesh filename=meshes/head_v0/head_tilt_L.stl; visual mesh filename=meshes/head_v0/head_tilt.stl
- link laser_tilt_mount_link: geometry collision mesh filename=meshes/tilting_laser_v0/tilting_hokuyo_L.stl; visual mesh filename=meshes/tilting_laser_v0/tilting_hokuyo.stl
- link r_shoulder_lift_link: geometry collision mesh filename=meshes/shoulder_v0/shoulder_lift.stl; visual mesh filename=meshes/shoulder_v0/shoulder_lift.stl
- link r_shoulder_pan_link: geometry collision mesh filename=meshes/shoulder_v0/shoulder_pan.stl; visual mesh filename=meshes/shoulder_v0/shoulder_pan.stl
- link torso_lift_link: geometry collision mesh filename=meshes/torso_v0/torso_lift_L.stl; visual mesh filename=meshes/torso_v0/torso_lift.stl
Joints:
- added joint l_elbow_flex_joint: type revolute, parent l_upper_arm_link, child l_elbow_flex_link, origin xyz=0.4 0 0 rpy=0 0 0, axis 0 1 0, limit lower=-2.3213 upper=0.00 effort=30 velocity=3.3
- added joint l_forearm_cam_frame_joint: type fixed, parent l_forearm_roll_link, child l_forearm_cam_frame, origin xyz=.135 0 .044 rpy=-1.57079632679 -0.562868683768 0
- added joint l_forearm_cam_optical_frame_joint: type fixed, parent l_forearm_cam_frame, child l_forearm_cam_optical_frame, origin xyz=0 0 0 rpy=-1.57079632679 0.0 -1.57079632679
- added joint l_forearm_joint: type fixed, parent l_forearm_roll_link, child l_forearm_link, origin xyz=0 0 0 rpy=0 0 0
- added joint l_forearm_roll_joint: type revolute, parent l_elbow_flex_link, child l_forearm_roll_link, origin xyz=0 0 0 rpy=0 0 0, axis 1 0 0, limit lower=-3.14 upper=3.14 effort=30 velocity=3.6
- added joint l_gripper_joint: type prismatic, parent l_gripper_r_finger_tip_link, child l_gripper_l_finger_tip_frame, axis 0 1 0, limit lower=0.0 upper=0.09 effort=1000.0 velocity=0.2
- added joint l_gripper_l_finger_joint: type revolute, parent l_gripper_palm_link, child l_gripper_l_finger_link, origin xyz=0.07691 0.01 0 rpy=0 0 0, axis 0 0 1, limit lower=0.0 upper=0.548 effort=1000.0 velocity=0.5
- added joint l_gripper_l_finger_tip_joint: type revolute, parent l_gripper_l_finger_link, child l_gripper_l_finger_tip_link, origin xyz=0.09137 0.00495 0 rpy=0 0 0, axis 0 0 -1, limit lower=0.0 upper=0.548 effort=1000.0 velocity=0.5, mimic joint=l_gripper_l_finger_joint multiplier=1 offset=0
- added joint l_gripper_led_joint: type fixed, parent l_gripper_palm_link, child l_gripper_led_frame, origin xyz=0.0513 0.0 .0244
- added joint l_gripper_motor_accelerometer_joint: type fixed, parent l_gripper_palm_link, child l_gripper_motor_accelerometer_link, origin xyz=0 0 0 rpy=0 0 0
- added joint l_gripper_motor_screw_joint: type revolute, parent l_gripper_motor_slider_link, child l_gripper_motor_screw_link, origin xyz=0.0 0 0 rpy=0 0 0, axis 0 1 0, limit lower=-3.14 upper=3.14 effort=1000.0 velocity=0.5
- added joint l_gripper_motor_slider_joint: type prismatic, parent l_gripper_palm_link, child l_gripper_motor_slider_link, origin xyz=0.16828 0 0 rpy=0 0 0, axis 1 0 0, limit lower=-0.1 upper=0.1 effort=1000.0 velocity=0.2
- added joint l_gripper_palm_joint: type fixed, parent l_wrist_roll_link, child l_gripper_palm_link, origin xyz=0 0 0 rpy=0 0 0
- added joint l_gripper_r_finger_joint: type revolute, parent l_gripper_palm_link, child l_gripper_r_finger_link, origin xyz=0.07691 -0.01 0 rpy=0 0 0, axis 0 0 -1, limit lower=0.0 upper=0.548 effort=1000.0 velocity=0.5, mimic joint=l_gripper_l_finger_joint multiplier=1 offset=0
- added joint l_gripper_r_finger_tip_joint: type revolute, parent l_gripper_r_finger_link, child l_gripper_r_finger_tip_link, origin xyz=0.09137 -0.00495 0 rpy=0 0 0, axis 0 0 1, limit lower=0.0 upper=0.548 effort=1000.0 velocity=0.5, mimic joint=l_gripper_l_finger_joint multiplier=1 offset=0
- added joint l_gripper_tool_joint: type fixed, parent l_gripper_palm_link, child l_gripper_tool_frame, origin xyz=0.18 0 0 rpy=0 0 0
- added joint l_shoulder_lift_joint: type revolute, parent l_shoulder_pan_link, child l_shoulder_lift_link, origin xyz=0.1 0 0 rpy=0 0 0, axis 0 1 0, limit lower=-0.5236 upper=1.3963 effort=30 velocity=2.082
- added joint l_shoulder_pan_joint: type revolute, parent torso_lift_link, child l_shoulder_pan_link, origin xyz=0.0 0.188 0.0 rpy=0 0 0, axis 0 0 1, limit lower=-0.714601836603 upper=2.2853981634 effort=30 velocity=2.088
- added joint l_upper_arm_joint: type fixed, parent l_upper_arm_roll_link, child l_upper_arm_link, origin xyz=0 0 0 rpy=0 0 0
- added joint l_upper_arm_roll_joint: type revolute, parent l_shoulder_lift_link, child l_upper_arm_roll_link, origin xyz=0 0 0 rpy=0 0 0, axis 1 0 0, limit lower=-0.8 upper=3.9 effort=30 velocity=3.27
- added joint l_wrist_flex_joint: type revolute, parent l_forearm_link, child l_wrist_flex_link, origin xyz=0.321 0 0 rpy=0 0 0, axis 0 1 0, limit lower=-2.18 upper=0.0 effort=10 velocity=3.078
- added joint l_wrist_roll_joint: type revolute, parent l_wrist_flex_link, child l_wrist_roll_link, origin xyz=0 0 0 rpy=0 0 0, axis 1 0 0, limit lower=-3.14 upper=3.14 effort=10 velocity=3.6
- added joint r_elbow_flex_joint: type revolute, parent r_upper_arm_link, child r_elbow_flex_link, origin xyz=0.4 0 0 rpy=0 0 0, axis 0 1 0, limit lower=-2.3213 upper=0.00 effort=30 velocity=3.3
- added joint r_forearm_joint: type fixed, parent r_forearm_roll_link, child r_forearm_link, origin xyz=0 0 0 rpy=0 0 0
- added joint r_forearm_roll_joint: type revolute, parent r_elbow_flex_link, child r_forearm_roll_link, origin xyz=0 0 0 rpy=0 0 0, axis 1 0 0, limit lower=-3.14 upper=3.14 effort=30 velocity=3.3
- added joint r_gripper_l_finger_joint: type revolute, parent r_gripper_palm_link, child r_gripper_l_finger_link, origin xyz=0.07691 0.01 0 rpy=0 0 0, axis 0 0 -1, limit lower=-0.548 upper=0.0 effort=1000.0 velocity=0.5
- added joint r_gripper_l_finger_tip_joint: type revolute, parent r_gripper_l_finger_link, child r_gripper_l_finger_tip_link, origin xyz=0.09137 0.00495 0 rpy=0 0 0, axis 0 0 -1, limit lower=0.0 upper=0.548 effort=1000.0 velocity=0.5, mimic joint=r_gripper_l_finger_joint multiplier=1 offset=0
- added joint r_gripper_led_joint: type fixed, parent r_gripper_palm_link, child r_gripper_led_frame, origin xyz=0.0513 0.0 .0244
- added joint r_gripper_motor_accelerometer_joint: type fixed, parent r_gripper_palm_link, child r_gripper_motor_accelerometer_link, origin xyz=0 0 0 rpy=0 0 0
- added joint r_gripper_motor_screw_joint: type revolute, parent r_gripper_motor_slider_link, child r_gripper_motor_screw_link, origin xyz=0.0 0 0 rpy=0 0 0, axis 0 1 0, limit lower=-3.14 upper=3.14 effort=1000.0 velocity=0.5
- added joint r_gripper_motor_slider_joint: type prismatic, parent r_gripper_palm_link, child r_gripper_motor_slider_link, origin xyz=0.16828 0 0 rpy=0 0 0, axis 1 0 0, limit lower=-0.1 upper=0.1 effort=1000.0 velocity=0.2
- added joint r_gripper_palm_joint: type fixed, parent r_wrist_roll_link, child r_gripper_palm_link, origin xyz=0 0 0 rpy=0 0 0
- added joint r_gripper_r_finger_joint: type revolute, parent r_gripper_palm_link, child r_gripper_r_finger_link, origin xyz=0.07691 -0.01 0 rpy=0 0 0, axis 0 0 1, limit lower=-0.548 upper=0 effort=1000.0 velocity=0.5
- added joint r_gripper_r_finger_tip_joint: type revolute, parent r_gripper_r_finger_link, child r_gripper_r_finger_tip_link, origin xyz=0.09137 -0.00495 0 rpy=0 0 0, axis 0 0 1, limit lower=0.0 upper=0.548 effort=1000.0 velocity=0.5, mimic joint=r_gripper_l_finger_joint multiplier=1 offset=0
- added joint r_gripper_tool_joint: type fixed, parent r_gripper_palm_link, child r_gripper_tool_frame, origin xyz=0.18 0 0 rpy=0 0 0
- added joint r_upper_arm_joint: type fixed, parent r_upper_arm_roll_link, child r_upper_arm_link, origin xyz=0 0 0 rpy=0 0 0
- added joint r_wrist_flex_joint: type revolute, parent r_forearm_link, child r_wrist_flex_link, origin xyz=0.321 0 0 rpy=0 0 0, axis 0 1 0, limit lower=-2.18 upper=0.0 effort=10 velocity=3.078
- added joint r_wrist_roll_joint: type revolute, parent r_wrist_flex_link, child r_wrist_roll_link, origin xyz=0 0 0 rpy=0 0 0, axis 1 0 0, limit lower=-3.14 upper=3.14 effort=10 velocity=3.6
