Commit message: Fix experiments

File: data/robots/drone/dddk_inner_sphere.urdf (robot description, URDF)
Before this commit: robot sphere, 1 links, 0 joints
Links:
- link body: geometry collision sphere radius=0.04; visual sphere radius=0.04

Commit message: Add construction time display to GUI

File: data/robots/drone/dddk_inner_sphere.urdf (robot description, URDF)
Before this commit: robot sphere, 1 links, 0 joints
Links:
- link body: geometry collision sphere radius=0.06; visual sphere radius=0.06
