Commit message: ContactConstraint contd

File: data/robots/planar/2dof_manip_no_endeffector.urdf (robot description, URDF)
Before this commit: robot planar_manipulator/2dof_manip_no_endeffector, 5 links, 4 joints
Links:
- link jlink0: geometry visual cylinder length=0.1 radius=0.2

Commit message: Minor

File: data/robots/planar/2dof_manip_no_endeffector.urdf (robot description, URDF)
Before this commit: robot planar_manipulator/2dof_manip_no_endeffector, 5 links, 4 joints
Links:
- link jlink0: geometry 

Commit message: Multiple Contacts wip

File: data/robots/planar/2dof_manip_no_endeffector.urdf (robot description, URDF)
Before this commit: robot planar_manipulator/2dof_manip_no_endeffector, 5 links, 4 joints
Links:
- link link0: geometry collision box size=0.1 1.5 0.1; visual box size=0.1 1.5 0.1
- link link1: geometry collision box size=0.1 1.5 0.1; visual box size=0.1 1.5 0.1

Commit message: Transition Constraint new Wip

File: data/robots/planar/2dof_manip_no_endeffector.urdf (robot description, URDF)
Before this commit: robot planar_manipulator/2dof_manip_no_endeffector, 5 links, 4 joints
Links:
- link jlink1: geometry collision cylinder length=0.1 radius=0.15; visual cylinder length=0.1 radius=0.15
- link link1: geometry collision box size=0.2 1.5 0.1; visual box size=0.2 1.5 0.1
