Commit message: Fix sig abort error (specified correct nr of links)

File: data/robots/magneto/magneto0.urdf (robot description, URDF)
Before this commit: robot magneto/magneto0, 3 links, 2 joints
Joints:
- removed joint joint_foot_leg_Z
- removed joint joint_leg_foot2_Z
- added joint joint_revolute_foot_leg_Z: type revolute, parent foot, child leg, origin xyz=0 0 0 rpy=0 0 0, axis 0 1 0, limit lower=-1.57 upper=1.57 effort=0.01 velocity=100
- added joint joint_revolute_leg_foot2_Z: type revolute, parent leg, child foot2, origin xyz=0.17 0 0 rpy=0 0 0, axis 0 1 0, limit lower=-1.57 upper=1.57 effort=0.01 velocity=100

File: data/robots/magneto/magneto1.urdf (robot description, URDF)
Before this commit: robot magneto/magneto1, 3 links, 2 joints
Joints:
- removed joint joint_foot_leg_Z
- removed joint joint_leg_foot2_Z
- added joint joint_revolute_foot_leg_Z: type revolute, parent foot, child leg, origin xyz=0 0 0 rpy=0 0 0, axis 0 1 0, limit lower=-1.57 upper=1.57 effort=0.01 velocity=100
- added joint joint_revolute_leg_foot2_Z: type revolute, parent leg, child foot2, origin xyz=0.6 0 0 rpy=0 0 0, axis 0 1 0, limit lower=-1.57 upper=1.57 effort=0.01 velocity=100

File: data/robots/magneto/magneto2.urdf (robot description, URDF)
Before this commit: robot magneto/magneto2, 7 links, 6 joints
Joints:
- removed joint joint_foot_leg1
- removed joint joint_leg1_joint1
- removed joint joint_leg2_joint1_Z
- removed joint joint_leg2_joint2
- removed joint joint_leg3_foot2
- removed joint joint_leg3_joint2_Z
- added joint joint_fixed_foot_leg1: type fixed, parent foot, child leg1, origin xyz=0 0 0 rpy=0 0 0
- added joint joint_fixed_leg1_joint1: type fixed, parent leg1, child joint1, origin xyz=0 0 0 rpy=0 0 0
- added joint joint_fixed_leg2_joint2: type fixed, parent leg2, child joint2, origin xyz=0 0 0 rpy=0 0 0
- added joint joint_fixed_leg3_foot2: type fixed, parent leg3, child foot2, origin xyz=0 0 0 rpy=0 0 0
- added joint joint_revolute_joint1_leg2_Z: type revolute, parent joint1, child leg2, origin xyz=0.29 0 0 rpy=0 0 0, axis 0 1 0, limit lower=-1.57 upper=1.57 effort=0.01 velocity=100
- added joint joint_revolute_joint2_leg3_Z: type revolute, parent joint2, child leg3, origin xyz=0.48000000000000004 0 0 rpy=0 0 0, axis 0 1 0, limit lower=-1.57 upper=1.57 effort=0.01 velocity=100
