Commit message: Repair cable robot

File: data/robots/cable/cable.urdf (robot description, URDF)
Before this commit: robot cable/cable, 178 links, 177 joints
Joints:
- joint joint_fixed_body0_body1_joint_link: origin xyz=-0.03001 0 0 rpy=0 0 0 -> xyz=-0.08001 0 0 rpy=0 0 0

File: data/robots/cable/cable_10_segments.urdf (robot description, URDF)
Before this commit: robot cable/cable_10_segments, 31 links, 30 joints
Joints:
- joint joint_fixed_body0_body1_joint_link: origin xyz=-0.03001 0 0 rpy=0 0 0 -> xyz=-0.08001 0 0 rpy=0 0 0

File: data/robots/cable/cable_11_segments.urdf (robot description, URDF)
Before this commit: robot cable/cable_11_segments, 34 links, 33 joints
Joints:
- joint joint_fixed_body0_body1_joint_link: origin xyz=-0.03001 0 0 rpy=0 0 0 -> xyz=-0.08001 0 0 rpy=0 0 0

File: data/robots/cable/cable_12_segments.urdf (robot description, URDF)
Before this commit: robot cable/cable_12_segments, 37 links, 36 joints
Joints:
- joint joint_fixed_body0_body1_joint_link: origin xyz=-0.03001 0 0 rpy=0 0 0 -> xyz=-0.08001 0 0 rpy=0 0 0

File: data/robots/cable/cable_13_segments.urdf (robot description, URDF)
Before this commit: robot cable/cable_13_segments, 40 links, 39 joints
Joints:
- joint joint_fixed_body0_body1_joint_link: origin xyz=-0.03001 0 0 rpy=0 0 0 -> xyz=-0.08001 0 0 rpy=0 0 0

File: data/robots/cable/cable_14_segments.urdf (robot description, URDF)
Before this commit: robot cable/cable_14_segments, 43 links, 42 joints
Joints:
- joint joint_fixed_body0_body1_joint_link: origin xyz=-0.03001 0 0 rpy=0 0 0 -> xyz=-0.08001 0 0 rpy=0 0 0

File: data/robots/cable/cable_15_segments.urdf (robot description, URDF)
Before this commit: robot cable/cable_15_segments, 46 links, 45 joints
Joints:
- joint joint_fixed_body0_body1_joint_link: origin xyz=-0.03001 0 0 rpy=0 0 0 -> xyz=-0.08001 0 0 rpy=0 0 0

File: data/robots/cable/cable_16_segments.urdf (robot description, URDF)
Before this commit: robot cable/cable_16_segments, 49 links, 48 joints
Joints:
- joint joint_fixed_body0_body1_joint_link: origin xyz=-0.03001 0 0 rpy=0 0 0 -> xyz=-0.08001 0 0 rpy=0 0 0

File: data/robots/cable/cable_17_segments.urdf (robot description, URDF)
Before this commit: robot cable/cable_17_segments, 52 links, 51 joints
Joints:
- joint joint_fixed_body0_body1_joint_link: origin xyz=-0.03001 0 0 rpy=0 0 0 -> xyz=-0.08001 0 0 rpy=0 0 0

File: data/robots/cable/cable_18_segments.urdf (robot description, URDF)
Before this commit: robot cable/cable_18_segments, 55 links, 54 joints
Joints:
- joint joint_fixed_body0_body1_joint_link: origin xyz=-0.03001 0 0 rpy=0 0 0 -> xyz=-0.08001 0 0 rpy=0 0 0

File: data/robots/cable/cable_19_segments.urdf (robot description, URDF)
Before this commit: robot cable/cable_19_segments, 58 links, 57 joints
Joints:
- joint joint_fixed_body0_body1_joint_link: origin xyz=-0.03001 0 0 rpy=0 0 0 -> xyz=-0.08001 0 0 rpy=0 0 0

File: data/robots/cable/cable_1_segments.urdf (robot description, URDF)
Before this commit: robot cable/cable_1_segments, 4 links, 3 joints
Joints:
- joint joint_fixed_body0_body1_joint_link: origin xyz=-0.03001 0 0 rpy=0 0 0 -> xyz=-0.08001 0 0 rpy=0 0 0

File: data/robots/cable/cable_20_segments.urdf (robot description, URDF)
Before this commit: robot cable/cable_20_segments, 61 links, 60 joints
Joints:
- joint joint_fixed_body0_body1_joint_link: origin xyz=-0.03001 0 0 rpy=0 0 0 -> xyz=-0.08001 0 0 rpy=0 0 0

File: data/robots/cable/cable_21_segments.urdf (robot description, URDF)
Before this commit: robot cable/cable_21_segments, 64 links, 63 joints
Joints:
- joint joint_fixed_body0_body1_joint_link: origin xyz=-0.03001 0 0 rpy=0 0 0 -> xyz=-0.08001 0 0 rpy=0 0 0

File: data/robots/cable/cable_22_segments.urdf (robot description, URDF)
Before this commit: robot cable/cable_22_segments, 67 links, 66 joints
Joints:
- joint joint_fixed_body0_body1_joint_link: origin xyz=-0.03001 0 0 rpy=0 0 0 -> xyz=-0.08001 0 0 rpy=0 0 0

File: data/robots/cable/cable_23_segments.urdf (robot description, URDF)
Before this commit: robot cable/cable_23_segments, 70 links, 69 joints
Joints:
- joint joint_fixed_body0_body1_joint_link: origin xyz=-0.03001 0 0 rpy=0 0 0 -> xyz=-0.08001 0 0 rpy=0 0 0

File: data/robots/cable/cable_24_segments.urdf (robot description, URDF)
Before this commit: robot cable/cable_24_segments, 73 links, 72 joints
Joints:
- joint joint_fixed_body0_body1_joint_link: origin xyz=-0.03001 0 0 rpy=0 0 0 -> xyz=-0.08001 0 0 rpy=0 0 0

File: data/robots/cable/cable_25_segments.urdf (robot description, URDF)
Before this commit: robot cable/cable_25_segments, 76 links, 75 joints
Joints:
- joint joint_fixed_body0_body1_joint_link: origin xyz=-0.03001 0 0 rpy=0 0 0 -> xyz=-0.08001 0 0 rpy=0 0 0

File: data/robots/cable/cable_26_segments.urdf (robot description, URDF)
Before this commit: robot cable/cable_26_segments, 79 links, 78 joints
Joints:
- joint joint_fixed_body0_body1_joint_link: origin xyz=-0.03001 0 0 rpy=0 0 0 -> xyz=-0.08001 0 0 rpy=0 0 0

File: data/robots/cable/cable_27_segments.urdf (robot description, URDF)
Before this commit: robot cable/cable_27_segments, 82 links, 81 joints
Joints:
- joint joint_fixed_body0_body1_joint_link: origin xyz=-0.03001 0 0 rpy=0 0 0 -> xyz=-0.08001 0 0 rpy=0 0 0
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